File: PCB/FPGA-power.kicad_sch (KiCad schematic)
At the start: 27 parts, among them U1 XC7A50T-FGG484

Commit message: renaming passives without unit for cleaner schematic
Parts:
- C16, C17, C18, C19, C20, C25, C27, C28, C29, C30, C31, C35, C36, C38, C39: value 470nF -> 470n
- C21, C22, C23, C32, C33, C37, C40: value 4.7uF -> 4.7u
- C24: value 330uF -> 330u
- C26: value 100uF -> 100u
- C34: value 47uF -> 47u
Changed lines of the file:
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@@
 			)
 		)
-		(property "Value" "470nF"
+		(property "Value" "470n"
 			(at 152.146 52.578 0)
 			(effects
@@
 			)
 		)
-		(property "Value" "47uF"
+		(property "Value" "47u"
 			(at 89.916 52.578 0)
 			(effects
@@
 			)
 		)
-		(property "Value" "470nF"
+		(property "Value" "470n"
 			(at 143.256 52.578 0)
 			(effects
@@
 			)
 		)
-		(property "Value" "4.7uF"
+		(property "Value" "4.7u"
 			(at 304.546 52.578 0)
 			(effects
@@
 			)
 		)
-		(property "Value" "4.7uF"
+		(property "Value" "4.7u"
 			(at 295.656 52.578 0)
 			(effects
@@
 			)
 		)
-		(property "Value" "330uF"
+		(property "Value" "330u"
 			(at 322.326 52.578 0)
 			(effects
@@
 			)
 		)
-		(property "Value" "4.7uF"
+		(property "Value" "4.7u"
 			(at 98.806 52.578 0)
 			(effects
@@
 			)
 		)
-		(property "Value" "100uF"
+		(property "Value" "100u"
 			(at 143.256 80.518 0)
 			(effects
@@
 			)
 		)
-		(property "Value" "4.7uF"
+		(property "Value" "4.7u"
 			(at 128.016 246.888 0)
 			(effects
@@
 			)
 		)
-		(property "Value" "470nF"
+		(property "Value" "470n"
 			(at 152.146 80.518 0)
 			(effects
@@
 			)
 		)
-		(property "Value" "470nF"
+		(property "Value" "470n"
 			(at 260.096 52.578 0)
 			(effects
@@
 			)
 		)
-		(property "Value" "470nF"
+		(property "Value" "470n"
 			(at 125.476 52.578 0)
 			(effects
@@
 			)
 		)
-		(property "Value" "4.7uF"
+		(property "Value" "4.7u"
 			(at 107.696 52.578 0)
 			(effects
@@
 			)
 		)
-		(property "Value" "470nF"
+		(property "Value" "470n"
 			(at 268.986 52.578 0)
 			(effects
@@
 			)
 		)
-		(property "Value" "470nF"
+		(property "Value" "470n"
 			(at 136.906 246.888 0)
 			(effects
@@
 			)
 		)
-		(property "Value" "470nF"
+		(property "Value" "470n"
 			(at 116.586 52.578 0)
 			(effects
@@
 			)
 		)
-		(property "Value" "4.7uF"
+		(property "Value" "4.7u"
 			(at 281.686 246.888 0)
 			(effects
@@
 			)
 		)
-		(property "Value" "470nF"
+		(property "Value" "470n"
 			(at 286.766 52.578 0)
 			(effects
@@
 			)
 		)
-		(property "Value" "470nF"
+		(property "Value" "470n"
 			(at 272.796 246.888 0)
 			(effects
@@
 			)
 		)
-		(property "Value" "470nF"
+		(property "Value" "470n"
 			(at 263.906 246.888 0)
 			(effects
@@
 			)
 		)
-		(property "Value" "4.7uF"
+		(property "Value" "4.7u"
 			(at 313.436 52.578 0)
 			(effects
@@
 			)
 		)
-		(property "Value" "470nF"
+		(property "Value" "470n"
 			(at 251.206 52.578 0)
 			(effects
@@
 			)
 		)
-		(property "Value" "470nF"
+		(property "Value" "470n"
 			(at 145.796 246.888 0)
 			(effects
@@
 			)
 		)
-		(property "Value" "470nF"
+		(property "Value" "470n"
 			(at 134.366 52.578 0)
 			(effects
@@
 			)
 		)
-		(property "Value" "470nF"
+		(property "Value" "470n"
 			(at 277.876 52.578 0)
 			(effects

Commit message: journaling about finding a buck converter
Other:
- note added: "FERRITE BEADS AND ANALOG RAILS"
Changed lines of the file:
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@@
 	(generator_version "9.0")
 	(paper "A3")
+	(text "FERRITE BEADS AND ANALOG RAILS"
+		(exclude_from_sim no)
+		(at 76.2 140.208 0)
+		(effects
+			(font
+				(size 3.81 3.81)
+			)
+		)
+	)
 	(text "VCCINT & VCCBRAM & VMGTAVCC = 1V\nVCCAUX = 1V8\nVCCO = 3V3\nVMGTAVTT = 1V2\nDDR3 Voltage = 1V5"
 		(exclude_from_sim no)
