File: PCB/power.kicad_sch (KiCad schematic)
At the start: 23 parts, among them U2 LTC3370

Commit message: custom MAX20029 symbol
Parts:
- removed C42, C43, C44: 22u, symbol Device:C
- removed C45: 10u, symbol Device:C
- removed C46, C47, C48, C49: 47u, symbol Device:C
- removed L2, L3, L4: 2.2u, symbol Device:L
- removed R2: 49.9k, symbol Device:R
- removed R3, R5, R7, R9: 100k, symbol Device:R
- removed R4: 24.9k, symbol Device:R
- removed R6: 88.7k, symbol Device:R
- removed R8: 124k, symbol Device:R
- removed TP1: Test Temperature, symbol Connector:TestPoint
- removed U2: LTC3370, Package_DFN_QFN:QFN-32-1EP_5x5mm_P0.5mm_EP3.45x3.45mm_ThermalVias, symbol FPGA Accelerator:LTC3370
- added U2: MAX20029ATIA/V+, easyeda2kicad:QFN-28_L5.0-W5.0-P0.50-TL-EP3.2, symbol FPGA Accelerator:MAX20029
- C41: value 22u -> C
- L1: value 2.2u -> L; DK P# 2457-XAL4020-222MEC-ND -> (none); LCSC C3151182 -> (none); MPN XAL4020-222MEC -> (none)
Connections:
- net +3V3 is gone; now on an unnamed net: C41.1
- net at L1.1: now also U2.3 (LX1)
- net +1V2: no longer names the net of L1.2
- net +1V2: now also U2.28 (OUTS1)
Other:
- note removed: "One 22uF per 2A channel VIN, 10uF on VCC"
- note removed: "VCCINT & VCCBRAM & VMGTAVCC = 1V VCCAUX = 1V8 VCCO = 3V3 VMGTAVTT = 1V2 DDR3 Voltage = 1V5"
- note removed: "VOUT = VFB(1 + R2/R1), VFB = 0.8V"

Commit message: halfway done buck wiring
Parts:
- removed L1: L, symbol Device:L
- added C42, C43, C44: 4.7u, symbol Device:C
- added R2, R3, R4, R5: 10K, symbol Device:R
- C41: value C -> 4.7u
Connections:
- net GND: now also C42.2, C43.2, C44.2
- net at U2.28 (OUTS1): no longer C41.1
- net +3V3: now reaches U2.1 (EN1)
- net +3V3: now also C41.1, U2.15 (PV3), U2.2 (PV1), U2.20 (PV4), U2.26 (VA), U2.7 (PV2), C42.1, C43.1, C44.1, R2.1, R3.1, R4.1, R5.1
- net at U2.10 (PG2): now also U2.13 (EN3), R3.2
- net at U2.12 (PG3): now also U2.21 (EN4), R4.2
- net at U2.23 (PG4): now also R5.2
- net at U2.27 (PG1): now also U2.9 (EN2), R2.2
Other:
- moved on the sheet: U2

Commit message: working on buck, changing values to proper standard, ie 4.7 -> 4u7
Parts:
- added C45: 47u, symbol Device:C
- added C46: 4u7, symbol Device:C
- added L1: 1.5u, symbol Device:L
- C41, C42, C43, C44: value 4.7u -> 4u7
Connections:
- net +3V3: now also C46.1
- net GND: now also U2.11 (GND), U2.17 (PGND3), U2.18 (PGND4), U2.24 (AGND), U2.25 (SYNC), U2.29 (EP), U2.4 (PGND1), U2.5 (PGND2), C45.2, C46.2
- net +1V0: now reaches U2.28 (OUTS1)
- net +1V0: now also C45.1, L1.2
- net at U2.3 (LX1): now also L1.1
Other:
- note added: "4.7uF per PV and VA"
- moved on the sheet: R2, R3, R4, R5

Commit message: basic wiring finished
Parts:
- added C47, C48, C50, C52: ~, symbol Device:C
- added C49, C51, C53: 47u, symbol Device:C
- added L2, L3, L4: 1.5u, symbol Device:L
- added R10, R11, R12, R13: 10K, symbol Device:R
- added R6, R7, R8, R9: R, symbol Device:R
- L1: LCSC (none) -> C42100; MPN (none) -> SWPA4030S1R5NT
- R2, R3, R4, R5: value 10K -> R
Connections:
- net +1V0: now also R2.1, R2.2, R3.1, C47.1, C47.2
- net +1V2: now also R4.1, R4.2, R5.1, U2.8 (OUTS2), C48.1, C48.2, C49.1, L2.2
- net +1V5: now also U2.22 (OUTS4), C50.1, C50.2, C51.1, L3.2, R6.1, R6.2, R7.1
- net +1V8: now also U2.14 (OUTS3), C52.1, C52.2, C53.1, L4.2, R8.1, R8.2, R9.1
- net +3V3: now also R10.1, R11.1, R12.1, R13.1; no longer R2.1, R3.1, R4.1, R5.1
- net GND: now also R3.2, R5.2, C49.2, C51.2, C53.2, R7.2, R9.2
- net at U2.27 (PG1), U2.9 (EN2): now also R10.2; no longer R2.2
- net at U2.10 (PG2), U2.13 (EN3): now also R11.2; no longer R3.2
- net at U2.12 (PG3), U2.21 (EN4): now also R12.2; no longer R4.2
- net at U2.16 (LX3): now also L4.1
- net at U2.19 (LX4): now also L3.1
- net at U2.23 (PG4): now also R13.2; no longer R5.2
- net at U2.6 (LX2): now also L2.1
Other:
- note added: "Default Switching Freq >"
- note added: "SEQUENCE VCC -> 1V0 -> 1V2 -> 1V5 -> 1V8"
- moved on the sheet: C41, C42, C43, C44, C45, C46, L1, U2

Commit message: finished wiring the buck converter
Parts:
- removed C47: ~, symbol Device:C
- removed R2, R3: R, symbol Device:R
- C48: value ~ -> 68pF
- C50: value ~ -> 33p
- C52: value ~ -> 22pF
- R4: value R -> 2k
- R5, R7, R9: value R -> 10k
- R6: value R -> 5k
- R8: value R -> 8k
Other:
- note added: "< Default VOUT is 1V"
- note added: "Divider: R1 = R2[( VOUT / 1 ) − 1]"
- note added: "Frequency compensation: C1 = 15e-12(R2 / R1)"
- moved on the sheet: C45

Commit message: cleaning stuff up, fixing power sequencing and decoupling
Parts:
- C46: value 4u7 -> 1u
Connections:
- net +1V5: now also U2.14 (OUTS3); no longer U2.22 (OUTS4)
- net +1V8: now also U2.22 (OUTS4); no longer U2.14 (OUTS3)
- net at L3.1: now also U2.16 (LX3); no longer U2.19 (LX4)
- net at L4.1: now also U2.19 (LX4); no longer U2.16 (LX3)
Other:
- note added: "4.7uF per PV and 1u for VA"
- note added: "SEQUENCE VCC -> 1V0 -> 1V2 -> 1V8 -> 1V5"
- note added: "VCCINT & VCCBRAM & VMGTAVCC = 1V VCCAUX = 1V8 VCCO = 3V3 VMGTAVTT = 1V2 DDR3 Voltage = 1V5"
- note removed: "4.7uF per PV and VA"
- note removed: "SEQUENCE VCC -> 1V0 -> 1V2 -> 1V5 -> 1V8"
- moved on the sheet: C41, C42, C43, C44, C46, C50, C51, C52, C53, L3, L4, R6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

Commit message: working on wiring the FT2232H, also modified some values to follow more standard conventions
Parts:
- R10, R11, R12, R13: value 10K -> 10k
Other:
- note added: "STATUS LED?"
Changed lines of the file:
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@@
 		)
 	)
+	(text "STATUS LED?"
+		(exclude_from_sim no)
+		(at 71.882 241.554 0)
+		(effects
+			(font
+				(size 5.08 5.08)
+			)
+		)
+	)
 	(text "Frequency compensation: C1 = 15e-12(R2 / R1)"
 		(exclude_from_sim no)
@@
 			)
 		)
-		(property "Value" "10K"
+		(property "Value" "10k"
 			(at 165.1 109.2199 0)
 			(effects
@@
 			)
 		)
-		(property "Value" "10K"
+		(property "Value" "10k"
 			(at 134.62 109.2199 0)
 			(effects
@@
 			)
 		)
-		(property "Value" "10K"
+		(property "Value" "10k"
 			(at 154.94 109.2199 0)
 			(effects
@@
 			)
 		)
-		(property "Value" "10K"
+		(property "Value" "10k"
 			(at 144.78 109.2199 0)
 			(effects
