File: PCB/power.kicad_sch (KiCad schematic)
At the start: 38 parts, among them U2 MAX20029ATIA/V+, U5 TPS2121RUXR

Commit message: USB ESD protection
Other:
- note removed: "STATUS LED?"
- note removed: "VCCINT & VCCBRAM & VMGTAVCC = 1V VCCAUX = 1V8 VCCO = 3V3 VMGTAVTT = 1V2 DDR3 Voltage = 1V5"
Changed lines of the file:
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@@
 		)
 	)
-	(text "VCCINT & VCCBRAM & VMGTAVCC = 1V\nVCCAUX = 1V8\nVCCO = 3V3\nVMGTAVTT = 1V2\nDDR3 Voltage = 1V5"
-		(exclude_from_sim no)
-		(at 18.034 30.226 0)
-		(effects
-			(font
-				(size 2.54 2.54)
-			)
-			(justify left)
-		)
-	)
-	(text "STATUS LED?"
-		(exclude_from_sim no)
-		(at 71.882 241.554 0)
-		(effects
-			(font
-				(size 5.08 5.08)
-			)
-		)
-	)
 	(text "Around 1ms ramp up - 47nF\nAround 3A min, 4A max current limiting\n"
 		(exclude_from_sim no)
@@
 	(wire
 		(pts
+			(xy 113.03 172.72) (xy 113.03 171.45)
+		)
+		(stroke
+			(width 0)
+			(type default)
+		)
+	)
+	(wire
+		(pts
 			(xy 212.09 100.33) (xy 212.09 102.87)
 		)
@@
 	(wire
 		(pts
-			(xy 113.03 171.45) (xy 113.03 170.18)
-		)
-		(stroke
-			(width 0)
-			(type default)
-		)
-	)
-	(wire
-		(pts
 			(xy 212.09 111.76) (xy 212.09 196.85)
 		)
@@
 	(symbol
 		(lib_id "power:GND")
-		(at 113.03 171.45 0)
+		(at 113.03 172.72 0)
 		(unit 1)
 		(exclude_from_sim no)
@@
 		(fields_autoplaced yes)
 		(property "Reference" "#PWR067"
-			(at 113.03 177.8 0)
+			(at 113.03 179.07 0)
 			(effects
 				(font
@@
 		)
 		(property "Value" "GND"
-			(at 113.03 176.53 0)
+			(at 113.03 177.8 0)
 			(effects
 				(font
@@
 		)
 		(property "Footprint" ""
-			(at 113.03 171.45 0)
+			(at 113.03 172.72 0)
 			(effects
 				(font
@@
 		)
 		(property "Datasheet" ""
-			(at 113.03 171.45 0)
+			(at 113.03 172.72 0)
 			(effects
 				(font
@@
 		)
 		(property "Description" "Power symbol creates a global label with name \"GND\" , ground"
-			(at 113.03 171.45 0)
+			(at 113.03 172.72 0)
 			(effects
 				(font

Commit message: wired the 100MHz clock for PLL's
Connections:
- net BUCK_PG4: now reaches R13.2, U2.23 (PG4)
Changed lines of the file:
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@@
+	)
+	(junction
+		(at 212.09 196.85)
+		(diameter 0)
+		(color 0 0 0 0)
 	)
 	(junction
@@
 	(wire
 		(pts
+			(xy 204.47 196.85) (xy 212.09 196.85)
+		)
+		(stroke
+			(width 0)
+			(type default)
+		)
+	)
+	(wire
+		(pts
 			(xy 312.42 149.86) (xy 312.42 151.13)
 		)
@@
 		)
 	)
+	(hierarchical_label "BUCK_PG4"
+		(shape output)
+		(at 204.47 196.85 180)
+		(effects
+			(font
+				(size 1.27 1.27)
+			)
+			(justify right)
+		)
+	)

Commit message: cleaning  up the schematic some more before sharing
Parts:
- added D4: LED, symbol Device:LED
- added R77: 1k, symbol Device:R
Connections:
- net +3V3: now also D4.2 (A)
- net GND: now also R77.2
- new net: D4.1 (K), R77.1

Commit message: added basic capacitor footprints
Parts:
- C41, C42, C43, C44, C66, C68, C70: footprint (none) -> Capacitor_SMD:C_0603_1608Metric
- C67, C69, C71: footprint (none) -> Capacitor_SMD:C_0201_0603Metric
- L1, L2, L3, L4: value 1.5u -> 1u5
Connections:
- net +1V5: now also L4.2; no longer L3.2
- net +1V8: now also L3.2; no longer L4.2
- net at U2.16 (LX3): now also L4.1; no longer L3.1
- net at U2.19 (LX4): now also L3.1; no longer L4.1

Commit message: LED parts and inductor footprints
Parts:
- D4: value LED -> KT-0805G; footprint (none) -> LED_SMD:LED_0805_2012Metric; LCSC (none) -> C2297; MPN (none) -> KT-0805G
- L1, L2, L3, L4: footprint (none) -> Inductor_SMD:L_Sunlord_SWPA4030S

Commit message: adding most of the resistor footprints
Parts:
- R10, R11, R12, R13, R34, R5, R7, R9: footprint (none) -> Resistor_SMD:R_0402_1005Metric
- R6: value 5k -> 4k99; footprint (none) -> Resistor_SMD:R_0603_1608Metric
- R8: value 8k -> 8k2; footprint (none) -> Resistor_SMD:R_0603_1608Metric
Other:
- note added: "< 0603 footprint, and dif divider because JLC basic! <"
- moved on the sheet: C48, C49, C50, C51, C52, C53

Commit message: finisehed upassigning resistor footprints
Parts:
- C72: footprint (none) -> Capacitor_SMD:C_0603_1608Metric
- R33: footprint (none) -> Resistor_SMD:R_0603_1608Metric
- R35: value 5k -> 4k99; footprint (none) -> Resistor_SMD:R_0603_1608Metric
- R4, R77: footprint (none) -> Resistor_SMD:R_0402_1005Metric
Changed lines of the file:
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@@
 			)
 		)
-		(property "Footprint" ""
+		(property "Footprint" "Capacitor_SMD:C_0603_1608Metric"
 			(at 140.6652 173.99 0)
 			(effects
@@
 			)
 		)
-		(property "Footprint" ""
+		(property "Footprint" "Resistor_SMD:R_0402_1005Metric"
 			(at 233.68 74.168 90)
 			(effects
@@
 			)
 		)
-		(property "Footprint" ""
+		(property "Footprint" "Resistor_SMD:R_0603_1608Metric"
 			(at 126.492 171.45 90)
 			(effects
@@
 			)
 		)
-		(property "Value" "5k"
+		(property "Value" "4k99"
 			(at 96.52 128.2699 0)
 			(effects
@@
 			)
 		)
-		(property "Footprint" ""
+		(property "Footprint" "Resistor_SMD:R_0603_1608Metric"
 			(at 92.202 127 90)
 			(effects
@@
 			)
 		)
-		(property "Footprint" ""
+		(property "Footprint" "Resistor_SMD:R_0402_1005Metric"
 			(at 310.642 144.78 90)
 			(effects
