File: PCB/power.kicad_sch (KiCad schematic)
At the start: 40 parts, among them U2 MAX20029ATIA/V+, U5 TPS2121RUXR

Commit message: fixing up my buck converter, getting ready for power routing
Connections:
- net at L3.1: now also U2.16 (LX3); no longer U2.19 (LX4)
- net at C50.2, R6.2, R7.1: now also U2.22 (OUTS4); no longer U2.14 (OUTS3)
- net at L4.1: now also U2.19 (LX4); no longer U2.16 (LX3)
- net at C52.2, R8.2, R9.1: now also U2.14 (OUTS3); no longer U2.22 (OUTS4)

Commit message: buck converter and power OR layout
Parts:
- added C112: 470n, Capacitor_SMD:C_0201_0603Metric, symbol Device:C
Connections:
- net +3V3: now also C112.1
- net GND: now also C112.2
Other:
- moved on the sheet: C70, C71
Changed lines of the file:
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@@
 	)
 	(junction
-		(at 127 121.92)
+		(at 134.62 134.62)
+		(diameter 0)
+		(color 0 0 0 0)
+	)
+	(junction
+		(at 134.62 121.92)
 		(diameter 0)
 		(color 0 0 0 0)
@@
 	)
 	(junction
-		(at 135.89 134.62)
+		(at 143.51 134.62)
 		(diameter 0)
 		(color 0 0 0 0)
@@
 	)
 	(junction
-		(at 135.89 121.92)
+		(at 143.51 121.92)
+		(diameter 0)
+		(color 0 0 0 0)
+	)
+	(junction
+		(at 127 121.92)
 		(diameter 0)
 		(color 0 0 0 0)
@@
 	(wire
 		(pts
+			(xy 127 134.62) (xy 134.62 134.62)
+		)
+		(stroke
+			(width 0)
+			(type default)
+		)
+	)
+	(wire
+		(pts
 			(xy 288.29 76.2) (xy 297.18 76.2)
 		)
@@
 	(wire
 		(pts
-			(xy 135.89 132.08) (xy 135.89 134.62)
+			(xy 143.51 132.08) (xy 143.51 134.62)
 		)
 		(stroke
@@
 	(wire
 		(pts
-			(xy 127 121.92) (xy 110.49 121.92)
+			(xy 134.62 121.92) (xy 127 121.92)
 		)
 		(stroke
@@
 	(wire
 		(pts
-			(xy 135.89 119.38) (xy 135.89 121.92)
+			(xy 143.51 119.38) (xy 143.51 121.92)
 		)
 		(stroke
@@
 	(wire
 		(pts
-			(xy 135.89 121.92) (xy 127 121.92)
+			(xy 143.51 121.92) (xy 134.62 121.92)
 		)
 		(stroke
@@
 	(wire
 		(pts
+			(xy 134.62 134.62) (xy 143.51 134.62)
+		)
+		(stroke
+			(width 0)
+			(type default)
+		)
+	)
+	(wire
+		(pts
 			(xy 312.42 139.7) (xy 332.74 139.7)
 		)
@@
 	(wire
 		(pts
-			(xy 135.89 121.92) (xy 135.89 124.46)
+			(xy 143.51 121.92) (xy 143.51 124.46)
 		)
 		(stroke
@@
 	(wire
 		(pts
+			(xy 127 121.92) (xy 127 124.46)
+		)
+		(stroke
+			(width 0)
+			(type default)
+		)
+	)
+	(wire
+		(pts
 			(xy 124.46 176.53) (xy 124.46 175.26)
 		)
@@
 	(wire
 		(pts
+			(xy 127 121.92) (xy 110.49 121.92)
+		)
+		(stroke
+			(width 0)
+			(type default)
+		)
+	)
+	(wire
+		(pts
 			(xy 55.88 154.94) (xy 85.09 154.94)
 		)
@@
 	(wire
 		(pts
-			(xy 135.89 134.62) (xy 127 134.62)
-		)
-		(stroke
-			(width 0)
-			(type default)
-		)
-	)
-	(wire
-		(pts
 			(xy 297.18 88.9) (xy 288.29 88.9)
 		)
@@
 	(wire
 		(pts
-			(xy 127 121.92) (xy 127 124.46)
+			(xy 134.62 121.92) (xy 134.62 124.46)
 		)
 		(stroke
@@
 	(wire
 		(pts
+			(xy 127 132.08) (xy 127 134.62)
+		)
+		(stroke
+			(width 0)
+			(type default)
+		)
+	)
+	(wire
+		(pts
 			(xy 261.62 88.9) (xy 270.51 88.9)
 		)
@@
 	(wire
 		(pts
-			(xy 127 132.08) (xy 127 134.62)
+			(xy 134.62 132.08) (xy 134.62 134.62)
 		)
 		(stroke
@@
 	(wire
 		(pts
-			(xy 135.89 137.16) (xy 135.89 134.62)
+			(xy 143.51 137.16) (xy 143.51 134.62)
 		)
 		(stroke
@@
 	(symbol
 		(lib_id "Device:C")
-		(at 135.89 128.27 0)
+		(at 143.51 128.27 0)
 		(unit 1)
 		(body_style 1)
@@
 		(dnp no)
 		(property "Reference" "C70"
-			(at 136.906 125.222 0)
+			(at 144.526 125.222 0)
 			(show_name no)
 			(do_not_autoplace no)
@@
 		)
 		(property "Value" "4u7"
-			(at 136.906 131.318 0)
+			(at 144.526 131.318 0)
 			(show_name no)
 			(do_not_autoplace no)
@@
 		)
 		(property "Footprint" "Capacitor_SMD:C_0603_1608Metric"
-			(at 136.8552 132.08 0)
+			(at 144.4752 132.08 0)
 			(hide yes)
 			(show_name no)
@@
 		)
 		(property "Datasheet" ""
-			(at 135.89 128.27 0)
+			(at 143.51 128.27 0)
 			(hide yes)
 			(show_name no)
@@
 		)
 		(property "Description" "Unpolarized capacitor"
-			(at 135.89 128.27 0)
+			(at 143.51 128.27 0)
 			(hide yes)
 			(show_name no)
@@
 	)
 	(symbol
+		(lib_id "Device:C")
+		(at 127 128.27 0)
+		(unit 1)
+		(body_style 1)
+		(exclude_from_sim no)
+		(in_bom yes)
+		(on_board yes)
+		(in_pos_files yes)
+		(dnp no)
+		(property "Reference" "C112"
+			(at 128.016 125.222 0)
+			(show_name no)
+			(do_not_autoplace no)
+			(effects
+				(font
+					(size 1.27 1.27)
+				)
+				(justify left)
+			)
+		)
+		(property "Value" "470n"
+			(at 128.016 131.318 0)
+			(show_name no)
+			(do_not_autoplace no)
+			(effects
+				(font
+					(size 1.27 1.27)
+				)
+				(justify left)
+			)
+		)
+		(property "Footprint" "Capacitor_SMD:C_0201_0603Metric"
+			(at 127.9652 132.08 0)
+			(hide yes)
+			(show_name no)
+			(do_not_autoplace no)
+			(effects
+				(font
+					(size 1.27 1.27)
+				)
+			)
+		)
+		(property "Datasheet" ""
+			(at 127 128.27 0)
+			(hide yes)
+			(show_name no)
+			(do_not_autoplace no)
+			(effects
+				(font
+					(size 1.27 1.27)
+				)
+			)
+		)
+		(property "Description" "Unpolarized capacitor"
+			(at 127 128.27 0)
+			(hide yes)
+			(show_name no)
+			(do_not_autoplace no)
+			(effects
+				(font
+					(size 1.27 1.27)
+				)
+			)
+		)
+		(pin "2"
+		)
+		(pin "1"
+		)
+		(instances
+			(project "PCB"
+				(path "/ed0095eb-57a0-4856-9ac4-7b40bd214a3a/82e75441-9b85-4304-afce-254bf3f07a53"
+					(reference "C112")
+					(unit 1)
+				)
+			)
+		)
+	)
+	(symbol
 		(lib_id "power:+3V3")
 		(at 201.93 100.33 0)
@@
 	(symbol
 		(lib_id "power:+3V3")
-		(at 135.89 119.38 0)
+		(at 143.51 119.38 0)
 		(unit 1)
 		(body_style 1)
@@
 		(fields_autoplaced yes)
 		(property "Reference" "#PWR068"
-			(at 135.89 123.19 0)
+			(at 143.51 123.19 0)
 			(hide yes)
 			(show_name no)
@@
 		)
 		(property "Value" "+3V3"
-			(at 135.89 114.3 0)
+			(at 143.51 114.3 0)
 			(show_name no)
 			(do_not_autoplace no)
@@
 		)
 		(property "Footprint" ""
-			(at 135.89 119.38 0)
+			(at 143.51 119.38 0)
 			(hide yes)
 			(show_name no)
@@
 		)
 		(property "Datasheet" ""
-			(at 135.89 119.38 0)
+			(at 143.51 119.38 0)
 			(hide yes)
 			(show_name no)
@@
 		)
 		(property "Description" "Power symbol creates a global label with name \"+3V3\""
-			(at 135.89 119.38 0)
+			(at 143.51 119.38 0)
 			(hide yes)
 			(show_name no)
@@
 	(symbol
 		(lib_id "Device:C")
-		(at 127 128.27 0)
+		(at 134.62 128.27 0)
 		(unit 1)
 		(body_style 1)
@@
 		(dnp no)
 		(property "Reference" "C71"
-			(at 128.016 125.222 0)
+			(at 135.636 125.222 0)
 			(show_name no)
 			(do_not_autoplace no)
@@
 		)
 		(property "Value" "470n"
-			(at 128.016 131.318 0)
+			(at 135.636 131.318 0)
 			(show_name no)
 			(do_not_autoplace no)
@@
 		)
 		(property "Footprint" "Capacitor_SMD:C_0201_0603Metric"
-			(at 127.9652 132.08 0)
+			(at 135.5852 132.08 0)
 			(hide yes)
 			(show_name no)
@@
 		)
 		(property "Datasheet" ""
-			(at 127 128.27 0)
+			(at 134.62 128.27 0)
 			(hide yes)
 			(show_name no)
@@
 		)
 		(property "Description" "Unpolarized capacitor"
-			(at 127 128.27 0)
+			(at 134.62 128.27 0)
 			(hide yes)
 			(show_name no)
@@
 	(symbol
 		(lib_id "power:GND")
-		(at 135.89 137.16 0)
+		(at 143.51 137.16 0)
 		(unit 1)
 		(body_style 1)
@@
 		(dnp no)
 		(property "Reference" "#PWR071"
-			(at 135.89 143.51 0)
+			(at 143.51 143.51 0)
 			(hide yes)
 			(show_name no)
@@
 		)
 		(property "Value" "GND"
-			(at 135.89 142.24 0)
+			(at 143.51 142.24 0)
 			(show_name no)
 			(do_not_autoplace no)
@@
 		)
 		(property "Footprint" ""
-			(at 135.89 137.16 0)
+			(at 143.51 137.16 0)
 			(hide yes)
 			(show_name no)
@@
 		)
 		(property "Datasheet" ""
-			(at 135.89 137.16 0)
+			(at 143.51 137.16 0)
 			(hide yes)
 			(show_name no)
@@
 		)
 		(property "Description" "Power symbol creates a global label with name \"GND\" , ground"
-			(at 135.89 137.16 0)
+			(at 143.51 137.16 0)
 			(hide yes)
 			(show_name no)

Commit message: finished fills and a bit of routing for the buck
Parts:
- U2: footprint easyeda2kicad:QFN-28_L5.0-W5.0-P0.50-TL-EP3.2 -> Package_DFN_QFN:QFN-28-1EP_5x5mm_P0.5mm_EP3.25x3.25mm_ThermalVias
Changed lines of the file:
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@@
 			)
 		)
-		(property "Footprint" "easyeda2kicad:QFN-28_L5.0-W5.0-P0.50-TL-EP3.2"
+		(property "Footprint" "Package_DFN_QFN:QFN-28-1EP_5x5mm_P0.5mm_EP3.25x3.25mm_ThermalVias"
 			(at 259.08 210.312 0)
 			(hide yes)

Commit message: new power rail YAY
Parts:
- added C147, C173: 4u7, Capacitor_SMD:C_0603_1608Metric, symbol Device:C
- added L5: 1u5, Inductor_SMD:L_Sunlord_SWPA4030S, symbol Device:L
- added U8: TPS61240DRVR, Package_SON:WSON-6-1EP_2x2mm_P0.65mm_EP1x1.6mm, symbol FPGA Accelerator:TPS61240DRVR
Connections:
- net +3V3: now also C147.1, L5.1, U8.4 (EN), U8.6 (VI)
- net GND: now also C147.2, C173.2, U8.1 (GND)
- new net: L5.2, U8.5 (SW)
- new net +5V: C173.1, U8.2 (VOUT), U8.3 (FB)
Other:
- note added: "A small 5V boost converter for HDMI and other future peripherals!"
- moved on the sheet: C112, C41, C42, C43, C44, C45, C46, C48, C49, C50, C51, C52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

Commit message: going more insane with HDMI routing
Connections:
- net GND: now also U8.7 (GND)

Commit message: working on DRC errors!
Parts:
- U5: footprint Package_DFN_QFN:Texas_VQFN-HR-12_2x2.5mm_P0.5mm_ThermalVias -> FPGA:Texas_VQFN-HR-12_2x2.5mm_P0.5mm_ThermalVias
Changed lines of the file:
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@@
 			)
 		)
-		(property "Footprint" "Package_DFN_QFN:Texas_VQFN-HR-12_2x2.5mm_P0.5mm_ThermalVias"
+		(property "Footprint" "FPGA:Texas_VQFN-HR-12_2x2.5mm_P0.5mm_ThermalVias"
 			(at 97.79 87.63 0)
 			(hide yes)
