File: PCB/configurations.kicad_sch (KiCad schematic)
At the start: 26 parts, among them J2 Conn_ARM_SWD_TagConnect_TC2030, J3 USB_C_Receptacle_USB2.0_16P, U1 XC7A50T-FGG484, U3 FT2232HQ, U4 M93C56-WMN6TP, Y1 12MHz

Commit message: cleaned up the schematic, wired some config pins
Parts:
- added R29: 1k, symbol Device:R
Connections:
- net +3V3: now also R29.1
- net TCK: now also J2.4 (SWCLK), R19.2; no longer R16.2, R22.2, U1.V12 (TCK_0)
- net TDI: now also J2.3 (~{RESET}), R18.2; no longer R19.2, U1.R13 (TDI_0)
- net TDO: now also J2.6 (SWO), R17.2; no longer R18.2, U1.U13 (TDO_0)
- net TMS: now also J2.2 (SWDIO), R16.2; no longer R17.2, R23.2, U1.T13 (TMS_0)
- net at R17.1: now also U1.U13 (TDO_0); no longer J2.2 (SWDIO)
- net at U3.14 (~{RESET}): now also R29.2
- net at R18.1: now also U1.R13 (TDI_0); no longer J2.6 (SWO)
- net at R16.1: now also R22.2, U1.T13 (TMS_0); no longer J2.4 (SWCLK)
- net at R19.1: now also R23.2, U1.V12 (TCK_0); no longer J2.3 (~{RESET})
Other:
- note added: "Damping resistors as close as possible to both JTAG inputs"
- moved on the sheet: R14, R15, R19, R2, R22, R23, R3

Commit message: fixed JTAGG, working on power architecture
Parts:
- added R30, R31: 10k, symbol Device:R
Connections:
- net +3V3: now also R30.1, R31.1
- net at R16.1, U1.T13 (TMS_0): now also R23.2; no longer R22.2
- net at R17.1, U1.U13 (TDO_0): now also R30.2
- net at R18.1, U1.R13 (TDI_0): now also R31.2
- net at R19.1, U1.V12 (TCK_0): now also R22.2; no longer R23.2
Other:
- moved on the sheet: R14, R15, R16, R17, R18, R19, R2, R23, R3

Commit message: finished wiring USB buck
Parts:
- added C60: 47u, symbol Device:C
- added C61: 4u7, symbol Device:C
- added C62: 470n, symbol Device:C
- added C63: 10u, symbol Device:C
- added C64: 470nF, symbol Device:C
- added C9: 47n, symbol Device:C
- added L5: 1.5u, symbol Device:L
- added R32: 100k, symbol Device:R
- added U6: TPS62132, Package_DFN_QFN:VQFN-16-1EP_3x3mm_P0.5mm_EP1.68x1.68mm_ThermalVias, symbol Regulator_Switching:TPS62132
Connections:
- net GND: now also C60.2, C61.2, C62.2, C63.2, C64.2, C9.2, U6.15 (GND), U6.16 (GND), U6.17 (GND), U6.5 (FB), U6.6 (GND), U6.7 (FSW), U6.8 (DEF)
- net +VBUS: now reaches J3.A4 (VBUS), J3.A9 (VBUS), J3.B4 (VBUS), J3.B9 (VBUS)
- net +VBUS: now also C63.1, C64.1, U6.10 (VIN), U6.11 (VIN), U6.12 (VIN), U6.13 (EN)
- new net: L5.1, U6.1 (SW), U6.2 (SW), U6.3 (SW)
- new net: R32.2, U6.4 (PG)
- new net: C9.1, U6.9 (SS/TR)
- new net +VBUS_3V3: C60.1, C61.1, C62.1, L5.2, R32.1, U6.14 (VOS)
Other:
- note added: "1.5uH & 47uF for BOM optimization"
- note added: "23.5ms start up, reduce inrush >"
- moved on the sheet: C57, C58, C59, J2, J3, R20, R21, R24, R25, R26, R27, R28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

Commit message: cleaning up the schematic
Parts:
- C64: value 470nF -> 470n
Other:
- moved on the sheet: C57, C58, C59, C60, C61, C62, C63, C64, C9, J2, L5, R24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

Commit message: working on the power MXU
Parts:
- removed C9: 47n, symbol Device:C
- added C65: 47n, symbol Device:C
Connections:
- net GND: now also C65.2
- net at U6.9 (SS/TR): now also C65.1
Changed lines of the file:
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@@
 	)
 	(symbol
+		(lib_id "Device:C")
+		(at 107.95 54.61 0)
+		(unit 1)
+		(exclude_from_sim no)
+		(in_bom yes)
+		(on_board yes)
+		(dnp no)
+		(fields_autoplaced yes)
+		(property "Reference" "C65"
+			(at 111.76 53.3399 0)
+			(effects
+				(font
+					(size 1.27 1.27)
+				)
+				(justify left)
+			)
+		)
+		(property "Value" "47n"
+			(at 111.76 55.8799 0)
+			(effects
+				(font
+					(size 1.27 1.27)
+				)
+				(justify left)
+			)
+		)
+		(property "Footprint" ""
+			(at 108.9152 58.42 0)
+			(effects
+				(font
+					(size 1.27 1.27)
+				)
+				(hide yes)
+			)
+		)
+		(property "Datasheet" "~"
+			(at 107.95 54.61 0)
+			(effects
+				(font
+					(size 1.27 1.27)
+				)
+				(hide yes)
+			)
+		)
+		(property "Description" "Unpolarized capacitor"
+			(at 107.95 54.61 0)
+			(effects
+				(font
+					(size 1.27 1.27)
+				)
+				(hide yes)
+			)
+		)
+		(pin "2"
+		)
+		(pin "1"
+		)
+		(instances
+			(project ""
+				(path "/ed0095eb-57a0-4856-9ac4-7b40bd214a3a/eed1a5c9-5dce-4964-b7ee-57ee65be1a9d"
+					(reference "C65")
+					(unit 1)
+				)
+			)
+		)
+	)
+	(symbol
 		(lib_id "power:GND")
 		(at 140.97 57.15 0)
@@
 					(unit 1)
 				)
-			)
-		)
-	)
-	(symbol
-		(lib_id "Device:C")
-		(at 107.95 54.61 0)
-		(unit 1)
-		(exclude_from_sim no)
-		(in_bom yes)
-		(on_board yes)
-		(dnp no)
-		(fields_autoplaced yes)
-		(property "Reference" "C9"
-			(at 111.76 53.3399 0)
-			(effects
-				(font
-					(size 1.27 1.27)
-				)
-				(justify left)
-			)
-		)
-		(property "Value" "47n"
-			(at 111.76 55.8799 0)
-			(effects
-				(font
-					(size 1.27 1.27)
-				)
-				(justify left)
-			)
-		)
-		(property "Footprint" ""
-			(at 108.9152 58.42 0)
-			(effects
-				(font
-					(size 1.27 1.27)
-				)
-				(hide yes)
-			)
-		)
-		(property "Datasheet" "~"
-			(at 107.95 54.61 0)
-			(effects
-				(font
-					(size 1.27 1.27)
-				)
-				(hide yes)
-			)
-		)
-		(property "Description" "Unpolarized capacitor"
-			(at 107.95 54.61 0)
-			(effects
-				(font
-					(size 1.27 1.27)
-				)
-				(hide yes)
-			)
-		)
-		(pin "1"
-		)
-		(pin "2"
-		)
-		(instances
-			(project ""
-				(path "/ed0095eb-57a0-4856-9ac4-7b40bd214a3a/eed1a5c9-5dce-4964-b7ee-57ee65be1a9d"
-					(reference "C9")
-					(unit 1)
-				)

Commit message: working on finishing the ft2232H wiring
Connections:
- net +3V3: now also U3.20 (VCCIO), U3.31 (VCCIO), U3.4 (VPHY), U3.42 (VCCIO), U3.50 (VREGIN), U3.56 (VCCIO), U3.9 (VPLL)
- net +1V8_VREGOUT: now reaches U3.12 (VCORE)
- net +1V8_VREGOUT: now also U3.37 (VCORE), U3.49 (VREGOUT), U3.64 (VCORE)
Other:
- note added: "3.3uF ON THIS LINE"
- note added: "Internal 1V8 LDO, different from global 1V8 to isolate the rail for the component! >"
- note added: "LCFilter?, Pg.10 >"

Commit message: decoupled all the rails
Parts:
- added C73, C74, C76, C77, C78, C79, C80, C81, C82, C83, C84: 470n, symbol Device:C
- added C75, C85: 4u7, symbol Device:C
Connections:
- net +3V3: now also C74.1, C77.1, C78.1, C79.1, C80.1, C81.1, C82.1, C83.1, C84.1, C85.1
- net GND: now also C73.2, C74.2, C75.2, C76.2, C77.2, C78.2, C79.2, C80.2, C81.2, C82.2, C83.2, C84.2, C85.2
- net +1V8_VREGOUT: no longer names the net of U3.12 (VCORE), U3.37 (VCORE), U3.49 (VREGOUT), U3.64 (VCORE)
- net +1V8_VREGOUT: now also C73.1, C75.1, C76.1
Other:
- note added: "VCORE"
- note removed: "3.3uF ON THIS LINE"
- note removed: "Internal 1V8 LDO, different from global 1V8 to isolate the rail for the component! >"
- moved on the sheet: C57, C58, C59, R24, R25, R26, R27, R28, R29, U3, U4, Y1

Commit message: more decoupling, cleaning stuff up
Parts:
- added C86: 470n, symbol Device:C
- C73: Purpose (none) -> VCORE
Connections:
- net GND: now also C86.2
- net at C73.1, C75.1, C76.1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: now also C86.1
Other:
- note added: "^ VCORE ^"
- note removed: "VCORE"
- moved on the sheet: C74, C75, C76, C85
