File: PCB/configurations.kicad_sch (KiCad schematic)
At the start: 6 parts, among them U1 XC7A50T-FGG484, U7 MT25QL128ABA1EW7-0SIT

Commit message: added the SPI net labels!
Connections:
- net QSPI_CLK: now reaches U1.L12 (CCLK_0)
Changed lines of the file:
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@@
+	(wire
+		(pts
+			(xy 218.44 133.35) (xy 207.01 133.35)
+		)
+		(stroke
+			(width 0)
+			(type default)
+		)
+	)
 	(wire
 		(pts
@@
 		)
 	)
+	(label "QSPI_CLK"
+		(at 218.44 133.35 180)
+		(effects
+			(font
+				(size 1.27 1.27)
+			)
+			(justify right bottom)
+		)
+	)

Commit message: some footprints added in, starting to work on flash
Parts:
- U1: footprint (none) -> Package_BGA:Xilinx_FGG484
- U7: LCSC (none) -> C2887898; MPN (none) -> MT25QL128ABA1EW7-0SIT
Changed lines of the file:
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@@
 		(dnp no)
 		(fields_autoplaced yes)
-		(property "Reference" "#PWR?"
+		(property "Reference" "#PWR0122"
 			(at 196.85 100.33 0)
 			(effects
@@
 			(project "PCB"
 				(path "/ed0095eb-57a0-4856-9ac4-7b40bd214a3a/eed1a5c9-5dce-4964-b7ee-57ee65be1a9d"
-					(reference "#PWR?")
+					(reference "#PWR0122")
 					(unit 1)
 				)
@@
 		(dnp no)
 		(fields_autoplaced yes)
-		(property "Reference" "#PWR?"
+		(property "Reference" "#PWR0124"
 			(at 243.84 157.48 0)
 			(effects
@@
 			(project "PCB"
 				(path "/ed0095eb-57a0-4856-9ac4-7b40bd214a3a/eed1a5c9-5dce-4964-b7ee-57ee65be1a9d"
-					(reference "#PWR?")
+					(reference "#PWR0124")
 					(unit 1)
 				)
@@
 			)
 		)
-		(property "Footprint" ""
+		(property "Footprint" "Package_BGA:Xilinx_FGG484"
 			(at 168.91 140.97 0)
 			(effects
@@
 			)
 		)
+		(property "MPN" "MT25QL128ABA1EW7-0SIT"
+			(at 342.9 143.51 0)
+			(effects
+				(font
+					(size 1.27 1.27)
+				)
+				(hide yes)
+			)
+		)
+		(property "LCSC" "C2887898"
+			(at 342.9 143.51 0)
+			(effects
+				(font
+					(size 1.27 1.27)
+				)
+				(hide yes)
+			)
+		)
 		(pin "3"
 		)
@@
 		(dnp no)
 		(fields_autoplaced yes)
-		(property "Reference" "#PWR?"
+		(property "Reference" "#PWR0123"
 			(at 234.95 129.54 0)
 			(effects
@@
 			(project "PCB"
 				(path "/ed0095eb-57a0-4856-9ac4-7b40bd214a3a/eed1a5c9-5dce-4964-b7ee-57ee65be1a9d"
-					(reference "#PWR?")
+					(reference "#PWR0123")
 					(unit 1)
 				)

Commit message: wiring QSPI
Parts:
- added C111: 100n, symbol Device:C
- added C112: 1u, symbol Device:C
- added R19, R20, R21: 10k, symbol Device:R
Connections:
- net +3V3: now also U7.8 (VCC), C111.1, C112.1, R19.1, R20.1, R21.1
- net GND: now also U7.4 (VSS), U7.9 (PAD), C111.2, C112.2
- net QSPI_CLK: now also U7.6 (C)
- net QSPI_CS: now reaches U7.1 (~{S})
- net QSPI_CS: now also R19.2
- net QSPI_DQ1: now reaches U7.2 (DQ1)
- net QSPI_DQ2: now reaches U7.3 (~{W}/DQ2)
- net QSPI_DQ2: now also R20.2
- net QSPI_DQ0: now reaches U7.5 (DQ0)
- net QSPI_DQ3: now reaches U7.7 (~{RESET}/DQ3)
- net QSPI_DQ3: now also R21.2
Other:
- moved on the sheet: R14, R15, R2, R3, U1F, U7

Commit message: hopping off for the night
Other:
- note added: "DOUBLE CHECK THIS, DONE ON LOW SLEEP"
Changed lines of the file:
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@@
+		)
+	)
+	(text "DOUBLE CHECK THIS, DONE ON LOW SLEEP"
+		(exclude_from_sim no)
+		(at 298.704 191.77 0)
+		(effects
+			(font
+				(size 1.27 1.27)
+			)
 		)
 	)
@@
 		(effects
 			(font
-				(size 1.27 1.27)
-			)
-			(justify left bottom)
-		)
-	)
-	(label "< Decoupling"
-		(at 140.97 104.14 0)
-		(effects
-			(font

Commit message: wiring some configuration pins, cleaning up the schematic
Parts:
- added R22, R23: 4.7k, symbol Device:R
- added TP1: DONE_STAT, symbol Connector:TestPoint
Connections:
- net +3V3: now also R22.2, R23.2
- net DONE: now reaches U1.G11 (DONE_0)
- net DONE: now also TP1.1
- net at U1.N12 (PROGRAM_B_0): now also R22.1
- net at U1.U12 (INIT_B_0): now also R23.1
Other:
- note removed: "DOUBLE CHECK THIS, DONE ON LOW SLEEP"

Commit message: finished the configurations
Connections:
- net +3V3: now also U1.U8 (CFGBVS_0)
- net GND: now also U1.L10 (VP_0), U1.L9 (VREFN_0), U1.M10 (VREFP_0), U1.M9 (VN_0), U1.N10 (DXP_0), U1.N9 (DXN_0)
Other:
- note added: "< No temp sense, no internals, tying low (UG475)"
- note added: "Bank 13/14 need to be 3V3 because of CFGBVS"
Changed lines of the file:
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@@
+		)
+	)
+	(text "Bank 13/14 need to be 3V3 because of CFGBVS"
+		(exclude_from_sim no)
+		(at 103.886 105.41 0)
+		(effects
+			(font
+				(size 1.27 1.27)
+			)
 		)
 	)
@@
 		)
 	)
+	(text "< No temp sense, no internals, tying low (UG475)"
+		(exclude_from_sim no)
+		(at 174.752 173.482 0)
+		(effects
+			(font
+				(size 1.27 1.27)
+			)
+		)
+	)
 	(junction
 		(at 300.99 154.94)
@@
 	)
 	(junction
+		(at 166.37 153.67)
+		(diameter 0)
+		(color 0 0 0 0)
+	)
+	(junction
 		(at 309.88 157.48)
+		(diameter 0)
+		(color 0 0 0 0)
+	)
+	(junction
+		(at 146.05 179.07)
 		(diameter 0)
 		(color 0 0 0 0)
@@
 	)
 	(junction
+		(at 146.05 171.45)
+		(diameter 0)
+		(color 0 0 0 0)
+	)
+	(junction
 		(at 292.1 127)
 		(diameter 0)
@@
 	)
 	(junction
+		(at 146.05 166.37)
+		(diameter 0)
+		(color 0 0 0 0)
+	)
+	(junction
+		(at 146.05 173.99)
+		(diameter 0)
+		(color 0 0 0 0)
+	)
+	(junction
 		(at 339.09 133.35)
 		(diameter 0)
@@
 	)
 	(junction
+		(at 146.05 181.61)
+		(diameter 0)
+		(color 0 0 0 0)
+	)
+	(junction
 		(at 323.85 120.65)
 		(diameter 0)
@@
 	(wire
 		(pts
+			(xy 146.05 173.99) (xy 146.05 179.07)
+		)
+		(stroke
+			(width 0)
+			(type default)
+		)
+	)
+	(wire
+		(pts
 			(xy 309.88 157.48) (xy 313.69 157.48)
 		)
@@
 	(wire
 		(pts
+			(xy 146.05 166.37) (xy 146.05 171.45)
+		)
+		(stroke
+			(width 0)
+			(type default)
+		)
+	)
+	(wire
+		(pts
 			(xy 181.61 137.16) (xy 181.61 143.51)
 		)
@@
 	(wire
 		(pts
+			(xy 166.37 158.75) (xy 166.37 153.67)
+		)
+		(stroke
+			(width 0)
+			(type default)
+		)
+	)
+	(wire
+		(pts
 			(xy 323.85 120.65) (xy 327.66 120.65)
 		)
@@
 	(wire
 		(pts
+			(xy 146.05 171.45) (xy 146.05 173.99)
+		)
+		(stroke
+			(width 0)
+			(type default)
+		)
+	)
+	(wire
+		(pts
 			(xy 172.72 128.27) (xy 172.72 129.54)
 		)
@@
 	(wire
 		(pts
+			(xy 144.78 171.45) (xy 146.05 171.45)
+		)
+		(stroke
+			(width 0)
+			(type default)
+		)
+	)
+	(wire
+		(pts
 			(xy 158.75 151.13) (xy 166.37 151.13)
 		)
@@
 	(wire
 		(pts
+			(xy 146.05 163.83) (xy 146.05 166.37)
+		)
+		(stroke
+			(width 0)
+			(type default)
+		)
+	)
+	(wire
+		(pts
 			(xy 339.09 120.65) (xy 339.09 133.35)
 		)
@@
 	(wire
 		(pts
+			(xy 144.78 166.37) (xy 146.05 166.37)
+		)
+		(stroke
+			(width 0)
+			(type default)
+		)
+	)
+	(wire
+		(pts
 			(xy 292.1 135.89) (xy 292.1 144.78)
 		)
@@
 	(wire
 		(pts
+			(xy 144.78 173.99) (xy 146.05 173.99)
+		)
+		(stroke
+			(width 0)
+			(type default)
+		)
+	)
+	(wire
+		(pts
 			(xy 292.1 127) (xy 300.99 127)
 		)
@@
 		)
 	)
+	(wire
+		(pts
+			(xy 144.78 163.83) (xy 146.05 163.83)
+		)
+		(stroke
+			(width 0)
+			(type default)
+		)
+	)
 	(bus
 		(pts
@@
 	(wire
 		(pts
+			(xy 146.05 181.61) (xy 144.78 181.61)
+		)
+		(stroke
+			(width 0)
+			(type default)
+		)
+	)
+	(wire
+		(pts
 			(xy 190.5 144.78) (xy 190.5 140.97)
 		)
@@
 		)
 	)
+	(wire
+		(pts
+			(xy 146.05 189.23) (xy 146.05 181.61)
+		)
+		(stroke
+			(width 0)
+			(type default)
+		)
+	)
 	(bus
 		(pts
@@
 		)
 	)
+	(wire
+		(pts
+			(xy 144.78 158.75) (xy 166.37 158.75)
+		)
+		(stroke
+			(width 0)
+			(type default)
+		)
+	)
+	(wire
+		(pts
+			(xy 146.05 181.61) (xy 146.05 179.07)
+		)
+		(stroke
+			(width 0)
+			(type default)
+		)
+	)
 	(bus
 		(pts
@@
 		(pts
 			(xy 144.78 123.19) (xy 160.02 123.19)
+		)
+		(stroke
+			(width 0)
+			(type default)
+		)
+	)
+	(wire
+		(pts
+			(xy 146.05 179.07) (xy 144.78 179.07)
 		)
 		(stroke
@@
 					(unit 1)
 				)
+			)
+		)
+	)
+	(symbol
+		(lib_id "power:GND")
+		(at 146.05 189.23 0)
+		(unit 1)
+		(exclude_from_sim no)
+		(in_bom yes)
+		(on_board yes)
+		(dnp no)
+		(fields_autoplaced yes)
+		(property "Reference" "#PWR056"
+			(at 146.05 195.58 0)
+			(effects
+				(font
+					(size 1.27 1.27)
+				)
+				(hide yes)
+			)
+		)
+		(property "Value" "GND"
+			(at 146.05 194.31 0)
+			(effects
+				(font
+					(size 1.27 1.27)
+				)
+			)
+		)
+		(property "Footprint" ""
+			(at 146.05 189.23 0)
+			(effects
+				(font
+					(size 1.27 1.27)
+				)
+				(hide yes)
+			)
+		)
+		(property "Datasheet" ""
+			(at 146.05 189.23 0)
+			(effects
+				(font
+					(size 1.27 1.27)
+				)
+				(hide yes)
+			)
+		)
+		(property "Description" "Power symbol creates a global label with name \"GND\" , ground"
+			(at 146.05 189.23 0)
+			(effects
+				(font
+					(size 1.27 1.27)
+				)
+				(hide yes)
+			)
+		)
+		(pin "1"
+		)
+		(instances
+			(project ""
+				(path "/ed0095eb-57a0-4856-9ac4-7b40bd214a3a/eed1a5c9-5dce-4964-b7ee-57ee65be1a9d"
+					(reference "#PWR056")
+					(unit 1)
+				)

Commit message: an LED + changing the decoupling on the m.2 edge connector
Parts:
- removed TP1: DONE_STAT, symbol Connector:TestPoint
- added D1: LED, symbol Device:LED
- added R24: 1k, symbol Device:R
Connections:
- net +3V3: now also D1.2 (A)
- net DONE: now also R24.1
- new net: D1.1 (K), R24.2
Other:
- note added: "DONE sinks current! >"
Changed lines of the file:
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@@
 		)
 	)
+	(text "DONE sinks current! >"
+		(exclude_from_sim no)
+		(at 86.614 87.884 0)
+		(effects
+			(font
+				(size 1.27 1.27)
+			)
+		)
+	)
 	(junction
 		(at 300.99 154.94)
@@
 	(wire
 		(pts
-			(xy 144.78 148.59) (xy 153.67 148.59)
+			(xy 144.78 148.59) (xy 156.21 148.59)
 		)
 		(stroke
@@
 	(wire
 		(pts
+			(xy 128.27 87.63) (xy 125.73 87.63)
+		)
+		(stroke
+			(width 0)
+			(type default)
+		)
+	)
+	(wire
+		(pts
 			(xy 323.85 120.65) (xy 327.66 120.65)
 		)
@@
 	(wire
 		(pts
+			(xy 100.33 87.63) (xy 107.95 87.63)
+		)
+		(stroke
+			(width 0)
+			(type default)
+		)
+	)
+	(wire
+		(pts
 			(xy 309.88 127) (xy 309.88 128.27)
 		)
@@
 	(wire
 		(pts
+			(xy 118.11 87.63) (xy 115.57 87.63)
+		)
+		(stroke
+			(width 0)
+			(type default)
+		)
+	)
+	(wire
+		(pts
 			(xy 146.05 181.61) (xy 146.05 179.07)
 		)
@@
 	)
 	(label "DONE"
-		(at 147.32 148.59 0)
+		(at 156.21 148.59 180)
 		(effects
 			(font
 				(size 1.27 1.27)
 			)
-			(justify left bottom)
+			(justify right bottom)
 		)
 	)
@@
 		)
 	)
+	(label "DONE"
+		(at 100.33 87.63 0)
+		(effects
+			(font
+				(size 1.27 1.27)
+			)
+			(justify left bottom)
+		)
+	)
 	(label "QSPI_CLK"
 		(at 156.21 135.89 180)
@@
 	)
 	(symbol
-		(lib_id "Connector:TestPoint")
-		(at 153.67 148.59 270)
-		(unit 1)
-		(exclude_from_sim no)
-		(in_bom yes)
-		(on_board yes)
-		(dnp no)
-		(property "Reference" "TP1"
-			(at 155.448 146.812 90)
-			(effects
-				(font
-					(size 1.016 1.016)
-				)
-				(justify left)
-			)
-		)
-		(property "Value" "DONE_STAT"
-			(at 154.94 150.876 0)
-			(effects
-				(font
-					(size 1.016 1.016)
-				)
-				(justify left)
-				(hide yes)
-			)
-		)
-		(property "Footprint" ""
-			(at 153.67 153.67 0)
-			(effects
-				(font
-					(size 1.27 1.27)
-				)
-				(hide yes)
-			)
-		)
-		(property "Datasheet" "~"
-			(at 153.67 153.67 0)
-			(effects
-				(font
-					(size 1.27 1.27)
-				)
-				(hide yes)
-			)
-		)
-		(property "Description" "test point"
-			(at 153.67 148.59 0)
-			(effects
-				(font
-					(size 1.27 1.27)
-				)
-				(hide yes)
-			)
-		)
-		(pin "1"
-		)
-		(instances
-			(project "PCB"
-				(path "/ed0095eb-57a0-4856-9ac4-7b40bd214a3a/eed1a5c9-5dce-4964-b7ee-57ee65be1a9d"
-					(reference "TP1")
-					(unit 1)
-				)
-			)
-		)
-	)
-	(symbol
 		(lib_id "power:+3V3")
 		(at 292.1 124.46 0)
@@
 					(unit 1)
 				)
+			)
+		)
+	)
+	(symbol
+		(lib_id "Device:R")
+		(at 111.76 87.63 90)
+		(unit 1)
+		(exclude_from_sim no)
+		(in_bom yes)
+		(on_board yes)
+		(dnp no)
+		(fields_autoplaced yes)
+		(property "Reference" "R24"
+			(at 111.76 81.28 90)
+			(effects
+				(font
+					(size 1.27 1.27)
+				)
+			)
+		)
+		(property "Value" "1k"
+			(at 111.76 83.82 90)
+			(effects
+				(font
+					(size 1.27 1.27)
+				)
+			)
+		)
+		(property "Footprint" ""
+			(at 111.76 89.408 90)
+			(effects
+				(font
+					(size 1.27 1.27)
+				)
+				(hide yes)
+			)
+		)
+		(property "Datasheet" "~"
+			(at 111.76 87.63 0)
+			(effects
+				(font
+					(size 1.27 1.27)
+				)
+				(hide yes)
+			)
+		)
+		(property "Description" "Resistor"
+			(at 111.76 87.63 0)
+			(effects
+				(font
+					(size 1.27 1.27)
+				)
+				(hide yes)
+			)
+		)
+		(pin "1"
+		)
+		(pin "2"
+		)
+		(instances
+			(project ""
+				(path "/ed0095eb-57a0-4856-9ac4-7b40bd214a3a/eed1a5c9-5dce-4964-b7ee-57ee65be1a9d"
+					(reference "R24")
+					(unit 1)
+				)
+			)
+		)
+	)
+	(symbol
+		(lib_id "Device:LED")
+		(at 121.92 87.63 0)
+		(unit 1)
+		(exclude_from_sim no)
+		(in_bom yes)
+		(on_board yes)
+		(dnp no)
+		(fields_autoplaced yes)
+		(property "Reference" "D1"
+			(at 120.3325 81.28 0)
+			(effects
+				(font
+					(size 1.27 1.27)
+				)
+			)
+		)
+		(property "Value" "LED"
+			(at 120.3325 83.82 0)
+			(effects
+				(font
+					(size 1.27 1.27)
+				)
+			)
+		)
+		(property "Footprint" ""
+			(at 121.92 87.63 0)
+			(effects
+				(font
+					(size 1.27 1.27)
+				)
+				(hide yes)
+			)
+		)
+		(property "Datasheet" "~"
+			(at 121.92 87.63 0)
+			(effects
+				(font
+					(size 1.27 1.27)
+				)
+				(hide yes)
+			)
+		)
+		(property "Description" "Light emitting diode"
+			(at 121.92 87.63 0)
+			(effects
+				(font
+					(size 1.27 1.27)
+				)
+				(hide yes)
+			)
+		)
+		(property "Sim.Pins" "1=K 2=A"
+			(at 121.92 87.63 0)
+			(effects
+				(font
+					(size 1.27 1.27)
+				)
+				(hide yes)
+			)
+		)
+		(pin "2"
+		)
+		(pin "1"
+		)
+		(instances
+			(project ""
+				(path "/ed0095eb-57a0-4856-9ac4-7b40bd214a3a/eed1a5c9-5dce-4964-b7ee-57ee65be1a9d"
+					(reference "D1")
+					(unit 1)
+				)
+			)
+		)
+	)
+	(symbol
+		(lib_id "power:+3V3")
+		(at 128.27 87.63 0)
+		(unit 1)
+		(exclude_from_sim no)
+		(in_bom yes)
+		(on_board yes)
+		(dnp no)
+		(fields_autoplaced yes)
+		(property "Reference" "#PWR057"
+			(at 128.27 91.44 0)
+			(effects
+				(font
+					(size 1.27 1.27)
+				)
+				(hide yes)
+			)
+		)
+		(property "Value" "+3V3"
+			(at 128.27 82.55 0)
+			(effects
+				(font
+					(size 1.27 1.27)
+				)
+			)
+		)
+		(property "Footprint" ""
+			(at 128.27 87.63 0)
+			(effects
+				(font
+					(size 1.27 1.27)
+				)
+				(hide yes)
+			)
+		)
+		(property "Datasheet" ""
+			(at 128.27 87.63 0)
+			(effects
+				(font
+					(size 1.27 1.27)
+				)
+				(hide yes)
+			)
+		)
+		(property "Description" "Power symbol creates a global label with name \"+3V3\""
+			(at 128.27 87.63 0)
+			(effects
+				(font
+					(size 1.27 1.27)
+				)
+				(hide yes)
+			)
+		)
+		(pin "1"
+		)
+		(instances
+			(project ""
+				(path "/ed0095eb-57a0-4856-9ac4-7b40bd214a3a/eed1a5c9-5dce-4964-b7ee-57ee65be1a9d"
+					(reference "#PWR057")
+					(unit 1)
+				)
