File: PCB/configurations.kicad_sch (KiCad schematic)
At the start: 15 parts, among them U1 XC7A50T-FGG484, U7 MT25QL128ABA1EW7-0SIT

Commit message: cleaning the schematic up
Parts:
- D1: value LED -> KT-0805G; LCSC (none) -> C2297; MPN (none) -> KT-0805G
Other:
- moved on the sheet: D1, R24
Changed lines of the file:
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@@
 	(text "DONE sinks current! >"
 		(exclude_from_sim no)
-		(at 86.614 87.884 0)
+		(at 85.344 85.344 0)
 		(effects
 			(font
@@
 	(wire
 		(pts
-			(xy 128.27 87.63) (xy 125.73 87.63)
+			(xy 132.08 85.09) (xy 127 85.09)
 		)
 		(stroke
@@
 	(wire
 		(pts
-			(xy 100.33 87.63) (xy 107.95 87.63)
+			(xy 99.06 85.09) (xy 106.68 85.09)
 		)
 		(stroke
@@
 	(wire
 		(pts
-			(xy 118.11 87.63) (xy 115.57 87.63)
+			(xy 119.38 85.09) (xy 114.3 85.09)
 		)
 		(stroke
@@
 	)
 	(label "DONE"
-		(at 100.33 87.63 0)
+		(at 99.06 85.09 0)
 		(effects
 			(font
@@
 	)
 	(hierarchical_label "{JTAG}"
-		(shape input)
+		(shape bidirectional)
 		(at 168.91 116.84 0)
 		(effects
@@
 	(symbol
 		(lib_id "Device:R")
-		(at 111.76 87.63 90)
+		(at 110.49 85.09 90)
 		(unit 1)
 		(exclude_from_sim no)
@@
 		(fields_autoplaced yes)
 		(property "Reference" "R24"
-			(at 111.76 81.28 90)
+			(at 110.49 78.74 90)
 			(effects
 				(font
@@
 		)
 		(property "Value" "1k"
-			(at 111.76 83.82 90)
+			(at 110.49 81.28 90)
 			(effects
 				(font
@@
 		)
 		(property "Footprint" ""
-			(at 111.76 89.408 90)
+			(at 110.49 86.868 90)
 			(effects
 				(font
@@
 		)
 		(property "Datasheet" "~"
-			(at 111.76 87.63 0)
+			(at 110.49 85.09 0)
 			(effects
 				(font
@@
 		)
 		(property "Description" "Resistor"
-			(at 111.76 87.63 0)
+			(at 110.49 85.09 0)
 			(effects
 				(font
@@
 	(symbol
 		(lib_id "Device:LED")
-		(at 121.92 87.63 0)
+		(at 123.19 85.09 0)
 		(unit 1)
 		(exclude_from_sim no)
@@
 		(on_board yes)
 		(dnp no)
-		(fields_autoplaced yes)
 		(property "Reference" "D1"
-			(at 120.3325 81.28 0)
+			(at 123.19 78.74 0)
 			(effects
 				(font
@@
 			)
 		)
-		(property "Value" "LED"
-			(at 120.3325 83.82 0)
+		(property "Value" "KT-0805G"
+			(at 123.19 81.28 0)
 			(effects
 				(font
@@
 		)
 		(property "Footprint" ""
-			(at 121.92 87.63 0)
+			(at 123.19 85.09 0)
 			(effects
 				(font
@@
 		)
 		(property "Datasheet" "~"
-			(at 121.92 87.63 0)
+			(at 123.19 85.09 0)
 			(effects
 				(font
@@
 		)
 		(property "Description" "Light emitting diode"
-			(at 121.92 87.63 0)
+			(at 123.19 85.09 0)
 			(effects
 				(font
@@
 		)
 		(property "Sim.Pins" "1=K 2=A"
-			(at 121.92 87.63 0)
+			(at 123.19 85.09 0)
+			(effects
+				(font
+					(size 1.27 1.27)
+				)
+				(hide yes)
+			)
+		)
+		(property "MPN" "KT-0805G"
+			(at 123.19 85.09 0)
+			(effects
+				(font
+					(size 1.27 1.27)
+				)
+				(hide yes)
+			)
+		)
+		(property "LCSC" "C2297"
+			(at 123.19 85.09 0)
 			(effects
 				(font
@@
 	(symbol
 		(lib_id "power:+3V3")
-		(at 128.27 87.63 0)
+		(at 132.08 85.09 0)
 		(unit 1)
 		(exclude_from_sim no)
@@
 		(fields_autoplaced yes)
 		(property "Reference" "#PWR057"
-			(at 128.27 91.44 0)
+			(at 132.08 88.9 0)
 			(effects
 				(font
@@
 		)
 		(property "Value" "+3V3"
-			(at 128.27 82.55 0)
+			(at 132.08 80.01 0)
 			(effects
 				(font
@@
 		)
 		(property "Footprint" ""
-			(at 128.27 87.63 0)
+			(at 132.08 85.09 0)
 			(effects
 				(font
@@
 		)
 		(property "Datasheet" ""
-			(at 128.27 87.63 0)
+			(at 132.08 85.09 0)
 			(effects
 				(font
@@
 		)
 		(property "Description" "Power symbol creates a global label with name \"+3V3\""
-			(at 128.27 87.63 0)
+			(at 132.08 85.09 0)
 			(effects
 				(font

Commit message: added some configuration features and cleaned it up
Parts:
- removed R23: 4.7k, symbol Device:R
- added R27: 4k7, symbol Device:R_Small
- added SW1: SW_Push, symbol Switch:SW_Push
- R22: value 4.7k -> 4k7
Connections:
- net +3V3: now also R22.1, R27.2; no longer R22.2
- net GND: now also SW1.2
- net PROG_B: now reaches U1.N12 (PROGRAM_B_0)
- net PROG_B: now also R22.2, SW1.1; no longer R22.1
- net at U1.U12 (INIT_B_0): now also R27.1
Other:
- note added: "< DONE sinks current, LED turns off when done"
- note added: "< Manual configuration reset, it's a devboard so why not"
- note added: "MAYBE ADD ADC??"
- note removed: "DONE sinks current! >"
- moved on the sheet: C111, C112, D1, R14, R15, R19, R2, R20, R21, R24, R3, U1F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

Commit message: finished DDR wiring
Other:
- note added: "REVISIT BUTTONS"
Changed lines of the file:
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@@
+		)
+	)
+	(text "REVISIT BUTTONS"
+		(exclude_from_sim no)
+		(at 56.134 90.17 0)
+		(effects
+			(font
+				(size 1.905 1.905)
+			)
 		)
 	)

Commit message: cleaning up my DDR3 symbols, journaling about some DDR3
Other:
- note added: "REVISIT BUTTON MPN'S"
- note removed: "REVISIT BUTTONS"
Changed lines of the file:
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@@
 		)
 	)
-	(text "REVISIT BUTTONS"
+	(text "REVISIT BUTTON MPN'S"
 		(exclude_from_sim no)
-		(at 56.134 90.17 0)
+		(at 50.8 89.916 0)
 		(effects
 			(font

Commit message: cleaninng up the board, fixing some pullups, PCIe command pins
Parts:
- R19, R20, R21: value 10k -> 4k7
Other:
- note added: "Bank 14/15 need to be 3V3 because of CFGBVS"
- note removed: "Bank 13/14 need to be 3V3 because of CFGBVS"
Changed lines of the file:
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@@
 		)
 	)
-	(text "Bank 13/14 need to be 3V3 because of CFGBVS"
+	(text "Bank 14/15 need to be 3V3 because of CFGBVS"
 		(exclude_from_sim no)
 		(at 103.886 129.54 0)
@@
 	)
 	(symbol
+		(lib_id "Device:R")
+		(at 309.88 156.21 0)
+		(unit 1)
+		(exclude_from_sim no)
+		(in_bom yes)
+		(on_board yes)
+		(dnp no)
+		(fields_autoplaced yes)
+		(property "Reference" "R21"
+			(at 312.42 154.9399 0)
+			(effects
+				(font
+					(size 1.27 1.27)
+				)
+				(justify left)
+			)
+		)
+		(property "Value" "4k7"
+			(at 312.42 157.4799 0)
+			(effects
+				(font
+					(size 1.27 1.27)
+				)
+				(justify left)
+			)
+		)
+		(property "Footprint" ""
+			(at 308.102 156.21 90)
+			(effects
+				(font
+					(size 1.27 1.27)
+				)
+				(hide yes)
+			)
+		)
+		(property "Datasheet" "~"
+			(at 309.88 156.21 0)
+			(effects
+				(font
+					(size 1.27 1.27)
+				)
+				(hide yes)
+			)
+		)
+		(property "Description" "Resistor"
+			(at 309.88 156.21 0)
+			(effects
+				(font
+					(size 1.27 1.27)
+				)
+				(hide yes)
+			)
+		)
+		(pin "1"
+		)
+		(pin "2"
+		)
+		(instances
+			(project "PCB"
+				(path "/ed0095eb-57a0-4856-9ac4-7b40bd214a3a/eed1a5c9-5dce-4964-b7ee-57ee65be1a9d"
+					(reference "R21")
+					(unit 1)
+				)
+			)
+		)
+	)
+	(symbol
 		(lib_id "power:+3V3")
 		(at 167.64 173.99 0)
@@
 			)
 		)
-		(property "Value" "10k"
+		(property "Value" "4k7"
 			(at 294.64 157.4799 0)
 			(effects
@@
 	)
 	(symbol
-		(lib_id "Device:R")
-		(at 300.99 156.21 0)
+		(lib_id "power:+3V3")
+		(at 93.98 90.17 0)
 		(unit 1)
 		(exclude_from_sim no)
@@
 		(on_board yes)
 		(dnp no)
-		(fields_autoplaced yes)
-		(property "Reference" "R20"
-			(at 303.53 154.9399 0)
+		(property "Reference" "#PWR05"
+			(at 93.98 93.98 0)
 			(effects
 				(font
 					(size 1.27 1.27)
 				)
-				(justify left)
+				(hide yes)
 			)
 		)
-		(property "Value" "10k"
-			(at 303.53 157.4799 0)
+		(property "Value" "+3V3"
+			(at 93.472 86.106 0)
 			(effects
 				(font
 					(size 1.27 1.27)
 				)
-				(justify left)
 			)
 		)
 		(property "Footprint" ""
-			(at 299.212 156.21 90)
+			(at 93.98 90.17 0)
 			(effects
 				(font
@@
 			)
 		)
-		(property "Datasheet" "~"
-			(at 300.99 156.21 0)
+		(property "Datasheet" ""
+			(at 93.98 90.17 0)
 			(effects
 				(font
@@
 			)
 		)
-		(property "Description" "Resistor"
-			(at 300.99 156.21 0)
+		(property "Description" "Power symbol creates a global label with name \"+3V3\""
+			(at 93.98 90.17 0)
 			(effects
 				(font
@@
 		(pin "1"
 		)
-		(pin "2"
-		)
 		(instances
 			(project "PCB"
 				(path "/ed0095eb-57a0-4856-9ac4-7b40bd214a3a/eed1a5c9-5dce-4964-b7ee-57ee65be1a9d"
-					(reference "R20")
+					(reference "#PWR05")
 					(unit 1)
 				)
@@
 	(symbol
 		(lib_id "power:+3V3")
-		(at 93.98 90.17 0)
+		(at 181.61 152.4 0)
 		(unit 1)
 		(exclude_from_sim no)
@@
 		(on_board yes)
 		(dnp no)
-		(property "Reference" "#PWR05"
-			(at 93.98 93.98 0)
+		(fields_autoplaced yes)
+		(property "Reference" "#PWR041"
+			(at 181.61 156.21 0)
 			(effects
 				(font
@@
 		)
 		(property "Value" "+3V3"
-			(at 93.472 86.106 0)
+			(at 181.61 147.32 0)
 			(effects
 				(font
@@
 		)
 		(property "Footprint" ""
-			(at 93.98 90.17 0)
+			(at 181.61 152.4 0)
 			(effects
 				(font
@@
 		)
 		(property "Datasheet" ""
-			(at 93.98 90.17 0)
+			(at 181.61 152.4 0)
 			(effects
 				(font
@@
 		)
 		(property "Description" "Power symbol creates a global label with name \"+3V3\""
-			(at 93.98 90.17 0)
+			(at 181.61 152.4 0)
 			(effects
 				(font
@@
 			(project "PCB"
 				(path "/ed0095eb-57a0-4856-9ac4-7b40bd214a3a/eed1a5c9-5dce-4964-b7ee-57ee65be1a9d"
-					(reference "#PWR05")
+					(reference "#PWR041")
 					(unit 1)
 				)
@@
 	)
 	(symbol
-		(lib_id "power:+3V3")
-		(at 181.61 152.4 0)
+		(lib_id "Device:R")
+		(at 300.99 156.21 0)
 		(unit 1)
 		(exclude_from_sim no)
@@
 		(dnp no)
 		(fields_autoplaced yes)
-		(property "Reference" "#PWR041"
-			(at 181.61 156.21 0)
+		(property "Reference" "R20"
+			(at 303.53 154.9399 0)
 			(effects
 				(font
 					(size 1.27 1.27)
 				)
-				(hide yes)
+				(justify left)
 			)
 		)
-		(property "Value" "+3V3"
-			(at 181.61 147.32 0)
+		(property "Value" "4k7"
+			(at 303.53 157.4799 0)
 			(effects
 				(font
 					(size 1.27 1.27)
 				)
+				(justify left)
 			)
 		)
 		(property "Footprint" ""
-			(at 181.61 152.4 0)
+			(at 299.212 156.21 90)
 			(effects
 				(font
@@
 			)
 		)
-		(property "Datasheet" ""
-			(at 181.61 152.4 0)
+		(property "Datasheet" "~"
+			(at 300.99 156.21 0)
 			(effects
 				(font
@@
 			)
 		)
-		(property "Description" "Power symbol creates a global label with name \"+3V3\""
-			(at 181.61 152.4 0)
+		(property "Description" "Resistor"
+			(at 300.99 156.21 0)
 			(effects
 				(font
@@
 		(pin "1"
 		)
+		(pin "2"
+		)
 		(instances
 			(project "PCB"
 				(path "/ed0095eb-57a0-4856-9ac4-7b40bd214a3a/eed1a5c9-5dce-4964-b7ee-57ee65be1a9d"
-					(reference "#PWR041")
+					(reference "R20")
 					(unit 1)
 				)
@@
 					(unit 1)
 				)
-			)
-		)
-	)
-	(symbol
-		(lib_id "Device:R")
-		(at 309.88 156.21 0)
-		(unit 1)
-		(exclude_from_sim no)
-		(in_bom yes)
-		(on_board yes)
-		(dnp no)
-		(fields_autoplaced yes)
-		(property "Reference" "R21"
-			(at 312.42 154.9399 0)
-			(effects
-				(font
-					(size 1.27 1.27)
-				)
-				(justify left)
-			)
-		)
-		(property "Value" "10k"
-			(at 312.42 157.4799 0)
-			(effects
-				(font
-					(size 1.27 1.27)
-				)
-				(justify left)
-			)
-		)
-		(property "Footprint" ""
-			(at 308.102 156.21 90)
-			(effects
-				(font
-					(size 1.27 1.27)
-				)
-				(hide yes)
-			)
-		)
-		(property "Datasheet" "~"
-			(at 309.88 156.21 0)
-			(effects
-				(font
-					(size 1.27 1.27)
-				)
-				(hide yes)
-			)
-		)
-		(property "Description" "Resistor"
-			(at 309.88 156.21 0)
-			(effects
-				(font
-					(size 1.27 1.27)
-				)
-				(hide yes)
-			)
-		)
-		(pin "1"
-		)
-		(pin "2"
-		)
-		(instances
-			(project "PCB"
-				(path "/ed0095eb-57a0-4856-9ac4-7b40bd214a3a/eed1a5c9-5dce-4964-b7ee-57ee65be1a9d"
-					(reference "R21")
-					(unit 1)
-				)

Commit message: cleaning  up the schematic some more before sharing
Other:
- note removed: "REVISIT BUTTON MPN'S"
Changed lines of the file:
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@@
-		)
-	)
-	(text "REVISIT BUTTON MPN'S"
-		(exclude_from_sim no)
-		(at 50.8 89.916 0)
-		(effects
-			(font
-				(size 1.905 1.905)
-			)
 		)
 	)

Commit message: added basic capacitor footprints
Parts:
- C111: footprint (none) -> Capacitor_SMD:C_0402_1005Metric
Changed lines of the file:
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@@
 			)
 		)
-		(property "Footprint" ""
+		(property "Footprint" "Capacitor_SMD:C_0402_1005Metric"
 			(at 335.28 156.5148 0)
 			(effects

Commit message: LED parts and inductor footprints
Parts:
- D1: value KT-0805G -> KT-0805Y; footprint (none) -> LED_SMD:LED_0805_2012Metric; LCSC C2297 -> C2296; MPN KT-0805G -> KT-0805Y
Changed lines of the file:
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@@
+	)
+	(symbol
+		(lib_id "Device:LED")
+		(at 93.98 68.58 180)
+		(unit 1)
+		(exclude_from_sim no)
+		(in_bom yes)
+		(on_board yes)
+		(dnp no)
+		(property "Reference" "D1"
+			(at 93.98 64.516 0)
+			(effects
+				(font
+					(size 1.27 1.27)
+				)
+			)
+		)
+		(property "Value" "KT-0805Y"
+			(at 93.98 61.976 0)
+			(effects
+				(font
+					(size 1.27 1.27)
+				)
+			)
+		)
+		(property "Footprint" "LED_SMD:LED_0805_2012Metric"
+			(at 93.98 68.58 0)
+			(effects
+				(font
+					(size 1.27 1.27)
+				)
+				(hide yes)
+			)
+		)
+		(property "Datasheet" "~"
+			(at 93.98 68.58 0)
+			(effects
+				(font
+					(size 1.27 1.27)
+				)
+				(hide yes)
+			)
+		)
+		(property "Description" "Light emitting diode"
+			(at 93.98 68.58 0)
+			(effects
+				(font
+					(size 1.27 1.27)
+				)
+				(hide yes)
+			)
+		)
+		(property "Sim.Pins" "1=K 2=A"
+			(at 93.98 68.58 0)
+			(effects
+				(font
+					(size 1.27 1.27)
+				)
+				(hide yes)
+			)
+		)
+		(property "MPN" "KT-0805Y"
+			(at 93.98 68.58 0)
+			(effects
+				(font
+					(size 1.27 1.27)
+				)
+				(hide yes)
+			)
+		)
+		(property "LCSC" "C2296"
+			(at 93.98 68.58 0)
+			(effects
+				(font
+					(size 1.27 1.27)
+				)
+				(hide yes)
+			)
+		)
+		(pin "2"
+		)
+		(pin "1"
+		)
+		(instances
+			(project "PCB"
+				(path "/ed0095eb-57a0-4856-9ac4-7b40bd214a3a/eed1a5c9-5dce-4964-b7ee-57ee65be1a9d"
+					(reference "D1")
+					(unit 1)
+				)
+			)
+		)
 	)
 	(symbol
@@
 					(unit 1)
 				)
-			)
-		)
-	)
-	(symbol
-		(lib_id "Device:LED")
-		(at 93.98 68.58 0)
-		(mirror y)
-		(unit 1)
-		(exclude_from_sim no)
-		(in_bom yes)
-		(on_board yes)
-		(dnp no)
-		(property "Reference" "D1"
-			(at 93.98 62.23 0)
-			(effects
-				(font
-					(size 1.27 1.27)
-				)
-			)
-		)
-		(property "Value" "KT-0805G"
-			(at 93.98 64.77 0)
-			(effects
-				(font
-					(size 1.27 1.27)
-				)
-			)
-		)
-		(property "Footprint" ""
-			(at 93.98 68.58 0)
-			(effects
-				(font
-					(size 1.27 1.27)
-				)
-				(hide yes)
-			)
-		)
-		(property "Datasheet" "~"
-			(at 93.98 68.58 0)
-			(effects
-				(font
-					(size 1.27 1.27)
-				)
-				(hide yes)
-			)
-		)
-		(property "Description" "Light emitting diode"
-			(at 93.98 68.58 0)
-			(effects
-				(font
-					(size 1.27 1.27)
-				)
-				(hide yes)
-			)
-		)
-		(property "Sim.Pins" "1=K 2=A"
-			(at 93.98 68.58 0)
-			(effects
-				(font
-					(size 1.27 1.27)
-				)
-				(hide yes)
-			)
-		)
-		(property "MPN" "KT-0805G"
-			(at 93.98 68.58 0)
-			(effects
-				(font
-					(size 1.27 1.27)
-				)
-				(hide yes)
-			)
-		)
-		(property "LCSC" "C2297"
-			(at 93.98 68.58 0)
-			(effects
-				(font
-					(size 1.27 1.27)
-				)
-				(hide yes)
-			)
-		)
-		(pin "2"
-		)
-		(pin "1"
-		)
-		(instances
-			(project ""
-				(path "/ed0095eb-57a0-4856-9ac4-7b40bd214a3a/eed1a5c9-5dce-4964-b7ee-57ee65be1a9d"
-					(reference "D1")
-					(unit 1)
-				)
