File: PCB/ddr3l.kicad_sch (KiCad schematic)
At the start: 6 parts, among them U11 MT41J128M16JT-125:K

Commit message: more bus shenanigans, fixing some pins
Other:
- note added: "DECOUPLING"
Changed lines of the file:
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@@
 	(generator_version "9.0")
 	(paper "A3")
+	(bus_alias "DDR_ADDRESS"
+		(members)
+	)
+	(bus_alias "DDR_CLOCK"
+		(members)
+	)
+	(bus_alias "DDR_COMMAND"
+		(members)
+	)
+	(bus_alias "DDR_DATA"
+		(members)
+	)
 	(text "MT41J128M16JT-125:K\n16 Bit data width\n8 Bank machines\nNormal ordering"
 		(exclude_from_sim no)
@@
 		)
 	)
+	(text "DECOUPLING"
+		(exclude_from_sim no)
+		(at 169.418 44.704 0)
+		(effects
+			(font
+				(size 1.27 1.27)
+			)
+		)
+	)
 	(text "< Check phils lab for RC filter on Q pins? "
 		(exclude_from_sim no)
@@
 	)
 	(bus_entry
+		(at 142.24 144.78)
+		(size -2.54 -2.54)
+		(stroke
+			(width 0)
+			(type default)
+		)
+	)
+	(bus_entry
 		(at 199.39 104.14)
 		(size 2.54 -2.54)
@@
 	)
 	(bus_entry
-		(at 139.7 144.78)
-		(size -2.54 -2.54)
-		(stroke
-			(width 0)
-			(type default)
-		)
-	)
-	(bus_entry
 		(at 199.39 106.68)
 		(size 2.54 -2.54)
@@
 	(bus
 		(pts
-			(xy 137.16 142.24) (xy 137.16 44.45)
+			(xy 137.16 44.45) (xy 137.16 147.32)
 		)
 		(stroke
@@
 		)
 	)
+	(bus
+		(pts
+			(xy 139.7 135.89) (xy 139.7 142.24)
+		)
+		(stroke
+			(width 0)
+			(type default)
+		)
+	)
 	(wire
 		(pts
@@
 	(wire
 		(pts
-			(xy 139.7 144.78) (xy 156.21 144.78)
-		)
-		(stroke
-			(width 0)
-			(type default)
-		)
-	)
-	(wire
-		(pts
 			(xy 187.96 144.78) (xy 186.69 144.78)
 		)
@@
 	(bus
 		(pts
-			(xy 137.16 147.32) (xy 137.16 142.24)
-		)
-		(stroke
-			(width 0)
-			(type default)
-		)
-	)
-	(bus
-		(pts
 			(xy 201.93 81.28) (xy 201.93 78.74)
 		)
@@
 		)
 		(stroke
+			(width 0)
+			(type default)
+		)
+	)
+	(wire
+		(pts
+			(xy 142.24 144.78) (xy 156.21 144.78)
+		)
+		(stroke

Commit message: adding bus labels and hierarchial labels to root
Connections:
- net DDR_LDM renamed DDR_DQM0
- net DDR_LDQS+ renamed DDR_DQS0+
- net DDR_LDQS- renamed DDR_DQS0-
- net DDR_UDM renamed DDR_DQM1
- net DDR_UDQS+ renamed DDR_DQS1+
- net DDR_UDQS- renamed DDR_DQS1-
Other:
- moved on the sheet: C57, C58, R16, R17, R18, U11
