File: PCB/ddr3l.kicad_sch (KiCad schematic)
At the start: 33 parts, among them U11 MT41J128M16JT-125:K

Commit message: cleaning up my DDR3 symbols, journaling about some DDR3
Other:
- moved on the sheet: R16
Changed lines of the file:
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@@
 	)
 	(bus_alias "DDR_COMMAND"
-		(members "~{DDR_CS}" "~{DDR_RAS}" "~{DDR_CAS}" "~{DDR_WE}" "~{DDR_ODT}"
-			"~{DDR_RESET}" "DDR_CKE"
+		(members "~{DDR_RAS}" "~{DDR_CAS}" "~{DDR_WE}" "~{DDR_ODT}" "~{DDR_RESET}"
+			"DDR_CKE"
 		)
 	)
@@
 	(wire
 		(pts
+			(xy 134.62 200.66) (xy 132.08 200.66)
+		)
+		(stroke
+			(width 0)
+			(type default)
+		)
+	)
+	(wire
+		(pts
 			(xy 101.6 134.62) (xy 67.31 134.62)
 		)
@@
 	(wire
 		(pts
+			(xy 134.62 201.93) (xy 134.62 200.66)
+		)
+		(stroke
+			(width 0)
+			(type default)
+		)
+	)
+	(wire
+		(pts
 			(xy 146.05 176.53) (xy 132.08 176.53)
 		)
@@
 	(wire
 		(pts
-			(xy 134.62 200.66) (xy 132.08 200.66)
-		)
-		(stroke
-			(width 0)
-			(type default)
-		)
-	)
-	(wire
-		(pts
 			(xy 132.08 121.92) (xy 146.05 121.92)
 		)
@@
 	(wire
 		(pts
-			(xy 134.62 209.55) (xy 134.62 208.28)
+			(xy 134.62 210.82) (xy 134.62 209.55)
 		)
 		(stroke
@@
 	(symbol
 		(lib_id "power:GND")
-		(at 134.62 209.55 0)
+		(at 134.62 210.82 0)
 		(unit 1)
 		(exclude_from_sim no)
@@
 		(fields_autoplaced yes)
 		(property "Reference" "#PWR044"
-			(at 134.62 215.9 0)
+			(at 134.62 217.17 0)
 			(effects
 				(font
@@
 		)
 		(property "Value" "GND"
-			(at 134.62 214.63 0)
+			(at 134.62 215.9 0)
 			(effects
 				(font
@@
 		)
 		(property "Footprint" ""
-			(at 134.62 209.55 0)
+			(at 134.62 210.82 0)
 			(effects
 				(font
@@
 		)
 		(property "Datasheet" ""
-			(at 134.62 209.55 0)
+			(at 134.62 210.82 0)
 			(effects
 				(font
@@
 		)
 		(property "Description" "Power symbol creates a global label with name \"GND\" , ground"
-			(at 134.62 209.55 0)
+			(at 134.62 210.82 0)
 			(effects
 				(font
@@
 	(symbol
 		(lib_id "Device:R")
-		(at 134.62 204.47 0)
+		(at 134.62 205.74 0)
 		(unit 1)
 		(exclude_from_sim no)
@@
 		(fields_autoplaced yes)
 		(property "Reference" "R16"
-			(at 137.16 203.1999 0)
+			(at 137.16 204.4699 0)
 			(effects
 				(font
@@
 		)
 		(property "Value" "240"
-			(at 137.16 205.7399 0)
+			(at 137.16 207.0099 0)
 			(effects
 				(font
@@
 		)
 		(property "Footprint" ""
-			(at 132.842 204.47 90)
+			(at 132.842 205.74 90)
 			(effects
 				(font
@@
 		)
 		(property "Datasheet" "~"
-			(at 134.62 204.47 0)
+			(at 134.62 205.74 0)
 			(effects
 				(font
@@
 		)
 		(property "Description" "Resistor"
-			(at 134.62 204.47 0)
+			(at 134.62 205.74 0)
 			(effects
 				(font
