File: PCB/PCB.kicad_sch (KiCad schematic)
At the start: 1 part, among them U1 XC7A50T-FGG484

Commit message: USB ESD protection
Other:
- sheet FPGA Power renamed FPGA Power and Decoupling
- sheet Quad Buck Converter renamed Power Input Regulation
- added sheet USB-C and JTAG (usb.kicad_sch)
Changed lines of the file:
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@@
 	)
 	(sheet
-		(at 128.27 16.51)
-		(size 59.69 58.42)
-		(exclude_from_sim no)
-		(in_bom yes)
-		(on_board yes)
-		(dnp no)
-		(fields_autoplaced yes)
-		(stroke
-			(width 0.1524)
-			(type solid)
-		)
-		(fill
-			(color 0 0 0 0.0000)
-		)
-		(property "Sheetname" "Quad Buck Converter"
-			(at 128.27 15.7984 0)
+		(at 78.74 15.24)
+		(size 59.69 58.42)
+		(exclude_from_sim no)
+		(in_bom yes)
+		(on_board yes)
+		(dnp no)
+		(fields_autoplaced yes)
+		(stroke
+			(width 0.1524)
+			(type solid)
+		)
+		(fill
+			(color 0 0 0 0.0000)
+		)
+		(property "Sheetname" "Power Input Regulation"
+			(at 78.74 14.5284 0)
 			(effects
 				(font
@@
 		)
 		(property "Sheetfile" "power.kicad_sch"
-			(at 128.27 75.5146 0)
+			(at 78.74 74.2446 0)
 			(effects
 				(font
@@
 	)
 	(sheet
-		(at 191.77 114.3)
+		(at 78.74 114.3)
 		(size 59.69 58.42)
 		(exclude_from_sim no)
@@
 		)
 		(property "Sheetname" "FPGA Banks"
-			(at 191.77 113.5884 0)
+			(at 78.74 113.5884 0)
 			(effects
 				(font
@@
 		)
 		(property "Sheetfile" "banks.kicad_sch"
-			(at 191.77 173.3046 0)
+			(at 78.74 173.3046 0)
 			(effects
 				(font
@@
 	)
 	(sheet
-		(at 191.77 16.51)
-		(size 59.69 58.42)
-		(exclude_from_sim no)
-		(in_bom yes)
-		(on_board yes)
-		(dnp no)
-		(fields_autoplaced yes)
-		(stroke
-			(width 0.1524)
-			(type solid)
-		)
-		(fill
-			(color 0 0 0 0.0000)
-		)
-		(property "Sheetname" "FPGA Power"
-			(at 191.77 15.7984 0)
+		(at 205.74 15.24)
+		(size 59.69 58.42)
+		(exclude_from_sim no)
+		(in_bom yes)
+		(on_board yes)
+		(dnp no)
+		(fields_autoplaced yes)
+		(stroke
+			(width 0.1524)
+			(type solid)
+		)
+		(fill
+			(color 0 0 0 0.0000)
+		)
+		(property "Sheetname" "USB-C and JTAG"
+			(at 205.74 14.5284 0)
+			(effects
+				(font
+					(size 1.27 1.27)
+				)
+				(justify left bottom)
+			)
+		)
+		(property "Sheetfile" "usb.kicad_sch"
+			(at 205.74 74.2446 0)
+			(effects
+				(font
+					(size 1.27 1.27)
+				)
+				(justify left top)
+			)
+		)
+		(instances
+			(project "PCB"
+				(path "/ed0095eb-57a0-4856-9ac4-7b40bd214a3a"
+					(page "7")
+				)
+			)
+		)
+	)
+	(sheet
+		(at 15.24 114.3)
+		(size 59.69 58.42)
+		(exclude_from_sim no)
+		(in_bom yes)
+		(on_board yes)
+		(dnp no)
+		(fields_autoplaced yes)
+		(stroke
+			(width 0.1524)
+			(type solid)
+		)
+		(fill
+			(color 0 0 0 0.0000)
+		)
+		(property "Sheetname" "FPGA Power and Decoupling"
+			(at 15.24 113.5884 0)
 			(effects
 				(font
@@
 		)
 		(property "Sheetfile" "FPGA-power.kicad_sch"
-			(at 191.77 75.5146 0)
+			(at 15.24 173.3046 0)
 			(effects
 				(font
@@
 	)
 	(sheet
-		(at 128.27 114.3)
+		(at 142.24 15.24)
 		(size 59.69 58.42)
 		(exclude_from_sim no)
@@
 		)
 		(property "Sheetname" "FPGA Configurations"
-			(at 128.27 113.5884 0)
+			(at 142.24 14.5284 0)
 			(effects
 				(font
@@
 		)
 		(property "Sheetfile" "configurations.kicad_sch"
-			(at 128.27 173.3046 0)
-			(effects
-				(font
+			(at 142.24 74.2446 0)
+			(effects
+				(font

Commit message: wired JTAG bus
Other:
- sheet FPGA Configurations ports: added JTAG; removed none
- sheet USB-C and JTAG ports: added {JTAG}; removed none
Changed lines of the file:
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@@
 	(generator_version "9.0")
 	(paper "A3")
+	(wire
+		(pts
+			(xy 252.73 142.24) (xy 276.86 142.24)
+		)
+		(stroke
+			(width 0)
+			(type default)
+		)
+	)
 	(symbol
 		(lib_id "FPGA Accelerator:XC7A50T-FGG484")
@@
 	)
 	(sheet
-		(at 205.74 15.24)
+		(at 193.04 114.3)
 		(size 59.69 58.42)
 		(exclude_from_sim no)
@@
 		)
 		(property "Sheetname" "USB-C and JTAG"
-			(at 205.74 14.5284 0)
+			(at 193.04 113.5884 0)
 			(effects
 				(font
@@
 		)
 		(property "Sheetfile" "usb.kicad_sch"
-			(at 205.74 74.2446 0)
+			(at 193.04 173.3046 0)
 			(effects
 				(font
@@
 			)
 		)
+		(pin "{JTAG}" output
+			(at 252.73 142.24 0)
+			(effects
+				(font
+					(size 1.27 1.27)
+				)
+				(justify right)
+			)
+		)
 		(instances
 			(project "PCB"
@@
 	)
 	(sheet
-		(at 142.24 15.24)
+		(at 276.86 114.3)
 		(size 59.69 58.42)
 		(exclude_from_sim no)
@@
 		)
 		(property "Sheetname" "FPGA Configurations"
-			(at 142.24 14.5284 0)
+			(at 276.86 113.5884 0)
 			(effects
 				(font
@@
 		)
 		(property "Sheetfile" "configurations.kicad_sch"
-			(at 142.24 74.2446 0)
+			(at 276.86 173.3046 0)
 			(effects
 				(font
@@
 			)
 		)
+		(pin "JTAG" input
+			(at 276.86 142.24 180)
+			(effects
+				(font
+					(size 1.27 1.27)
+				)
+				(justify left)
+			)
+		)

Commit message: found the DDR3 memory I'm going to use
Other:
- note added: "MT41J128M16JT-125:K 16 Bit data width 8 Bank machines Normal ordering"
Changed lines of the file:
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@@
 	(generator_version "9.0")
 	(paper "A3")
+	(text "MT41J128M16JT-125:K\n16 Bit data width\n8 Bank machines\nNormal ordering"
+		(exclude_from_sim no)
+		(at 348.488 60.198 0)
+		(effects
+			(font
+				(size 2.54 2.54)
+			)
+		)
+	)
 	(wire
 		(pts

Commit message: adding DDR3L IC to schematic
Parts:
- added U11: MT41J128M16JT-125:K, Package_BGA:Micron_FBGA-96_8x14mm_Layout9x16_P0.8mm, symbol Memory_RAM:MT41K256M16TW
Connections:
- new net: U11.A1 (V_{DDQ}), U11.A8 (V_{DDQ}), U11.C1 (V_{DDQ}), U11.C9 (V_{DDQ}), U11.D2 (V_{DDQ}), U11.E9 (V_{DDQ}), U11.F1 (V_{DDQ}), U11.H2 (V_{DDQ}), U11.H9 (V_{DDQ})
- new net: U11.A9 (V_{SS}), U11.B3 (V_{SS}), U11.E1 (V_{SS}), U11.G8 (V_{SS}), U11.J2 (V_{SS}), U11.J8 (V_{SS}), U11.M1 (V_{SS}), U11.M9 (V_{SS}), U11.P1 (V_{SS}), U11.P9 (V_{SS}), U11.T1 (V_{SS}), U11.T9 (V_{SS})
- new net: U11.B1 (V_{SSQ}), U11.B9 (V_{SSQ}), U11.D1 (V_{SSQ}), U11.D8 (V_{SSQ}), U11.E2 (V_{SSQ}), U11.E8 (V_{SSQ}), U11.F9 (V_{SSQ}), U11.G1 (V_{SSQ}), U11.G9 (V_{SSQ})
- new net: U11.B2 (V_{DD}), U11.D9 (V_{DD}), U11.G7 (V_{DD}), U11.K2 (V_{DD}), U11.K8 (V_{DD}), U11.N1 (V_{DD}), U11.N9 (V_{DD}), U11.R1 (V_{DD}), U11.R9 (V_{DD})

Commit message: working on basic DDR3L wiring
Parts:
- removed U11: MT41J128M16JT-125:K, Package_BGA:Micron_FBGA-96_8x14mm_Layout9x16_P0.8mm, symbol Memory_RAM:MT41K256M16TW
Other:
- added sheet DDR3L (ddr3l.kicad_sch)
- note removed: "MT41J128M16JT-125:K 16 Bit data width 8 Bank machines Normal ordering"

Commit message: adding bus labels and hierarchial labels to root
Other:
- sheet DDR3L ports: added {DDR_ADDRESS}, {DDR_CLOCK}, {DDR_COMMAND}, {DDR_DATA}; removed none
Changed lines of the file:
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@@
+			)
+		)
+		(pin "{DDR_ADDRESS}" bidirectional
+			(at 194.31 72.39 180)
+			(effects
+				(font
+					(size 1.27 1.27)
+				)
+				(justify left)
+			)
+		)
+		(pin "{DDR_CLOCK}" input
+			(at 194.31 67.31 180)
+			(effects
+				(font
+					(size 1.27 1.27)
+				)
+				(justify left)
+			)
+		)
+		(pin "{DDR_COMMAND}" input
+			(at 194.31 62.23 180)
+			(effects
+				(font
+					(size 1.27 1.27)
+				)
+				(justify left)
+			)
+		)
+		(pin "{DDR_DATA}" bidirectional
+			(at 194.31 57.15 180)
+			(effects
+				(font
+					(size 1.27 1.27)
+				)
+				(justify left)
 			)
 		)

Commit message: some footprints added in, starting to work on flash
Parts:
- U1: footprint (none) -> Package_BGA:Xilinx_FGG484
Changed lines of the file:
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@@
 			)
 		)
-		(property "Footprint" ""
+		(property "Footprint" "Package_BGA:Xilinx_FGG484"
 			(at 645.16 57.15 0)
 			(effects
@@
 			)
 		)
-		(property "Footprint" ""
+		(property "Footprint" "Package_BGA:Xilinx_FGG484"
 			(at 515.62 213.36 0)
 			(effects
@@
 			)
 		)
-		(property "Footprint" ""
+		(property "Footprint" "Package_BGA:Xilinx_FGG484"
 			(at 622.3 175.26 0)
 			(effects
