File: PCB/PCB.kicad_sch (KiCad schematic)
At the start: 1 part, among them U1 XC7A50T-FGG484

Commit message: wiring QSPI
Other:
- sheet FPGA Banks ports: added {QSPI}; removed none
- sheet FPGA Configurations ports: added {JTAG}, {QSPI}; removed JTAG
Changed lines of the file:
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@@
 		)
 	)
+	(wire
+		(pts
+			(xy 307.34 210.82) (xy 252.73 210.82)
+		)
+		(stroke
+			(width 0)
+			(type default)
+		)
+	)
+	(wire
+		(pts
+			(xy 307.34 172.72) (xy 307.34 210.82)
+		)
+		(stroke
+			(width 0)
+			(type default)
+		)
+	)
 	(symbol
 		(lib_id "FPGA Accelerator:XC7A50T-FGG484")
@@
 	)
 	(sheet
-		(at 78.74 114.3)
+		(at 193.04 181.61)
 		(size 59.69 58.42)
 		(exclude_from_sim no)
@@
 		)
 		(property "Sheetname" "FPGA Banks"
-			(at 78.74 113.5884 0)
+			(at 193.04 180.8984 0)
 			(effects
 				(font
@@
 		)
 		(property "Sheetfile" "banks.kicad_sch"
-			(at 78.74 173.3046 0)
+			(at 193.04 240.6146 0)
 			(effects
 				(font
@@
 			)
 		)
+		(pin "{QSPI}" bidirectional
+			(at 252.73 210.82 0)
+			(effects
+				(font
+					(size 1.27 1.27)
+				)
+				(justify right)
+			)
+		)
 		(instances
 			(project "PCB"
@@
 			)
 		)
-		(pin "JTAG" input
+		(pin "{JTAG}" input
 			(at 276.86 142.24 180)
 			(effects
 				(font
+					(size 1.27 1.27)
+				)
+				(justify left)
+			)
+		)
+		(pin "{QSPI}" input
+			(at 307.34 172.72 270)
+			(effects
+				(font

Commit message: cleaning the schematic up
Parts:
- removed U1: XC7A50T-FGG484, Package_BGA:Xilinx_FGG484, symbol FPGA Accelerator:XC7A50T-FGG484
Other:
- sheet FPGA Banks renamed Artix 7 Banks
- added sheet PCIe GTP Transceivers (PCIe GTP Transceivers.kicad_sch)

Commit message: finished wiring the m.2 connector
Other:
- sheet M.2 M-Key Edge Connector ports: added {PCIe_CLK}, {PCIe_COMMAND}, {PCIe_RX}, {PCIe_TX}; removed none
Changed lines of the file:
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@@
+			)
+		)
+		(pin "{PCIe_CLK}" output
+			(at 179.07 73.66 0)
+			(effects
+				(font
+					(size 1.27 1.27)
+				)
+				(justify right)
+			)
+		)
+		(pin "{PCIe_COMMAND}" bidirectional
+			(at 179.07 69.85 0)
+			(effects
+				(font
+					(size 1.27 1.27)
+				)
+				(justify right)
+			)
+		)
+		(pin "{PCIe_RX}" input
+			(at 179.07 66.04 0)
+			(effects
+				(font
+					(size 1.27 1.27)
+				)
+				(justify right)
+			)
+		)
+		(pin "{PCIe_TX}" output
+			(at 179.07 62.23 0)
+			(effects
+				(font
+					(size 1.27 1.27)
+				)
+				(justify right)
 			)
 		)

Commit message: wiring the m.2 connector to the MGT transceivers
Other:
- sheet PCIe GTP Transceivers ports: added {PCIe_CLK}, {PCIe_RX}, {PCIe_TX}; removed none
Changed lines of the file:
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@@
 	(generator_version "9.0")
 	(paper "A3")
-	(wire
+	(bus
 		(pts
-			(xy 214.63 186.69) (xy 214.63 193.04)
+			(xy 267.97 57.15) (xy 273.05 57.15)
 		)
 		(stroke
@@
 		)
 	)
-	(wire
+	(bus
 		(pts
-			(xy 179.07 156.21) (xy 184.15 156.21)
+			(xy 267.97 135.89) (xy 273.05 135.89)
 		)
 		(stroke
@@
 		)
 	)
-	(sheet
-		(at 184.15 39.37)
+	(bus
+		(pts
+			(xy 303.53 166.37) (xy 303.53 172.72)
+		)
+		(stroke
+			(width 0)
+			(type default)
+		)
+	)
+	(bus
+		(pts
+			(xy 267.97 68.58) (xy 273.05 68.58)
+		)
+		(stroke
+			(width 0)
+			(type default)
+		)
+	)
+	(bus
+		(pts
+			(xy 267.97 60.96) (xy 273.05 60.96)
+		)
+		(stroke
+			(width 0)
+			(type default)
+		)
+	)
+	(sheet
+		(at 20.32 20.32)
 		(size 59.69 58.42)
 		(exclude_from_sim no)
@@
 		)
 		(property "Sheetname" "Power Input Regulation"
-			(at 184.15 38.6584 0)
+			(at 20.32 19.6084 0)
 			(effects
 				(font
@@
 		)
 		(property "Sheetfile" "power.kicad_sch"
-			(at 184.15 98.3746 0)
+			(at 20.32 79.3246 0)
 			(effects
 				(font
@@
 	)
 	(sheet
-		(at 119.38 193.04)
+		(at 208.28 172.72)
 		(size 59.69 58.42)
 		(exclude_from_sim no)
@@
 		)
 		(property "Sheetname" "DDR3L"
-			(at 119.38 192.3284 0)
+			(at 208.28 172.0084 0)
 			(effects
 				(font
@@
 		)
 		(property "Sheetfile" "ddr3l.kicad_sch"
-			(at 119.38 252.0446 0)
+			(at 208.28 231.7246 0)
 			(effects
 				(font
@@
 		)
 		(pin "{DDR_ADDRESS}" bidirectional
-			(at 179.07 214.63 0)
+			(at 267.97 194.31 0)
 			(effects
 				(font
@@
 		)
 		(pin "{DDR_CLOCK}" input
-			(at 179.07 219.71 0)
+			(at 267.97 199.39 0)
 			(effects
 				(font
@@
 		)
 		(pin "{DDR_COMMAND}" input
-			(at 179.07 224.79 0)
+			(at 267.97 204.47 0)
 			(effects
 				(font
@@
 		)
 		(pin "{DDR_DATA}" bidirectional
-			(at 179.07 229.87 0)
+			(at 267.97 209.55 0)
 			(effects
 				(font
@@
 	)
 	(sheet
-		(at 119.38 39.37)
+		(at 208.28 34.29)
 		(size 59.69 58.42)
 		(exclude_from_sim no)
@@
 		)
 		(property "Sheetname" "M.2 M-Key Edge Connector"
-			(at 119.38 38.6584 0)
+			(at 208.28 33.5784 0)
 			(effects
 				(font
@@
 		)
 		(property "Sheetfile" "m.2-m-key.kicad_sch"
-			(at 119.38 98.3746 0)
+			(at 208.28 93.2946 0)
 			(effects
 				(font
@@
 		)
 		(pin "{PCIe_CLK}" output
-			(at 179.07 73.66 0)
+			(at 267.97 68.58 0)
 			(effects
 				(font
@@
 		)
 		(pin "{PCIe_COMMAND}" bidirectional
-			(at 179.07 69.85 0)
+			(at 267.97 64.77 0)
 			(effects
 				(font
@@
 		)
 		(pin "{PCIe_RX}" input
-			(at 179.07 66.04 0)
+			(at 267.97 60.96 0)
 			(effects
 				(font
@@
 		)
 		(pin "{PCIe_TX}" output
-			(at 179.07 62.23 0)
+			(at 267.97 57.15 0)
 			(effects
 				(font
@@
 	)
 	(sheet
-		(at 248.92 128.27)
+		(at 273.05 34.29)
 		(size 59.69 58.42)
 		(exclude_from_sim no)
@@
 		)
 		(property "Sheetname" "PCIe GTP Transceivers"
-			(at 248.92 127.5584 0)
+			(at 273.05 33.5784 0)
 			(effects
 				(font
@@
 		)
 		(property "Sheetfile" "PCIe GTP Transceivers.kicad_sch"
-			(at 248.92 187.2746 0)
-			(effects
-				(font
-					(size 1.27 1.27)
-				)
-				(justify left top)
+			(at 273.05 93.2946 0)
+			(effects
+				(font
+					(size 1.27 1.27)
+				)
+				(justify left top)
+			)
+		)
+		(pin "{PCIe_CLK}" input
+			(at 273.05 68.58 180)
+			(effects
+				(font
+					(size 1.27 1.27)
+				)
+				(justify left)
+			)
+		)
+		(pin "{PCIe_RX}" output
+			(at 273.05 60.96 180)
+			(effects
+				(font
+					(size 1.27 1.27)
+				)
+				(justify left)
+			)
+		)
+		(pin "{PCIe_TX}" input
+			(at 273.05 57.15 180)
+			(effects
+				(font
+					(size 1.27 1.27)
+				)
+				(justify left)
 			)
 		)
@@
 	)
 	(sheet
-		(at 184.15 193.04)
+		(at 273.05 172.72)
 		(size 59.69 58.42)
 		(exclude_from_sim no)
@@
 		)
 		(property "Sheetname" "Artix 7 Banks"
-			(at 184.15 192.3284 0)
+			(at 273.05 172.0084 0)
 			(effects
 				(font
@@
 		)
 		(property "Sheetfile" "banks.kicad_sch"
-			(at 184.15 252.0446 0)
+			(at 273.05 231.7246 0)
 			(effects
 				(font
@@
 		)
 		(pin "{QSPI}" bidirectional
-			(at 214.63 193.04 90)
+			(at 303.53 172.72 90)
 			(effects
 				(font
@@
 	)
 	(sheet
-		(at 119.38 128.27)
+		(at 208.28 107.95)
 		(size 59.69 58.42)
 		(exclude_from_sim no)
@@
 		)
 		(property "Sheetname" "USB-C and JTAG"
-			(at 119.38 127.5584 0)
+			(at 208.28 107.2384 0)
 			(effects
 				(font
@@
 		)
 		(property "Sheetfile" "usb.kicad_sch"
-			(at 119.38 187.2746 0)
+			(at 208.28 166.9546 0)
 			(effects
 				(font
@@
 		)
 		(pin "{JTAG}" bidirectional
-			(at 179.07 156.21 0)
+			(at 267.97 135.89 0)
 			(effects
 				(font
@@
 	)
 	(sheet
-		(at 248.92 39.37)
+		(at 85.09 20.32)
 		(size 59.69 58.42)
 		(exclude_from_sim no)
@@
 		)
 		(property "Sheetname" "FPGA Power and Decoupling"
-			(at 248.92 38.6584 0)
+			(at 85.09 19.6084 0)
 			(effects
 				(font
@@
 		)
 		(property "Sheetfile" "FPGA-power.kicad_sch"
-			(at 248.92 98.3746 0)
+			(at 85.09 79.3246 0)
 			(effects
 				(font
@@
 	)
 	(sheet
-		(at 184.15 128.27)
+		(at 273.05 107.95)
 		(size 59.69 58.42)
 		(exclude_from_sim no)
@@
 		)
 		(property "Sheetname" "FPGA Configurations"
-			(at 184.15 127.5584 0)
+			(at 273.05 107.2384 0)
 			(effects
 				(font
@@
 		)
 		(property "Sheetfile" "configurations.kicad_sch"
-			(at 184.15 187.2746 0)
+			(at 273.05 166.9546 0)
 			(effects
 				(font
@@
 		)
 		(pin "{QSPI}" bidirectional
-			(at 214.63 186.69 270)
+			(at 303.53 166.37 270)
 			(effects
 				(font
@@
 		)
 		(pin "{JTAG}" bidirectional
-			(at 184.15 156.21 180)
-			(effects
-				(font
+			(at 273.05 135.89 180)
+			(effects
+				(font

Commit message: cleaning up DDR3 even more, finishing it's journaling
Other:
- sheet DDR3L renamed DDR3
- sheet DDR3: file ddr3l.kicad_sch -> ddr3.kicad_sch
Changed lines of the file:
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@@
 			(color 0 0 0 0.0000)
 		)
-		(property "Sheetname" "DDR3L"
+		(property "Sheetname" "DDR3"
 			(at 208.28 172.0084 0)
 			(effects
@@
 			)
 		)
-		(property "Sheetfile" "ddr3l.kicad_sch"
+		(property "Sheetfile" "ddr3.kicad_sch"
 			(at 208.28 231.7246 0)
 			(effects

Commit message: cleaninng up the board, fixing some pullups, PCIe command pins
Other:
- company: (none) -> Kai Pereira
- title: (none) -> M.2 FPGA Hardware Accelerator Devboard
Changed lines of the file:
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@@
 	(generator_version "9.0")
 	(paper "A3")
+	(title_block
+		(title "M.2 FPGA Hardware Accelerator Devboard")
+		(rev "v1.0")
+		(company "Kai Pereira")
+		(comment 1 "https://github.com/KaiPereira/M.2-FPGA-Accelerator")
+	)
 	(bus
 		(pts

Commit message: cleaning up the schematic some more, getting ready to wire the clocks, HDMI and ethernet!
Other:
- sheet FPGA Configurations renamed Artix 7 Configurations and Flash
- sheet FPGA Power and Decoupling renamed Artix 7 Power and Decoupling
- sheet PCIe GTP Transceivers renamed Artix 7 PCIe GTP Transceivers
- added sheet Ethernet (ethernet.kicad_sch)
- added sheet HDMI (hdmi.kicad_sch)

Commit message: cleaning up the schematic even more, it looks sick now
Other:
- sheet Artix 7 Banks ports: added {DDR_ADDRESS}, {DDR_CLK}, {DDR_COMMAND}, {DDR_DATA}, {PCIe_COMMAND}; removed none
- sheet DDR3 ports: added {DDR_CLK}; removed {DDR_CLOCK}
Changed lines of the file:
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@@
 	(bus
 		(pts
-			(xy 261.62 82.55) (xy 274.32 82.55)
+			(xy 261.62 139.7) (xy 274.32 139.7)
+		)
+		(stroke
+			(width 0)
+			(type default)
+		)
+	)
+	(bus
+		(pts
+			(xy 261.62 81.28) (xy 274.32 81.28)
 		)
 		(stroke
@@
 	(bus
 		(pts
-			(xy 232.41 110.49) (xy 232.41 116.84)
-		)
-		(stroke
-			(width 0)
-			(type default)
-		)
-	)
-	(bus
-		(pts
-			(xy 129.54 151.13) (xy 140.97 151.13)
+			(xy 231.14 110.49) (xy 231.14 116.84)
+		)
+		(stroke
+			(width 0)
+			(type default)
+		)
+	)
+	(bus
+		(pts
+			(xy 129.54 147.32) (xy 140.97 147.32)
+		)
+		(stroke
+			(width 0)
+			(type default)
+		)
+	)
+	(bus
+		(pts
+			(xy 129.54 151.13) (xy 201.93 151.13)
 		)
 		(stroke
@@
 		(pts
 			(xy 129.54 143.51) (xy 140.97 143.51)
+		)
+		(stroke
+			(width 0)
+			(type default)
+		)
+	)
+	(bus
+		(pts
+			(xy 261.62 151.13) (xy 274.32 151.13)
+		)
+		(stroke
+			(width 0)
+			(type default)
+		)
+	)
+	(bus
+		(pts
+			(xy 261.62 147.32) (xy 274.32 147.32)
+		)
+		(stroke
+			(width 0)
+			(type default)
+		)
+	)
+	(bus
+		(pts
+			(xy 261.62 143.51) (xy 274.32 143.51)
 		)
 		(stroke
@@
 		)
 		(pin "{DDR_ADDRESS}" bidirectional
-			(at 274.32 153.67 180)
-			(effects
-				(font
-					(size 1.27 1.27)
-				)
-				(justify left)
-			)
-		)
-		(pin "{DDR_CLOCK}" input
-			(at 274.32 148.59 180)
+			(at 274.32 143.51 180)
 			(effects
 				(font
@@
 		)
 		(pin "{DDR_COMMAND}" input
-			(at 274.32 143.51 180)
+			(at 274.32 151.13 180)
 			(effects
 				(font
@@
 		)
 		(pin "{DDR_DATA}" bidirectional
-			(at 274.32 138.43 180)
+			(at 274.32 139.7 180)
+			(effects
+				(font
+					(size 1.27 1.27)
+				)
+				(justify left)
+			)
+		)
+		(pin "{DDR_CLK}" input
+			(at 274.32 147.32 180)
 			(effects
 				(font
@@
 			)
 		)
-		(pin "{PCIe_CLK}" output
-			(at 129.54 151.13 0)
-			(effects
-				(font
-					(size 1.27 1.27)
-				)
-				(justify right)
-			)
-		)
-		(pin "{PCIe_COMMAND}" bidirectional
-			(at 129.54 147.32 0)
-			(effects
-				(font
-					(size 1.27 1.27)
-				)
-				(justify right)
-			)
-		)
 		(pin "{PCIe_RX}" input
 			(at 129.54 143.51 0)
@@
 			)
 		)
+		(pin "{PCIe_CLK}" output
+			(at 129.54 147.32 0)
+			(effects
+				(font
+					(size 1.27 1.27)
+				)
+				(justify right)
+			)
+		)
+		(pin "{PCIe_COMMAND}" bidirectional
+			(at 129.54 151.13 0)
+			(effects
+				(font
+					(size 1.27 1.27)
+				)
+				(justify right)
+			)
+		)
 		(instances
 			(project "PCB"
@@
 			)
 		)
-		(pin "{PCIe_CLK}" input
-			(at 140.97 151.13 180)
-			(effects
-				(font
-					(size 1.27 1.27)
-				)
-				(justify left)
-			)
-		)
 		(pin "{PCIe_RX}" output
 			(at 140.97 143.51 180)
@@
 			)
 		)
+		(pin "{PCIe_CLK}" input
+			(at 140.97 147.32 180)
+			(effects
+				(font
+					(size 1.27 1.27)
+				)
+				(justify left)
+			)
+		)
 		(instances
 			(project "PCB"
@@
 			)
 		)
+		(pin "{PCIe_COMMAND}" bidirectional
+			(at 201.93 151.13 180)
+			(effects
+				(font
+					(size 1.27 1.27)
+				)
+				(justify left)
+			)
+		)
+		(pin "{DDR_ADDRESS}" bidirectional
+			(at 261.62 143.51 0)
+			(effects
+				(font
+					(size 1.27 1.27)
+				)
+				(justify right)
+			)
+		)
+		(pin "{DDR_CLK}" output
+			(at 261.62 147.32 0)
+			(effects
+				(font
+					(size 1.27 1.27)
+				)
+				(justify right)
+			)
+		)
+		(pin "{DDR_COMMAND}" output
+			(at 261.62 151.13 0)
+			(effects
+				(font
+					(size 1.27 1.27)
+				)
+				(justify right)
+			)
+		)
+		(pin "{DDR_DATA}" bidirectional
+			(at 261.62 139.7 0)
+			(effects
+				(font
+					(size 1.27 1.27)
+				)
+				(justify right)
+			)
+		)
 		(pin "{QSPI}" bidirectional
-			(at 232.41 116.84 90)
+			(at 231.14 116.84 90)
 			(effects
 				(font
@@
 		)
 		(pin "{JTAG}" bidirectional
-			(at 274.32 82.55 180)
+			(at 274.32 81.28 180)
 			(effects
 				(font
@@
 		)
 		(pin "{QSPI}" bidirectional
-			(at 232.41 110.49 270)
+			(at 231.14 110.49 270)
 			(effects
 				(font
@@
 		)
 		(pin "{JTAG}" bidirectional
-			(at 261.62 82.55 0)
-			(effects
-				(font
+			(at 261.62 81.28 0)
+			(effects
+				(font
