File: PCB/PCB.kicad_sch (KiCad schematic)
At the start: 0 parts

Commit message: almost done wiring HDMI
Other:
- sheet Artix 7 Banks ports: added {HDMI}; removed none
- sheet HDMI ports: added {HDMI}; removed none
Changed lines of the file:
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@@
+	(bus
+		(pts
+			(xy 236.22 175.26) (xy 236.22 189.23)
+		)
+		(stroke
+			(width 0)
+			(type default)
+		)
+	)
 	(bus
 		(pts
@@
 			)
 		)
+		(pin "{HDMI}" bidirectional
+			(at 236.22 175.26 270)
+			(effects
+				(font
+					(size 1.27 1.27)
+				)
+				(justify left)
+			)
+		)
 		(instances
 			(project "PCB"
@@
 			)
 		)
+		(pin "{HDMI}" bidirectional
+			(at 236.22 189.23 90)
+			(effects
+				(font
+					(size 1.27 1.27)
+				)
+				(justify right)
+			)
+		)

Commit message: kind of finished wiring ethernet, cleaning stuff up
Other:
- sheet Artix 7 Banks ports: added {EPHY}; removed none
- sheet Ethernet ports: added {EPHY}; removed none
Changed lines of the file:
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@@
+	(bus
+		(pts
+			(xy 231.14 182.88) (xy 231.14 175.26)
+		)
+		(stroke
+			(width 0)
+			(type default)
+		)
+	)
 	(bus
 		(pts
@@
 	(bus
 		(pts
+			(xy 173.99 189.23) (xy 173.99 182.88)
+		)
+		(stroke
+			(width 0)
+			(type default)
+		)
+	)
+	(bus
+		(pts
 			(xy 129.54 147.32) (xy 140.97 147.32)
 		)
@@
 		(pts
 			(xy 261.62 151.13) (xy 274.32 151.13)
+		)
+		(stroke
+			(width 0)
+			(type default)
+		)
+	)
+	(bus
+		(pts
+			(xy 173.99 182.88) (xy 231.14 182.88)
 		)
 		(stroke
@@
 			)
 		)
+		(pin "{EPHY}" bidirectional
+			(at 173.99 189.23 90)
+			(effects
+				(font
+					(size 1.27 1.27)
+				)
+				(justify right)
+			)
+		)
 		(instances
 			(project "PCB"
@@
 			(effects
 				(font
+					(size 1.27 1.27)
+				)
+				(justify left)
+			)
+		)
+		(pin "{EPHY}" bidirectional
+			(at 231.14 175.26 270)
+			(effects
+				(font

Commit message: basic HDMI ESD protection I think
Changed lines of the file:
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@@
 	(bus
 		(pts
-			(xy 236.22 175.26) (xy 236.22 189.23)
+			(xy 233.68 175.26) (xy 233.68 189.23)
 		)
 		(stroke
@@
 	(bus
 		(pts
-			(xy 231.14 182.88) (xy 231.14 175.26)
+			(xy 228.6 182.88) (xy 228.6 175.26)
 		)
 		(stroke
@@
 	(bus
 		(pts
-			(xy 173.99 189.23) (xy 173.99 182.88)
+			(xy 172.72 189.23) (xy 172.72 182.88)
 		)
 		(stroke
@@
 	(bus
 		(pts
-			(xy 173.99 182.88) (xy 231.14 182.88)
+			(xy 172.72 182.88) (xy 228.6 182.88)
 		)
 		(stroke
@@
 		)
 		(pin "{EPHY}" bidirectional
-			(at 173.99 189.23 90)
+			(at 172.72 189.23 90)
 			(effects
 				(font
@@
 			)
 		)
+		(pin "{EPHY}" bidirectional
+			(at 228.6 175.26 270)
+			(effects
+				(font
+					(size 1.27 1.27)
+				)
+				(justify left)
+			)
+		)
 		(pin "{HDMI}" bidirectional
-			(at 236.22 175.26 270)
-			(effects
-				(font
-					(size 1.27 1.27)
-				)
-				(justify left)
-			)
-		)
-		(pin "{EPHY}" bidirectional
-			(at 231.14 175.26 270)
+			(at 233.68 175.26 270)
 			(effects
 				(font
@@
 		)
 		(pin "{HDMI}" bidirectional
-			(at 236.22 189.23 90)
-			(effects
-				(font
+			(at 233.68 189.23 90)
+			(effects
+				(font

Commit message: wired the 100MHz clock for PLL's
Other:
- sheet Artix 7 Banks ports: added BUCK_PG4; removed none
- sheet Power Input Regulation ports: added BUCK_PG4; removed none
Changed lines of the file:
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@@
+		)
+	)
+	(wire
+		(pts
+			(xy 129.54 82.55) (xy 245.11 82.55)
+		)
+		(stroke
+			(width 0)
+			(type default)
 		)
 	)
@@
 		(pts
 			(xy 261.62 151.13) (xy 274.32 151.13)
+		)
+		(stroke
+			(width 0)
+			(type default)
+		)
+	)
+	(wire
+		(pts
+			(xy 245.11 82.55) (xy 245.11 116.84)
 		)
 		(stroke
@@
 			)
 		)
+		(pin "BUCK_PG4" output
+			(at 129.54 82.55 0)
+			(effects
+				(font
+					(size 1.27 1.27)
+				)
+				(justify right)
+			)
+		)
 		(instances
 			(project "PCB"
@@
 			)
 		)
+		(pin "BUCK_PG4" input
+			(at 245.11 116.84 90)
+			(effects
+				(font
+					(size 1.27 1.27)
+				)
+				(justify right)
+			)
+		)

Commit message: completely finished the clock, cleaned up the schematic
Changed lines of the file:
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@@
 	(wire
 		(pts
-			(xy 129.54 82.55) (xy 245.11 82.55)
+			(xy 134.62 81.28) (xy 134.62 128.27)
 		)
 		(stroke
@@
 	(wire
 		(pts
-			(xy 245.11 82.55) (xy 245.11 116.84)
+			(xy 134.62 128.27) (xy 201.93 128.27)
 		)
 		(stroke
@@
 		(pts
 			(xy 261.62 147.32) (xy 274.32 147.32)
+		)
+		(stroke
+			(width 0)
+			(type default)
+		)
+	)
+	(wire
+		(pts
+			(xy 129.54 81.28) (xy 134.62 81.28)
 		)
 		(stroke
@@
 		)
 		(pin "BUCK_PG4" output
-			(at 129.54 82.55 0)
+			(at 129.54 81.28 0)
 			(effects
 				(font
@@
 		)
 		(pin "BUCK_PG4" input
-			(at 245.11 116.84 90)
-			(effects
-				(font
-					(size 1.27 1.27)
-				)
-				(justify right)
-			)
-		)
+			(at 201.93 128.27 180)
+			(effects
+				(font
+					(size 1.27 1.27)
+				)
+				(justify left)
+			)
+		)

Commit message: added UART debugging
Other:
- sheet Artix 7 Banks ports: added {UART}; removed none
- sheet USB-C and JTAG ports: added {UART}; removed none
Changed lines of the file:
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@@
-		)
-	)
-	(bus
-		(pts
-			(xy 261.62 81.28) (xy 274.32 81.28)
-		)
-		(stroke
-			(width 0)
-			(type default)
 		)
 	)
@@
 	(bus
 		(pts
+			(xy 261.62 78.74) (xy 274.32 78.74)
+		)
+		(stroke
+			(width 0)
+			(type default)
+		)
+	)
+	(bus
+		(pts
+			(xy 233.68 83.82) (xy 274.32 83.82)
+		)
+		(stroke
+			(width 0)
+			(type default)
+		)
+	)
+	(bus
+		(pts
 			(xy 228.6 182.88) (xy 228.6 175.26)
 		)
@@
 	(bus
 		(pts
-			(xy 231.14 110.49) (xy 231.14 116.84)
+			(xy 228.6 110.49) (xy 228.6 116.84)
 		)
 		(stroke
@@
 		(pts
 			(xy 129.54 151.13) (xy 201.93 151.13)
+		)
+		(stroke
+			(width 0)
+			(type default)
+		)
+	)
+	(bus
+		(pts
+			(xy 233.68 116.84) (xy 233.68 83.82)
 		)
 		(stroke
@@
 			)
 		)
-		(pin "{QSPI}" bidirectional
-			(at 231.14 116.84 90)
-			(effects
-				(font
-					(size 1.27 1.27)
-				)
-				(justify right)
-			)
-		)
 		(pin "{EPHY}" bidirectional
 			(at 228.6 175.26 270)
@@
 				)
 				(justify left)
+			)
+		)
+		(pin "{QSPI}" bidirectional
+			(at 228.6 116.84 90)
+			(effects
+				(font
+					(size 1.27 1.27)
+				)
+				(justify right)
+			)
+		)
+		(pin "{UART}" bidirectional
+			(at 233.68 116.84 90)
+			(effects
+				(font
+					(size 1.27 1.27)
+				)
+				(justify right)
 			)
 		)
@@
 		)
 		(pin "{JTAG}" bidirectional
-			(at 274.32 81.28 180)
+			(at 274.32 78.74 180)
+			(effects
+				(font
+					(size 1.27 1.27)
+				)
+				(justify left)
+			)
+		)
+		(pin "{UART}" bidirectional
+			(at 274.32 83.82 180)
 			(effects
 				(font
@@
 			)
 		)
+		(pin "{JTAG}" bidirectional
+			(at 261.62 78.74 0)
+			(effects
+				(font
+					(size 1.27 1.27)
+				)
+				(justify right)
+			)
+		)
 		(pin "{QSPI}" bidirectional
-			(at 231.14 110.49 270)
-			(effects
-				(font
-					(size 1.27 1.27)
-				)
-				(justify left)
-			)
-		)
-		(pin "{JTAG}" bidirectional
-			(at 261.62 81.28 0)
-			(effects
-				(font
-					(size 1.27 1.27)
-				)
-				(justify right)
-			)
-		)
+			(at 228.6 110.49 270)
+			(effects
+				(font
+					(size 1.27 1.27)
+				)
+				(justify left)
+			)
+		)

Commit message: finisehed upassigning resistor footprints
Other:
- note added: "For a production board: - make R8, R6, R35 and R33, 0402 and exact! - make 47nF caps 0402"
Changed lines of the file:
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@@
 		(comment 1 "https://github.com/KaiPereira/M.2-FPGA-Accelerator")
+	)
+	(text "For a production board: \n- make R8, R6, R35 and R33, 0402 and exact!\n- make 47nF caps 0402"
+		(exclude_from_sim no)
+		(at 16.256 18.542 0)
+		(effects
+			(font
+				(size 1.27 1.27)
+			)
+			(justify left)
+		)
 	)
 	(bus
