File: PCB/m.2-m-key.kicad_sch (KiCad schematic)
At the start: 16 parts, among them J1 M.2 M-Key Edge Connector

Commit message: fixed JTAGG, working on power architecture
Other:
- moved on the sheet: C1, C10, C11, C12, C13, C14, C15, C2, C3, C4, C5, C6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

Commit message: finished wiring USB buck
Parts:
- removed C9: 100n, Capacitor_SMD:C_0201_0603Metric, symbol Device:C
- C1, C2, C3, C4, C5, C6, C7, C8: value 100n -> 470n
Connections:
- net +3V3 renamed +VM2_3V3

Commit message: working on the power MXU
Parts:
- added C9: 470n, Capacitor_SMD:C_0201_0603Metric, symbol Device:C
Connections:
- net +VM2_3V3: now also C9.1
- net GND: now also C9.2
Other:
- moved on the sheet: C1, C10, C11, C12, C13, C14, C15, C2, C3, C4, C5, C6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

Commit message: cleaning up the schematic a bit after this grind
Other:
- note added: "One 470nF per pin One 1uF + 10uF per group"
- note removed: "One 100nF per pin One 1uF + 10uF per group"
- moved on the sheet: C1, C10, C11, C12, C13, C14, C15, C2, C3, C4, C5, C6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

Commit message: backlogging journal decoupling/filtering, don!
Other:
- note added: "< Too much inrush?"
Changed lines of the file:
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@@
 	(generator_version "9.0")
 	(paper "A4")
+	(text "< Too much inrush? "
+		(exclude_from_sim no)
+		(at 260.096 52.832 0)
+		(effects
+			(font
+				(size 1.27 1.27)
+			)
+		)
+	)
 	(text "One 470nF per pin\nOne 1uF + 10uF per group"
 		(exclude_from_sim no)

Commit message: finished the configurations
Parts:
- C1, C2, C3, C4, C5, C6, C7, C8, C9: value 470n -> 100n

Commit message: an LED + changing the decoupling on the m.2 edge connector
Parts:
- removed C10, C11, C12: 1u, Capacitor_SMD:C_0402_1005Metric, symbol Device:C
- removed C13, C14: 10u, Capacitor_SMD:C_0603_1608Metric, symbol Device:C
- removed C3, C4, C5, C6, C7, C8, C9: 100n, Capacitor_SMD:C_0201_0603Metric, symbol Device:C
- C1, C2: value 100n -> 4u7; footprint Capacitor_SMD:C_0201_0603Metric -> Capacitor_SMD:C_0603_1608Metric
- C15: value 10u -> 4u7
Other:
- note removed: "< Too much inrush?"
- note removed: "One 470nF per pin One 1uF + 10uF per group"
- moved on the sheet: C15

Commit message: working on wiring PCIe buses
Parts:
- removed J1: M.2 M-Key Edge Connector, symbol Connector:Bus_M.2_Socket_M
- added C10, C3, C4, C5, C6, C7, C8, C9: 100n, symbol Device:C_Small
- added J3: Bus_M.2_Socket_M, symbol FPGA Accelerator:Bus_M.2_Socket_M
Connections:
- net +VM2_3V3: now also J3.12 (3.3V), J3.14 (3.3V), J3.16 (3.3V), J3.18 (3.3V), J3.2 (3.3V), J3.4 (3.3V), J3.70 (3.3V), J3.72 (3.3V), J3.74 (3.3V)
- net GND: now also J3.1 (GND), J3.15 (GND), J3.21 (GND), J3.27 (GND), J3.3 (GND), J3.33 (GND), J3.39 (GND), J3.45 (GND), J3.51 (GND), J3.57 (GND), J3.71 (GND), J3.73 (GND), J3.75 (GND), J3.9 (GND)
- new net: C9.2, J3.5 (PERn3)
- new net: C10.2, J3.7 (PERp3)
- new net: C3.2, J3.43 (PERp0/SATA-B-)
- new net: C7.2, J3.17 (PERn2)
- new net: C4.2, J3.41 (PERn0/SATA-B+)
- new net: C5.2, J3.29 (PERn1)
- new net: C6.2, J3.31 (PERp1)
- new net: C8.2, J3.19 (PERp2)
- new net PCIe_RX0+: C3.1
- new net PCIe_RX0-: C4.1
- new net PCIe_RX1+: C6.1
- new net PCIe_RX1-: C5.1
- new net PCIe_RX2+: C8.1
- new net PCIe_RX2-: C7.1
- new net PCIe_RX3+: C10.1
- new net PCIe_RX3-: C9.1
- new net PCIe_TX0+: J3.49 (PETp0/SATA-A+)
- new net PCIe_TX0-: J3.47 (PETn0/SATA-A-)
- new net PCIe_TX1+: J3.37 (PETp1)
- new net PCIe_TX1-: J3.35 (PETn1)
- new net PCIe_TX2+: J3.25 (PETp2)
- new net PCIe_TX2-: J3.23 (PETn2)
- new net PCIe_TX3+: J3.13 (PETp3)
- new net PCIe_TX3-: J3.11 (PETn3)
