File: PCB/m.2-m-key.kicad_sch (KiCad schematic)
At the start: 12 parts, among them J1 Bus_M.2_Edge_M

Commit message: finished wiring the m.2 connector
Connections:
- no-connect marks 2 -> 4
Other:
- note added: "< Don't need (PCIe)"
- note added: "I inverted the bus symbol, to create an edge connector symbol DOUBLE CHECK the transmit/receive are the right orientation!! Pg 150, https://picture.iczhiku.com/resource/eetop/sHksKPigIJigRbbx.pdf All the NC's are SATA only features!"
- note removed: "I inverted the bus symbol, to create an edge connector symbol DOUBLE CHECK the transmit/receive are the right orientation!! Pg 150, https://picture.iczhiku.com/resource/eetop/sHksKPigIJigRbbx.pdf"
Changed lines of the file:
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@@
 	(generator_version "9.0")
 	(paper "A4")
+	(bus_alias "PCIe_CLK"
+		(members "PCIe_REFCLK+" "PCIe_REFCLK-")
+	)
+	(bus_alias "PCIe_COMMAND"
+		(members "~{PCIe_PERST}" "~{PCIe_CLKREQ}" "~{PCIe_PEWAKE}")
+	)
+	(bus_alias "PCIe_RX"
+		(members "PCIe_RX0+" "PCIe_RX0-" "PCIe_RX1+" "PCIe_RX1-" "PCIe_RX2+" "PCIe_RX2-"
+			"PCIe_RX3+" "PCIe_RX3-"
+		)
+	)
+	(bus_alias "PCIe_TX"
+		(members "PCIe_TX0+" "PCIe_TX0-" "PCIe_TX1+" "PCIe_TX1-" "PCIe_TX2+" "PCIe_TX2-"
+			"PCIe_TX3+" "PCIe_TX3-"
+		)
+	)
 	(text "Transmiting (TX) TO the FPGA,\nReceiving (RX) FROM the FPGA > "
 		(exclude_from_sim no)
@@
 		)
 	)
-	(text "I inverted the bus symbol, to create an edge connector symbol\nDOUBLE CHECK the transmit/receive are the right orientation!!\nPg 150, https://picture.iczhiku.com/resource/eetop/sHksKPigIJigRbbx.pdf"
+	(text "< Don't need (PCIe)"
 		(exclude_from_sim no)
-		(at 55.372 48.514 0)
+		(at 188.214 142.494 0)
+		(effects
+			(font
+				(size 1.27 1.27)
+			)
+		)
+	)
+	(text "I inverted the bus symbol, to create an edge connector symbol\nDOUBLE CHECK the transmit/receive are the right orientation!!\nPg 150, https://picture.iczhiku.com/resource/eetop/sHksKPigIJigRbbx.pdf\n\nAll the NC's are SATA only features!"
+		(exclude_from_sim no)
+		(at 55.372 47.752 0)
 		(effects
 			(font
@@
 	)
 	(no_connect
+		(at 173.99 124.46)
+	)
+	(no_connect
+		(at 173.99 142.24)
+	)
+	(no_connect

Commit message: dampening and cleaning up the schematic
Parts:
- added C11, C12: 100n, symbol Device:C_Small
- added R25, R26: 22, symbol Device:R_Small
Connections:
- net PCIe_REFCLK+: now also C11.1; no longer J1.55 (REFCLKp)
- net PCIe_REFCLK-: now also C12.1; no longer J1.53 (REFCLKn)
- net ~{PCIe_CLKREQ}: now also R26.1; no longer J1.52 (~{CLKREQ})
- net ~{PCIe_PEWAKE}: now also R25.1; no longer J1.54 (~{PEWAKE})
- new net: J1.54 (~{PEWAKE}), R25.2
- new net: C12.2, J1.53 (REFCLKn)
- new net: C11.2, J1.55 (REFCLKp)
- new net: J1.52 (~{CLKREQ}), R26.2
Other:
- note added: "< Don't need low power states"
- note added: "Dampening for long, slow traces >"
- note removed: "< Don't need (PCIe)"
- note removed: "RESEARCH MORE ON WHAT the AC CAPS are for!!"
- moved on the sheet: C1, C10, C15, C2, C3, C4, C5, C6, C7, C8, C9, J1

Commit message: changing ac couping value to 220n for backward compatibility
Parts:
- C10, C11, C12, C3, C4, C5, C6, C7, C8, C9: value 100n -> 220n
Connections:
- net PCIe_TX1+: now also C5.1; no longer C6.1
- net PCIe_TX1-: now also C6.1; no longer C5.1
- net PCIe_TX2+: now also C7.1; no longer C8.1
- net PCIe_TX2-: now also C8.1; no longer C7.1
- net PCIe_TX3+: now also C9.1; no longer C10.1
- net PCIe_TX3-: now also C10.1; no longer C9.1
- net at C9.2: now also J1.7 (PETp3); no longer J1.5 (PETn3)
- net at C10.2: now also J1.5 (PETn3); no longer J1.7 (PETp3)
- net at C7.2: now also J1.19 (PETp2); no longer J1.17 (PETn2)
- net at J1.29 (PETn1): now also C6.2; no longer C5.2
- net at J1.31 (PETp1): now also C5.2; no longer C6.2
- net at C8.2: now also J1.17 (PETn2); no longer J1.19 (PETp2)
Other:
- note added: "I inverted the bus symbol, to create an edge connector symbol DOUBLE CHECK the transmit/receive are the right orientation!! Pg 150, https://picture.iczhiku.com/resource/eetop/sHksKPigIJigRbbx.pdf All the NC's are SATA only features! AC Coupling should be near the edge connector to reduce impedance discontinuities! 220nF for backwards compatibility!"
- note removed: "I inverted the bus symbol, to create an edge connector symbol DOUBLE CHECK the transmit/receive are the right orientation!! Pg 150, https://picture.iczhiku.com/resource/eetop/sHksKPigIJigRbbx.pdf All the NC's are SATA only features!"

Commit message: wiring the m.2 connector to the MGT transceivers
Other:
- note added: "Transmiting (TX) FROM the FPGA TO the host Receiving (RX) FROM the host TO the FPGA >"
- note removed: "Transmiting (TX) TO the FPGA, Receiving (RX) FROM the FPGA >"
Changed lines of the file:
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@@
 		)
 	)
-	(text "Transmiting (TX) TO the FPGA,\nReceiving (RX) FROM the FPGA > "
+	(text "Transmiting (TX) FROM the FPGA TO the host\nReceiving (RX) FROM the host TO the FPGA > "
 		(exclude_from_sim no)
-		(at 59.69 98.552 0)
+		(at 46.228 100.584 0)
 		(effects
 			(font
@@
 		(dnp no)
 		(property "Reference" "C12"
-			(at 135.382 148.59 90)
+			(at 135.636 148.59 90)
 			(effects
 				(font
@@
 		(dnp no)
 		(property "Reference" "C11"
-			(at 129.032 146.05 90)
-			(effects
-				(font
+			(at 129.286 146.05 90)
+			(effects
+				(font

Commit message: added some configuration features and cleaned it up
Other:
- note added: "< Dampening for inrush for each group"
Changed lines of the file:
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@@
+		)
+	)
+	(text "< Dampening for inrush for each group"
+		(exclude_from_sim no)
+		(at 211.582 44.958 0)
+		(effects
+			(font
+				(size 1.27 1.27)
+			)
 		)
 	)
