File: PCB/ddr3.kicad_sch (KiCad schematic)
At the start: 33 parts, among them U11 MT41J128M16JT-125:K

Commit message: cleaning up DDR3 even more, finishing it's journaling
Parts:
- added C13: 10n, symbol Device:C
Connections:
- net GND: now also C13.2
- net at C110.1, C57.2, C58.1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: now also C13.1
Other:
- note added: "Decoupling as CLOSE AS POSSIBLE to VREF!"
- moved on the sheet: C110, C57, C58, C86, R17, R18

Commit message: cleaning up the schematic even more, it looks sick now
Changed lines of the file:
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@@
 		(members "DDR_A[0..14]" "DDR_BA[0..2]")
 	)
-	(bus_alias "DDR_CLOCK"
+	(bus_alias "DDR_CLK"
 		(members "DDR_CLK+" "DDR_CLK-")
 	)
@@
 		)
 	)
-	(hierarchical_label "{DDR_CLOCK}"
+	(hierarchical_label "{DDR_CLK}"
 		(shape input)
 		(at 55.88 92.71 180)
