File: PCB/PCIe GTP Transceivers.kicad_sch (KiCad schematic)
At the start: 1 part, among them U1 XC7A50T-FGG484

Commit message: cleaning the schematic up
Parts:
- removed U1: XC7A50T-FGG484, Package_BGA:Xilinx_FGG484, symbol FPGA Accelerator:XC7A50T-FGG484
- added U1: XC7A50T-FGG484, Package_BGA:Xilinx_FGG484, symbol FPGA Accelerator:XC7A50T-FGG484

Commit message: some more PCIe wiring - clk
Parts:
- added C11, C12: 100n, symbol Device:C_Small
Connections:
- net at U1.E6 (MGTREFCLK0N_216): now also C12.2
- net at U1.F6 (MGTREFCLK0P_216): now also C11.2
- no-connect marks 0 -> 2
Other:
- note added: "Close to FPGA, not edge connector >"
Changed lines of the file:
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@@
 	(generator_version "9.0")
 	(paper "A3")
+	(text "Close to FPGA, not edge connector >"
+		(exclude_from_sim no)
+		(at 130.302 160.02 0)
+		(effects
+			(font
+				(size 1.27 1.27)
+			)
+		)
+	)
+	(no_connect
+		(at 171.45 163.83)
+	)
+	(no_connect
+		(at 171.45 166.37)
+	)
+	(wire
+		(pts
+			(xy 162.56 158.75) (xy 171.45 158.75)
+		)
+		(stroke
+			(width 0)
+			(type default)
+		)
+	)
+	(wire
+		(pts
+			(xy 168.91 161.29) (xy 171.45 161.29)
+		)
+		(stroke
+			(width 0)
+			(type default)
+		)
+	)
+	(wire
+		(pts
+			(xy 152.4 158.75) (xy 157.48 158.75)
+		)
+		(stroke
+			(width 0)
+			(type default)
+		)
+	)
+	(wire
+		(pts
+			(xy 152.4 161.29) (xy 163.83 161.29)
+		)
+		(stroke
+			(width 0)
+			(type default)
+		)
+	)
 	(symbol
 		(lib_id "FPGA Accelerator:XC7A50T-FGG484")
@@
 				)
 			)
+		)
+	)
+	(symbol
+		(lib_id "Device:C_Small")
+		(at 166.37 161.29 90)
+		(unit 1)
+		(exclude_from_sim no)
+		(in_bom yes)
+		(on_board yes)
+		(dnp no)
+		(property "Reference" "C12"
+			(at 168.402 160.02 90)
+			(effects
+				(font
+					(size 1.016 1.016)
+				)
+			)
+		)
+		(property "Value" "100n"
+			(at 163.322 160.02 90)
+			(effects
+				(font
+					(size 1.016 1.016)
+				)
+			)
+		)
+		(property "Footprint" ""
+			(at 166.37 161.29 0)
+			(effects
+				(font
+					(size 1.27 1.27)
+				)
+				(hide yes)
+			)
+		)
+		(property "Datasheet" "~"
+			(at 166.37 161.29 0)
+			(effects
+				(font
+					(size 1.27 1.27)
+				)
+				(hide yes)
+			)
+		)
+		(property "Description" "Unpolarized capacitor, small symbol"
+			(at 166.37 161.29 0)
+			(effects
+				(font
+					(size 1.27 1.27)
+				)
+				(hide yes)
+			)
+		)
+		(pin "2"
+		)
+		(pin "1"
+		)
+		(instances
+			(project "PCB"
+				(path "/ed0095eb-57a0-4856-9ac4-7b40bd214a3a/afe9695b-690d-4189-aece-4d8f452c930a"
+					(reference "C12")
+					(unit 1)
+				)
+			)
+		)
+	)
+	(symbol
+		(lib_id "Device:C_Small")
+		(at 160.02 158.75 90)
+		(unit 1)
+		(exclude_from_sim no)
+		(in_bom yes)
+		(on_board yes)
+		(dnp no)
+		(property "Reference" "C11"
+			(at 162.56 157.48 90)
+			(effects
+				(font
+					(size 1.016 1.016)
+				)
+			)
+		)
+		(property "Value" "100n"
+			(at 156.972 157.48 90)
+			(effects
+				(font
+					(size 1.016 1.016)
+				)
+			)
+		)
+		(property "Footprint" ""
+			(at 160.02 158.75 0)
+			(effects
+				(font
+					(size 1.27 1.27)
+				)
+				(hide yes)
+			)
+		)
+		(property "Datasheet" "~"
+			(at 160.02 158.75 0)
+			(effects
+				(font
+					(size 1.27 1.27)
+				)
+				(hide yes)
+			)
+		)
+		(property "Description" "Unpolarized capacitor, small symbol"
+			(at 160.02 158.75 0)
+			(effects
+				(font
+					(size 1.27 1.27)
+				)
+				(hide yes)
+			)
+		)
+		(pin "2"
+		)
+		(pin "1"
+		)
+		(instances
+			(project "PCB"
+				(path "/ed0095eb-57a0-4856-9ac4-7b40bd214a3a/afe9695b-690d-4189-aece-4d8f452c930a"
+					(reference "C11")
+					(unit 1)
+				)
+			)

Commit message: finished wiring the m.2 connector
Connections:
- net PCIe_REFCLK-: now reaches C12.1
- net PCIe_REFCLK+: now reaches C11.1
Changed lines of the file:
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@@
 	(text "Close to FPGA, not edge connector >"
 		(exclude_from_sim no)
-		(at 130.302 160.02 0)
+		(at 112.522 157.48 0)
 		(effects
 			(font
@@
 		(at 171.45 166.37)
 	)
+	(bus_entry
+		(at 134.62 158.75)
+		(size 2.54 2.54)
+		(stroke
+			(width 0)
+			(type default)
+		)
+	)
+	(bus_entry
+		(at 134.62 156.21)
+		(size 2.54 2.54)
+		(stroke
+			(width 0)
+			(type default)
+		)
+	)
 	(wire
 		(pts
 			(xy 162.56 158.75) (xy 171.45 158.75)
+		)
+		(stroke
+			(width 0)
+			(type default)
+		)
+	)
+	(wire
+		(pts
+			(xy 137.16 161.29) (xy 163.83 161.29)
+		)
+		(stroke
+			(width 0)
+			(type default)
+		)
+	)
+	(bus
+		(pts
+			(xy 134.62 151.13) (xy 134.62 156.21)
 		)
 		(stroke
@@
 	(wire
 		(pts
-			(xy 152.4 158.75) (xy 157.48 158.75)
+			(xy 137.16 158.75) (xy 157.48 158.75)
 		)
 		(stroke
@@
 		)
 	)
-	(wire
+	(bus
 		(pts
-			(xy 152.4 161.29) (xy 163.83 161.29)
+			(xy 134.62 156.21) (xy 134.62 158.75)
 		)
 		(stroke
@@
 		)
 	)
+	(bus
+		(pts
+			(xy 129.54 151.13) (xy 134.62 151.13)
+		)
+		(stroke
+			(width 0)
+			(type default)
+		)
+	)
+	(label "PCIe_REFCLK+"
+		(at 138.43 158.75 0)
+		(effects
+			(font
+				(size 1.27 1.27)
+			)
+			(justify left bottom)
+		)
+	)
+	(label "PCIe_REFCLK-"
+		(at 138.43 161.29 0)
+		(effects
+			(font
+				(size 1.27 1.27)
+			)
+			(justify left bottom)
+		)
+	)
+	(hierarchical_label "{PCIe_CLK}"
+		(shape input)
+		(at 129.54 151.13 180)
+		(effects
+			(font
+				(size 1.27 1.27)
+			)
+			(justify right)
+		)
+	)

Commit message: dampening and cleaning up the schematic
Parts:
- removed C11, C12: 100n, symbol Device:C_Small
Connections:
- net PCIe_REFCLK+: now also U1.F6 (MGTREFCLK0P_216)
- net PCIe_REFCLK-: now also U1.E6 (MGTREFCLK0N_216)
Other:
- note removed: "Close to FPGA, not edge connector >"
Changed lines of the file:
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@@
 	(generator_version "9.0")
 	(paper "A3")
-	(text "Close to FPGA, not edge connector >"
-		(exclude_from_sim no)
-		(at 112.522 157.48 0)
-		(effects
-			(font
-				(size 1.27 1.27)
-			)
-		)
-	)
 	(no_connect
 		(at 171.45 163.83)
@@
 	)
 	(bus_entry
-		(at 134.62 158.75)
+		(at 149.86 158.75)
 		(size 2.54 2.54)
 		(stroke
@@
 	)
 	(bus_entry
-		(at 134.62 156.21)
+		(at 149.86 156.21)
 		(size 2.54 2.54)
 		(stroke
@@
 	(wire
 		(pts
-			(xy 162.56 158.75) (xy 171.45 158.75)
+			(xy 152.4 161.29) (xy 171.45 161.29)
 		)
 		(stroke
@@
 		)
 	)
-	(wire
+	(bus
 		(pts
-			(xy 137.16 161.29) (xy 163.83 161.29)
+			(xy 149.86 151.13) (xy 149.86 156.21)
 		)
 		(stroke
@@
 		)
 	)
-	(bus
+	(wire
 		(pts
-			(xy 134.62 151.13) (xy 134.62 156.21)
+			(xy 152.4 158.75) (xy 171.45 158.75)
 		)
 		(stroke
@@
 		)
 	)
-	(wire
+	(bus
 		(pts
-			(xy 168.91 161.29) (xy 171.45 161.29)
+			(xy 149.86 156.21) (xy 149.86 158.75)
 		)
 		(stroke
@@
 		)
 	)
-	(wire
+	(bus
 		(pts
-			(xy 137.16 158.75) (xy 157.48 158.75)
+			(xy 144.78 151.13) (xy 149.86 151.13)
 		)
 		(stroke
@@
 		)
 	)
-	(bus
-		(pts
-			(xy 134.62 156.21) (xy 134.62 158.75)
-		)
-		(stroke
-			(width 0)
-			(type default)
-		)
-	)
-	(bus
-		(pts
-			(xy 129.54 151.13) (xy 134.62 151.13)
-		)
-		(stroke
-			(width 0)
-			(type default)
-		)
-	)
 	(label "PCIe_REFCLK+"
-		(at 138.43 158.75 0)
+		(at 153.67 158.75 0)
 		(effects
 			(font
@@
 	)
 	(label "PCIe_REFCLK-"
-		(at 138.43 161.29 0)
+		(at 153.67 161.29 0)
 		(effects
 			(font
@@
 	(hierarchical_label "{PCIe_CLK}"
 		(shape input)
-		(at 129.54 151.13 180)
+		(at 144.78 151.13 180)
 		(effects
 			(font
@@
 				)
 			)
-		)
-	)
-	(symbol
-		(lib_id "Device:C_Small")
-		(at 166.37 161.29 90)
-		(unit 1)
-		(exclude_from_sim no)
-		(in_bom yes)
-		(on_board yes)
-		(dnp no)
-		(property "Reference" "C12"
-			(at 168.402 160.02 90)
-			(effects
-				(font
-					(size 1.016 1.016)
-				)
-			)
-		)
-		(property "Value" "100n"
-			(at 163.322 160.02 90)
-			(effects
-				(font
-					(size 1.016 1.016)
-				)
-			)
-		)
-		(property "Footprint" ""
-			(at 166.37 161.29 0)
-			(effects
-				(font
-					(size 1.27 1.27)
-				)
-				(hide yes)
-			)
-		)
-		(property "Datasheet" "~"
-			(at 166.37 161.29 0)
-			(effects
-				(font
-					(size 1.27 1.27)
-				)
-				(hide yes)
-			)
-		)
-		(property "Description" "Unpolarized capacitor, small symbol"
-			(at 166.37 161.29 0)
-			(effects
-				(font
-					(size 1.27 1.27)
-				)
-				(hide yes)
-			)
-		)
-		(pin "2"
-		)
-		(pin "1"
-		)
-		(instances
-			(project "PCB"
-				(path "/ed0095eb-57a0-4856-9ac4-7b40bd214a3a/afe9695b-690d-4189-aece-4d8f452c930a"
-					(reference "C12")
-					(unit 1)
-				)
-			)
-		)
-	)
-	(symbol
-		(lib_id "Device:C_Small")
-		(at 160.02 158.75 90)
-		(unit 1)
-		(exclude_from_sim no)
-		(in_bom yes)
-		(on_board yes)
-		(dnp no)
-		(property "Reference" "C11"
-			(at 162.56 157.48 90)
-			(effects
-				(font
-					(size 1.016 1.016)
-				)
-			)
-		)
-		(property "Value" "100n"
-			(at 156.972 157.48 90)
-			(effects
-				(font
-					(size 1.016 1.016)
-				)
-			)
-		)
-		(property "Footprint" ""
-			(at 160.02 158.75 0)
-			(effects
-				(font
-					(size 1.27 1.27)
-				)
-				(hide yes)
-			)
-		)
-		(property "Datasheet" "~"
-			(at 160.02 158.75 0)
-			(effects
-				(font
-					(size 1.27 1.27)
-				)
-				(hide yes)
-			)
-		)
-		(property "Description" "Unpolarized capacitor, small symbol"
-			(at 160.02 158.75 0)
-			(effects
-				(font
-					(size 1.27 1.27)
-				)
-				(hide yes)
-			)
-		)
-		(pin "2"
-		)
-		(pin "1"
-		)
-		(instances
-			(project "PCB"
-				(path "/ed0095eb-57a0-4856-9ac4-7b40bd214a3a/afe9695b-690d-4189-aece-4d8f452c930a"
-					(reference "C11")
-					(unit 1)
-				)
-			)

Commit message: wiring the m.2 connector to the MGT transceivers
Connections:
- net PCIe_RX2-: now reaches U1.A10 (MGTPRXN2_216)
- net PCIe_TX0-: now reaches U1.A4 (MGTPTXN0_216)
- net PCIe_TX2-: now reaches U1.A6 (MGTPTXN2_216)
- net PCIe_RX0-: now reaches U1.A8 (MGTPRXN0_216)
- net PCIe_RX2+: now reaches U1.B10 (MGTPRXP2_216)
- net PCIe_TX0+: now reaches U1.B4 (MGTPTXP0_216)
- net PCIe_TX2+: now reaches U1.B6 (MGTPTXP2_216)
- net PCIe_RX0+: now reaches U1.B8 (MGTPRXP0_216)
- net PCIe_RX1-: now reaches U1.C11 (MGTPRXN1_216)
- net PCIe_TX1-: now reaches U1.C5 (MGTPTXN1_216)
- net PCIe_TX3-: now reaches U1.C7 (MGTPTXN3_216)
- net PCIe_RX3-: now reaches U1.C9 (MGTPRXN3_216)
- net PCIe_RX1+: now reaches U1.D11 (MGTPRXP1_216)
- net PCIe_TX1+: now reaches U1.D5 (MGTPTXP1_216)
- net PCIe_TX3+: now reaches U1.D7 (MGTPTXP3_216)
- net PCIe_RX3+: now reaches U1.D9 (MGTPRXP3_216)

Commit message: added some configuration features and cleaned it up
Other:
- note added: "Double check clock pins >"
Changed lines of the file:
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@@
 	(generator_version "9.0")
 	(paper "A3")
+	(text "Double check clock pins >"
+		(exclude_from_sim no)
+		(at 131.318 159.004 0)
+		(effects
+			(font
+				(size 1.27 1.27)
+			)
+		)
+	)
 	(no_connect
 		(at 171.45 163.83)

Commit message: cleaning up the schematic even more, starting on HDMI
Other:
- moved on the sheet: U1D
