File: PCB/hdmi.kicad_sch (KiCad schematic)
At the start: 0 parts

Commit message: cleaning up the schematic even more, starting on HDMI
Parts:
- added J3: HDMI_A, symbol Connector:HDMI_A
Changed lines of the file:
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@@
 	(generator "eeschema")
 	(generator_version "9.0")
-	(paper "A3")
+	(paper "A4")
+	(symbol
+		(lib_id "Connector:HDMI_A")
+		(at 167.64 97.79 0)
+		(unit 1)
+		(exclude_from_sim no)
+		(in_bom yes)
+		(on_board yes)
+		(dnp no)
+		(fields_autoplaced yes)
+		(property "Reference" "J3"
+			(at 179.07 96.5199 0)
+			(effects
+				(font
+					(size 1.27 1.27)
+				)
+				(justify left)
+			)
+		)
+		(property "Value" "HDMI_A"
+			(at 179.07 99.0599 0)
+			(effects
+				(font
+					(size 1.27 1.27)
+				)
+				(justify left)
+			)
+		)
+		(property "Footprint" ""
+			(at 168.275 97.79 0)
+			(effects
+				(font
+					(size 1.27 1.27)
+				)
+				(hide yes)
+			)
+		)
+		(property "Datasheet" "https://en.wikipedia.org/wiki/HDMI"
+			(at 168.275 97.79 0)
+			(effects
+				(font
+					(size 1.27 1.27)
+				)
+				(hide yes)
+			)
+		)
+		(property "Description" "HDMI type A connector"
+			(at 167.64 97.79 0)
+			(effects
+				(font
+					(size 1.27 1.27)
+				)
+				(hide yes)
+			)
+		)
+		(pin "8"
+		)
+		(pin "18"
+		)
+		(pin "15"
+		)
+		(pin "13"
+		)
+		(pin "11"
+		)
+		(pin "17"
+		)
+		(pin "5"
+		)
+		(pin "16"
+		)
+		(pin "12"
+		)
+		(pin "14"
+		)
+		(pin "SH"
+		)
+		(pin "1"
+		)
+		(pin "10"
+		)
+		(pin "9"
+		)
+		(pin "7"
+		)
+		(pin "6"
+		)
+		(pin "4"
+		)
+		(pin "3"
+		)
+		(pin "2"
+		)
+		(pin "19"
+		)
+		(instances
+			(project ""
+				(path "/ed0095eb-57a0-4856-9ac4-7b40bd214a3a/e0bb63a6-1743-4d45-83e3-83dd5e1cd35c"
+					(reference "J3")
+					(unit 1)
+				)
+			)
+		)
+	)
 )

Commit message: basic HDMI wiring
Parts:
- removed J3: HDMI_A, symbol Connector:HDMI_A
- added C113, C114, C115, C116, C117, C119, C14, C16: 100n, symbol Device:C_Small
- added J3: HDMI_A, symbol FPGA Accelerator:HDMI_A
- added R47, R57: 4k7, symbol Device:R
Connections:
- new net: C117.2, J3.3 (D2-)
- new net: C116.2, J3.4 (D1+)
- new net: C114.2, J3.7 (D0+)
- new net: C119.2, J3.1 (D2+)
- new net: C16.2, J3.10 (CK+)
- new net: C14.2, J3.12 (CK-)
- new net: J3.15 (SCL), R57.2
- new net: J3.16 (SDA), R47.2
- new net: C115.2, J3.6 (D1-)
- new net: C113.2, J3.9 (D0-)
- new net +5V: R47.1, R57.1
- new net GND: J3.11 (CKS), J3.17 (GND), J3.2 (D2S), J3.5 (D1S), J3.8 (D0S), J3.SH

Commit message: more HDMI wiring
Parts:
- added C120: 100n, symbol Device:C
- added D2: D_Schottky, symbol Device:D_Schottky
Connections:
- net GND: now also C120.2
- net HDMI_D2-: now reaches C117.1
- net HDMI_D1+: now reaches C116.1
- net HDMI_D0+: now reaches C114.1
- net HDMI_CEC: now reaches J3.13 (CEC)
- net HDMI_UTIL: now reaches J3.14 (UTILITY)
- net HDMI_SCL: now reaches J3.15 (SCL), R57.2
- net HDMI_SDA: now reaches J3.16 (SDA), R47.2
- net at J3.18 (+5V): now also C120.1, D2.1 (K)
- net HDMI_HPD: now reaches J3.19 (HPD)
- net HDMI_D2+: now reaches C119.1
- net HDMI_D1-: now reaches C115.1
- net HDMI_D0-: now reaches C113.1
- net HDMI_CLK-: now reaches C14.1
- net HDMI_CLK+: now reaches C16.1
Other:
- note added: "ADD SCHOTTKY PART AND CEC MOSFET No 5V either...."

Commit message: almost done wiring HDMI
Parts:
- added C121: 1u, symbol Device:C
- R47: value 4k7 -> 30k
- R57: value 4k7 -> 1k
Connections:
- net GND: now also C121.2
- net HDMI_CEC: now also R47.2
- net HDMI_HPD: now also R57.1; no longer J3.19 (HPD)
- net HDMI_SCL: no longer R57.2
- net HDMI_SDA: no longer R47.2
- net at C120.1, D2.1 (K), J3.18 (+5V): now also C121.1
- net +VBUS: now reaches D2.2 (A)
- net +5V renamed +3V3
- net +3V3: no longer R57.1
- net HDMI_UTIL: no longer names the net of J3.14 (UTILITY)
- new net: J3.19 (HPD), R57.2
- no-connect marks 0 -> 1
Other:
- note added: "Current limit HPD for safe 5V I/O >"
- moved on the sheet: C113, C114, C115, C116, C117, C119, C120, C14, C16, D2, J3

Commit message: added th e level shifter for HDMI DCC
Parts:
- added C122, C123: 100n, symbol Device:C
- added R58: 100k, symbol Device:R
- added R59, R60, R61, R62: 4k7, symbol Device:R
- added U12: PCA9306DC1, Package_SO:VSSOP-8_2.3x2mm_P0.5mm, symbol Interface:PCA9306DC1
Connections:
- net +3V3: now also C123.1, R61.1, R62.1, U12.2 (VREF1)
- net +VBUS: now also R58.1, R59.1, R60.1
- net GND: now also C122.2, C123.2, U12.1 (GND)
- net HDMI_SCL: now also R61.2, U12.3 (SCL1); no longer J3.15 (SCL)
- net HDMI_SDA: now also R62.2, U12.4 (SDA1); no longer J3.16 (SDA)
- new net: C122.1, R58.2, U12.7 (VREF2), U12.8 (EN)
- new net HDMI_SCL_5V: J3.15 (SCL), R60.2, U12.6 (SCL2)
- new net HDMI_SDA_5V: J3.16 (SDA), R59.2, U12.5 (SDA2)
Other:
- note added: "Add SCHOTTKY and HDMI part"
- note added: "Current limit resistor!"
- note removed: "ADD SCHOTTKY PART AND CEC MOSFET No 5V either...."
- moved on the sheet: C113, C114, C115, C116, C117, C119, C120, C121, C14, C16, D2, J3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

Commit message: added all the HDMI parts in, done now!
Parts:
- removed D2: D_Schottky, symbol Device:D_Schottky
- added D3: 1N5819WS, Diode_SMD:D_SOD-323, symbol Diode:1N5819WS
- J3: value HDMI_A -> HDMI-019S; LCSC (none) -> C111617; MPN (none) -> HDMI-019S
Connections:
- net +VBUS: now also D3.2 (A)
- net at C120.1, C121.1, J3.18 (+5V): now also D3.1 (K)
Changed lines of the file:
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@@
 			)
 		)
-		(property "Value" "HDMI_A"
+		(property "Value" "HDMI-019S"
 			(at 119.38 106.6799 0)
 			(effects
@@
 		)
 		(property "Description" "HDMI type A connector"
+			(at 107.95 105.41 0)
+			(effects
+				(font
+					(size 1.27 1.27)
+				)
+				(hide yes)
+			)
+		)
+		(property "MPN" "HDMI-019S"
+			(at 107.95 105.41 0)
+			(effects
+				(font
+					(size 1.27 1.27)
+				)
+				(hide yes)
+			)
+		)
+		(property "LCSC" "C111617"
 			(at 107.95 105.41 0)
 			(effects
@@
 	)
 	(symbol
-		(lib_id "Device:D_Schottky")
-		(at 107.95 44.45 90)
-		(unit 1)
-		(exclude_from_sim no)
-		(in_bom yes)
-		(on_board yes)
-		(dnp no)
-		(fields_autoplaced yes)
-		(property "Reference" "D2"
-			(at 110.49 43.4974 90)
-			(effects
-				(font
-					(size 1.27 1.27)
-				)
-				(justify right)
-			)
-		)
-		(property "Value" "D_Schottky"
-			(at 110.49 46.0374 90)
-			(effects
-				(font
-					(size 1.27 1.27)
-				)
-				(justify right)
-			)
-		)
-		(property "Footprint" ""
-			(at 107.95 44.45 0)
-			(effects
-				(font
-					(size 1.27 1.27)
-				)
-				(hide yes)
-			)
-		)
-		(property "Datasheet" "~"
-			(at 107.95 44.45 0)
-			(effects
-				(font
-					(size 1.27 1.27)
-				)
-				(hide yes)
-			)
-		)
-		(property "Description" "Schottky diode"
-			(at 107.95 44.45 0)
-			(effects
-				(font
-					(size 1.27 1.27)
-				)
-				(hide yes)
-			)
-		)
-		(pin "1"
-		)
-		(pin "2"
-		)
-		(instances
-			(project ""
-				(path "/ed0095eb-57a0-4856-9ac4-7b40bd214a3a/e0bb63a6-1743-4d45-83e3-83dd5e1cd35c"
-					(reference "D2")
-					(unit 1)
-				)
-			)
-		)
-	)
-	(symbol
 		(lib_id "Device:R")
 		(at 229.87 96.52 270)
@@
 					(unit 1)
 				)
+			)
+		)
+	)
+	(symbol
+		(lib_id "Diode:1N5819WS")
+		(at 107.95 44.45 90)
+		(unit 1)
+		(exclude_from_sim no)
+		(in_bom yes)
+		(on_board yes)
+		(dnp no)
+		(fields_autoplaced yes)
+		(property "Reference" "D3"
+			(at 110.49 43.4974 90)
+			(effects
+				(font
+					(size 1.27 1.27)
+				)
+				(justify right)
+			)
+		)
+		(property "Value" "1N5819WS"
+			(at 110.49 46.0374 90)
+			(effects
+				(font
+					(size 1.27 1.27)
+				)
+				(justify right)
+			)
+		)
+		(property "Footprint" "Diode_SMD:D_SOD-323"
+			(at 112.395 44.45 0)
+			(effects
+				(font
+					(size 1.27 1.27)
+				)
+				(hide yes)
+			)
+		)
+		(property "Datasheet" "https://datasheet.lcsc.com/lcsc/2204281430_Guangdong-Hottech-1N5819WS_C191023.pdf"
+			(at 107.95 44.45 0)
+			(effects
+				(font
+					(size 1.27 1.27)
+				)
+				(hide yes)
+			)
+		)
+		(property "Description" "40V 600mV@1A 1A SOD-323 Schottky Barrier Diodes, SOD-323"
+			(at 107.95 44.45 0)
+			(effects
+				(font
+					(size 1.27 1.27)
+				)
+				(hide yes)
+			)
+		)
+		(property "MPN" "1N5819WS"
+			(at 107.95 44.45 90)
+			(effects
+				(font
+					(size 1.27 1.27)
+				)
+				(hide yes)
+			)
+		)
+		(property "LSCS" "C191023"
+			(at 107.95 44.45 90)
+			(effects
+				(font
+					(size 1.27 1.27)
+				)
+				(hide yes)
+			)
+		)
+		(pin "1"
+		)
+		(pin "2"
+		)
+		(instances
+			(project ""
+				(path "/ed0095eb-57a0-4856-9ac4-7b40bd214a3a/e0bb63a6-1743-4d45-83e3-83dd5e1cd35c"
+					(reference "D3")
+					(unit 1)
+				)

Commit message: crystal/LAN MPN's and starting to wire ethernet
Other:
- note removed: "Add SCHOTTKY and HDMI part"
Changed lines of the file:
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@@
-		)
-	)
-	(text "Add SCHOTTKY and HDMI part"
-		(exclude_from_sim no)
-		(at 172.466 69.85 0)
-		(effects
-			(font
-				(size 1.27 1.27)
-			)
 		)
 	)
