File: PCB/hdmi.kicad_sch (KiCad schematic)
At the start: 22 parts, among them J3 HDMI-019S, U12 PCA9306DC1

Commit message: some more ethernet wiring
Other:
- note added: "DOUBLE CHECK AC CAPS, ESD PROTECTION"
- moved on the sheet: C122, C123, R58, R59, R60, R61, R62, U12

Commit message: basic HDMI ESD protection I think
Parts:
- added U14, U15, U16: ESD224DQAR-TP, Package_DFN_QFN:Diodes_UDFN-10_1.0x2.5mm_P0.5mm, symbol Power_Protection:ESD224DQA
Connections:
- net GND: now also U14.3 (VSS), U14.8 (VSS), U15.3 (VSS), U15.8 (VSS), U16.3 (VSS), U16.8 (VSS)
- net HDMI_CEC: now also U16.1, U16.10
- net HDMI_CLK+: now also U15.4, U15.7
- net HDMI_CLK-: now also U15.5, U15.6
- net HDMI_D0+: now also U15.1, U15.10
- net HDMI_D0-: now also U15.2, U15.9
- net HDMI_D1+: now also U14.4, U14.7
- net HDMI_D1-: now also U14.5, U14.6
- net HDMI_D2+: now also U14.1, U14.10
- net HDMI_D2-: now also U14.2, U14.9
- net HDMI_HPD: now also U16.2, U16.9
- net HDMI_SCL: now also U16.4, U16.7
- net HDMI_SDA: now also U16.5, U16.6
Other:
- note added: "5V vs 3.6V?"
- note removed: "DOUBLE CHECK AC CAPS, ESD PROTECTION"
- moved on the sheet: C113, C114, C115, C116, C117, C119, C120, C121, C122, C123, C14, C16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

Commit message: finished HDMI ESD protection, took longer than I would have liked
Parts:
- removed U14, U15, U16: ESD224DQAR-TP, Package_DFN_QFN:Diodes_UDFN-10_1.0x2.5mm_P0.5mm, symbol Power_Protection:ESD224DQA
- added U14, U15, U16: UCL0524P, Package_DFN_QFN:Diodes_UDFN-10_1.0x2.5mm_P0.5mm, symbol kai-library:UCL0524P
Connections:
- net GND: now also U14.3, U14.8, U15.3, U15.8, U16.3, U16.8
- net HDMI_CEC: now also U14.4, U14.7
- net HDMI_SCL_5V: now also U14.1, U14.10
- net HDMI_SDA_5V: now also U14.2, U14.9
- net at J3.19 (HPD), R57.2: now also U14.5, U14.6
- net at C117.2, J3.3 (D2-): now also U15.2, U15.9
- net at C116.2, J3.4 (D1+): now also U15.4, U15.7
- net at C114.2, J3.7 (D0+): now also U16.1, U16.10
- net at C119.2, J3.1 (D2+): now also U15.1, U15.10
- net at C16.2, J3.10 (CK+): now also U16.4, U16.7
- net at C14.2, J3.12 (CK-): now also U16.5, U16.6
- net at C115.2, J3.6 (D1-): now also U15.5, U15.6
- net at C113.2, J3.9 (D0-): now also U16.2, U16.9
Other:
- note removed: "5V vs 3.6V?"
- moved on the sheet: C113, C114, C115, C116, C117, C119, C14, C16, J3, R47, R57

Commit message: cleaned up the schematic after that mess, looking beautiful :D
Other:
- note removed: "Current limit HPD for safe 5V I/O >"
- moved on the sheet: C113, C114, C115, C116, C117, C119, C120, C121, C122, C123, C14, C16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

Commit message: wired the 100MHz clock for PLL's
Changed lines of the file:
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@@
 	)
 	(junction
+		(at 106.68 128.27)
+		(diameter 0)
+		(color 0 0 0 0)
+	)
+	(junction
 		(at 104.14 118.11)
 		(diameter 0)
@@
 	)
 	(junction
-		(at 105.41 128.27)
+		(at 104.14 87.63)
 		(diameter 0)
 		(color 0 0 0 0)
 	)
 	(junction
-		(at 104.14 87.63)
+		(at 130.81 144.78)
 		(diameter 0)
 		(color 0 0 0 0)
 	)
 	(junction
-		(at 130.81 144.78)
+		(at 104.14 125.73)
 		(diameter 0)
 		(color 0 0 0 0)
 	)
 	(junction
-		(at 104.14 125.73)
+		(at 86.36 113.03)
 		(diameter 0)
 		(color 0 0 0 0)
@@
 	)
 	(junction
-		(at 87.63 113.03)
-		(diameter 0)
-		(color 0 0 0 0)
-	)
-	(junction
 		(at 88.9 130.81)
 		(diameter 0)
@@
 	)
 	(junction
-		(at 87.63 128.27)
+		(at 88.9 95.25)
 		(diameter 0)
 		(color 0 0 0 0)
 	)
 	(junction
-		(at 88.9 95.25)
+		(at 88.9 110.49)
 		(diameter 0)
 		(color 0 0 0 0)
 	)
 	(junction
-		(at 88.9 110.49)
+		(at 106.68 113.03)
 		(diameter 0)
 		(color 0 0 0 0)
@@
 	)
 	(junction
-		(at 105.41 113.03)
+		(at 88.9 115.57)
 		(diameter 0)
 		(color 0 0 0 0)
 	)
 	(junction
-		(at 88.9 115.57)
+		(at 104.14 90.17)
 		(diameter 0)
 		(color 0 0 0 0)
 	)
 	(junction
-		(at 104.14 90.17)
+		(at 86.36 128.27)
 		(diameter 0)
 		(color 0 0 0 0)
@@
 	(wire
 		(pts
-			(xy 87.63 128.27) (xy 87.63 142.24)
+			(xy 86.36 128.27) (xy 86.36 142.24)
 		)
 		(stroke
@@
 	(wire
 		(pts
-			(xy 105.41 128.27) (xy 105.41 142.24)
+			(xy 106.68 128.27) (xy 106.68 142.24)
 		)
 		(stroke
@@
 	(wire
 		(pts
-			(xy 87.63 92.71) (xy 87.63 113.03)
+			(xy 86.36 92.71) (xy 86.36 113.03)
 		)
 		(stroke
@@
 	(wire
 		(pts
+			(xy 86.36 128.27) (xy 88.9 128.27)
+		)
+		(stroke
+			(width 0)
+			(type default)
+		)
+	)
+	(wire
+		(pts
 			(xy 88.9 125.73) (xy 104.14 125.73)
 		)
@@
 	(wire
 		(pts
-			(xy 104.14 92.71) (xy 105.41 92.71)
+			(xy 104.14 92.71) (xy 106.68 92.71)
 		)
 		(stroke
@@
 	(wire
 		(pts
-			(xy 87.63 113.03) (xy 88.9 113.03)
-		)
-		(stroke
-			(width 0)
-			(type default)
-		)
-	)
-	(wire
-		(pts
 			(xy 104.14 130.81) (xy 115.57 130.81)
 		)
@@
 	(wire
 		(pts
-			(xy 87.63 113.03) (xy 87.63 128.27)
+			(xy 86.36 113.03) (xy 86.36 128.27)
 		)
 		(stroke
@@
 	(wire
 		(pts
-			(xy 105.41 92.71) (xy 105.41 113.03)
+			(xy 106.68 92.71) (xy 106.68 113.03)
 		)
 		(stroke
@@
 	(wire
 		(pts
-			(xy 105.41 113.03) (xy 105.41 128.27)
+			(xy 106.68 113.03) (xy 106.68 128.27)
 		)
 		(stroke
@@
 	(wire
 		(pts
-			(xy 88.9 92.71) (xy 87.63 92.71)
+			(xy 88.9 92.71) (xy 86.36 92.71)
 		)
 		(stroke
@@
 	(wire
 		(pts
+			(xy 86.36 113.03) (xy 88.9 113.03)
+		)
+		(stroke
+			(width 0)
+			(type default)
+		)
+	)
+	(wire
+		(pts
 			(xy 38.1 133.35) (xy 71.12 133.35)
 		)
@@
 	(wire
 		(pts
-			(xy 104.14 128.27) (xy 105.41 128.27)
+			(xy 104.14 128.27) (xy 106.68 128.27)
 		)
 		(stroke
@@
 	(wire
 		(pts
-			(xy 87.63 128.27) (xy 88.9 128.27)
-		)
-		(stroke
-			(width 0)
-			(type default)
-		)
-	)
-	(wire
-		(pts
 			(xy 138.43 60.96) (xy 138.43 72.39)
 		)
@@
 	(wire
 		(pts
-			(xy 104.14 113.03) (xy 105.41 113.03)
+			(xy 104.14 113.03) (xy 106.68 113.03)
 		)
 		(stroke
@@
 	(symbol
 		(lib_id "power:GND")
-		(at 87.63 142.24 0)
+		(at 86.36 142.24 0)
 		(unit 1)
 		(exclude_from_sim no)
@@
 		(fields_autoplaced yes)
 		(property "Reference" "#PWR0144"
-			(at 87.63 148.59 0)
+			(at 86.36 148.59 0)
 			(effects
 				(font
@@
 		)
 		(property "Value" "GND"
-			(at 87.63 147.32 0)
+			(at 86.36 147.32 0)
 			(effects
 				(font
@@
 		)
 		(property "Footprint" ""
-			(at 87.63 142.24 0)
+			(at 86.36 142.24 0)
 			(effects
 				(font
@@
 		)
 		(property "Datasheet" ""
-			(at 87.63 142.24 0)
+			(at 86.36 142.24 0)
 			(effects
 				(font
@@
 		)
 		(property "Description" "Power symbol creates a global label with name \"GND\" , ground"
-			(at 87.63 142.24 0)
+			(at 86.36 142.24 0)
 			(effects
 				(font
@@
 	(symbol
 		(lib_id "power:GND")
-		(at 105.41 142.24 0)
+		(at 106.68 142.24 0)
 		(unit 1)
 		(exclude_from_sim no)
@@
 		(fields_autoplaced yes)
 		(property "Reference" "#PWR0145"
-			(at 105.41 148.59 0)
+			(at 106.68 148.59 0)
 			(effects
 				(font
@@
 		)
 		(property "Value" "GND"
-			(at 105.41 147.32 0)
+			(at 106.68 147.32 0)
 			(effects
 				(font
@@
 		)
 		(property "Footprint" ""
-			(at 105.41 142.24 0)
+			(at 106.68 142.24 0)
 			(effects
 				(font
@@
 		)
 		(property "Datasheet" ""
-			(at 105.41 142.24 0)
+			(at 106.68 142.24 0)
 			(effects
 				(font
@@
 		)
 		(property "Description" "Power symbol creates a global label with name \"GND\" , ground"
-			(at 105.41 142.24 0)
+			(at 106.68 142.24 0)
 			(effects
 				(font

Commit message: cleaning  up the schematic some more before sharing
Other:
- moved on the sheet: D3

Commit message: added basic capacitor footprints
Parts:
- C113, C114, C115, C116, C117, C119, C120, C122, C123, C14, C16: footprint (none) -> Capacitor_SMD:C_0402_1005Metric
Changed lines of the file:
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@@
 			)
 		)
-		(property "Footprint" ""
+		(property "Footprint" "Capacitor_SMD:C_0402_1005Metric"
 			(at 73.66 110.49 0)
 			(effects
@@
 			)
 		)
-		(property "Footprint" ""
+		(property "Footprint" "Capacitor_SMD:C_0402_1005Metric"
 			(at 67.31 115.57 0)
 			(effects
@@
 			)
 		)
-		(property "Footprint" ""
+		(property "Footprint" "Capacitor_SMD:C_0402_1005Metric"
 			(at 67.31 123.19 0)
 			(effects
@@
 			)
 		)
-		(property "Footprint" ""
+		(property "Footprint" "Capacitor_SMD:C_0402_1005Metric"
 			(at 202.8952 105.41 0)
 			(effects
@@
 			)
 		)
-		(property "Footprint" ""
+		(property "Footprint" "Capacitor_SMD:C_0402_1005Metric"
 			(at 67.31 107.95 0)
 			(effects
@@
 			)
 		)
-		(property "Footprint" ""
+		(property "Footprint" "Capacitor_SMD:C_0402_1005Metric"
 			(at 73.66 118.11 0)
 			(effects
@@
 			)
 		)
-		(property "Footprint" ""
+		(property "Footprint" "Capacitor_SMD:C_0402_1005Metric"
 			(at 134.3152 74.93 0)
 			(effects
@@
 			)
 		)
-		(property "Footprint" ""
+		(property "Footprint" "Capacitor_SMD:C_0402_1005Metric"
 			(at 237.1852 105.41 0)
 			(effects
@@
 			)
 		)
-		(property "Footprint" ""
+		(property "Footprint" "Capacitor_SMD:C_0402_1005Metric"
 			(at 73.66 125.73 0)
 			(effects
@@
 			)
 		)
-		(property "Footprint" ""
+		(property "Footprint" "Capacitor_SMD:C_0402_1005Metric"
 			(at 73.66 133.35 0)
 			(effects
@@
 			)
 		)
-		(property "Footprint" ""
+		(property "Footprint" "Capacitor_SMD:C_0402_1005Metric"
 			(at 67.31 130.81 0)
 			(effects

Commit message: finisehed upassigning resistor footprints
Parts:
- R47: footprint (none) -> Resistor_SMD:R_0603_1608Metric
- R57, R58, R59, R60, R61, R62: footprint (none) -> Resistor_SMD:R_0402_1005Metric
Changed lines of the file:
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@@
 			)
 		)
-		(property "Footprint" ""
+		(property "Footprint" "Resistor_SMD:R_0402_1005Metric"
 			(at 189.992 104.14 90)
 			(effects
@@
 			)
 		)
-		(property "Footprint" ""
+		(property "Footprint" "Resistor_SMD:R_0402_1005Metric"
 			(at 67.31 99.568 90)
 			(effects
@@
 			)
 		)
-		(property "Footprint" ""
+		(property "Footprint" "Resistor_SMD:R_0402_1005Metric"
 			(at 249.682 104.14 90)
 			(effects
@@
 			)
 		)
-		(property "Footprint" ""
+		(property "Footprint" "Resistor_SMD:R_0402_1005Metric"
 			(at 258.572 104.14 90)
 			(effects
@@
 			)
 		)
-		(property "Footprint" ""
+		(property "Footprint" "Resistor_SMD:R_0402_1005Metric"
 			(at 181.102 104.14 90)
 			(effects
@@
 			)
 		)
-		(property "Footprint" ""
+		(property "Footprint" "Resistor_SMD:R_0402_1005Metric"
 			(at 243.84 94.742 90)
 			(effects
@@
 			)
 		)
-		(property "Footprint" ""
+		(property "Footprint" "Resistor_SMD:R_0603_1608Metric"
 			(at 56.642 78.74 90)
 			(effects
