File: PCB/hdmi.kicad_sch (KiCad schematic)
At the start: 25 parts, among them J7 HDMI_D_1.4, U12 PCA9306DC1, U14 UCL0524P, U15 UCL0524P, U16 UCL0524P

Commit message: a bunch of stuff!
Connections:
- net HDMI_CEC: no longer J7.15 (CEC), U14.7
- net HDMI_SCL_5V: no longer J7.17 (SCL), U14.10
- net HDMI_SDA_5V: no longer J7.18 (SDA), U14.9
- net at R57.2, U14.5: no longer J7.1 (HPD/HEAC-), U14.6
- net at C117.2, U15.2: no longer J7.5 (D2-), U15.9
- net at C116.2, U15.4: no longer J7.6 (D1+), U15.7
- net at C114.2, U16.1: no longer J7.9 (D0+), U16.10
- net at J7.11 (D0-), U16.9: no longer C113.2, U16.2
- net at J7.12 (CK+), U16.7: no longer C16.2, U16.4
- net at J7.14 (CK-), U16.6: no longer C14.2, U16.5
- net at J7.3 (D2+), U15.10: no longer C119.2, U15.1
- net at J7.8 (D1-), U15.6: no longer C115.2, U15.5
- new net: J7.1 (HPD/HEAC-), U14.6
- new net: J7.15 (CEC), U14.7
- new net: J7.17 (SCL), U14.10
- new net: J7.18 (SDA), U14.9
- new net: J7.5 (D2-), U15.9
- new net: J7.6 (D1+), U15.7
- new net: J7.9 (D0+), U16.10
- new net: C119.2, U15.1
- new net: C115.2, U15.5
- new net: C113.2, U16.2
- new net: C16.2, U16.4
- new net: C14.2, U16.5
Changed lines of the file:
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@@
-	)
-	(junction
-		(at 86.36 88.9)
-		(diameter 0)
-		(color 0 0 0 0)
 	)
 	(junction
@@
 	)
 	(junction
-		(at 86.36 109.22)
-		(diameter 0)
-		(color 0 0 0 0)
-	)
-	(junction
 		(at 130.81 146.05)
 		(diameter 0)
@@
 	)
 	(junction
-		(at 101.6 119.38)
-		(diameter 0)
-		(color 0 0 0 0)
-	)
-	(junction
-		(at 86.36 91.44)
-		(diameter 0)
-		(color 0 0 0 0)
-	)
-	(junction
-		(at 86.36 134.62)
-		(diameter 0)
-		(color 0 0 0 0)
-	)
-	(junction
 		(at 120.65 146.05)
 		(diameter 0)
@@
 	)
 	(junction
-		(at 101.6 124.46)
-		(diameter 0)
-		(color 0 0 0 0)
-	)
-	(junction
 		(at 251.46 96.52)
 		(diameter 0)
@@
 	)
 	(junction
-		(at 101.6 88.9)
-		(diameter 0)
-		(color 0 0 0 0)
-	)
-	(junction
 		(at 143.51 78.74)
 		(diameter 0)
@@
 	)
 	(junction
-		(at 101.6 127)
-		(diameter 0)
-		(color 0 0 0 0)
-	)
-	(junction
 		(at 83.82 114.3)
 		(diameter 0)
@@
 	)
 	(junction
-		(at 101.6 99.06)
-		(diameter 0)
-		(color 0 0 0 0)
-	)
-	(junction
-		(at 86.36 124.46)
-		(diameter 0)
-		(color 0 0 0 0)
-	)
-	(junction
-		(at 101.6 132.08)
-		(diameter 0)
-		(color 0 0 0 0)
-	)
-	(junction
-		(at 101.6 96.52)
-		(diameter 0)
-		(color 0 0 0 0)
-	)
-	(junction
-		(at 86.36 119.38)
-		(diameter 0)
-		(color 0 0 0 0)
-	)
-	(junction
-		(at 101.6 109.22)
-		(diameter 0)
-		(color 0 0 0 0)
-	)
-	(junction
-		(at 86.36 132.08)
-		(diameter 0)
-		(color 0 0 0 0)
-	)
-	(junction
 		(at 182.88 96.52)
 		(diameter 0)
@@
 	)
 	(junction
-		(at 86.36 96.52)
-		(diameter 0)
-		(color 0 0 0 0)
-	)
-	(junction
-		(at 86.36 111.76)
-		(diameter 0)
-		(color 0 0 0 0)
-	)
-	(junction
 		(at 104.14 114.3)
 		(diameter 0)
@@
 	)
 	(junction
-		(at 101.6 111.76)
-		(diameter 0)
-		(color 0 0 0 0)
-	)
-	(junction
 		(at 191.77 96.52)
 		(diameter 0)
@@
 	)
 	(junction
-		(at 86.36 116.84)
-		(diameter 0)
-		(color 0 0 0 0)
-	)
-	(junction
-		(at 101.6 91.44)
-		(diameter 0)
-		(color 0 0 0 0)
-	)
-	(junction
 		(at 83.82 129.54)
 		(diameter 0)
@@
 	)
 	(junction
-		(at 86.36 99.06)
-		(diameter 0)
-		(color 0 0 0 0)
-	)
-	(junction
 		(at 182.88 111.76)
 		(diameter 0)
@@
 	)
 	(junction
-		(at 101.6 134.62)
-		(diameter 0)
-		(color 0 0 0 0)
-	)
-	(junction
-		(at 101.6 116.84)
-		(diameter 0)
-		(color 0 0 0 0)
-	)
-	(junction
 		(at 130.81 66.04)
-		(diameter 0)
-		(color 0 0 0 0)
-	)
-	(junction
-		(at 86.36 127)
 		(diameter 0)
 		(color 0 0 0 0)
@@
 	(wire
 		(pts
-			(xy 86.36 124.46) (xy 101.6 124.46)
-		)
-		(stroke
-			(width 0)
-			(type default)
-		)
-	)
-	(wire
-		(pts
 			(xy 55.88 74.93) (xy 55.88 76.2)
 		)
@@
 	(wire
 		(pts
-			(xy 86.36 109.22) (xy 101.6 109.22)
-		)
-		(stroke
-			(width 0)
-			(type default)
-		)
-	)
-	(wire
-		(pts
 			(xy 101.6 88.9) (xy 113.03 88.9)
 		)
@@
 	(wire
 		(pts
-			(xy 86.36 132.08) (xy 101.6 132.08)
-		)
-		(stroke
-			(width 0)
-			(type default)
-		)
-	)
-	(wire
-		(pts
 			(xy 83.82 93.98) (xy 83.82 114.3)
 		)
@@
 	(wire
 		(pts
-			(xy 86.36 127) (xy 101.6 127)
-		)
-		(stroke
-			(width 0)
-			(type default)
-		)
-	)
-	(wire
-		(pts
 			(xy 191.77 107.95) (xy 191.77 114.3)
 		)
@@
 	(wire
 		(pts
-			(xy 86.36 96.52) (xy 101.6 96.52)
-		)
-		(stroke
-			(width 0)
-			(type default)
-		)
-	)
-	(wire
-		(pts
 			(xy 231.14 109.22) (xy 231.14 96.52)
 		)
@@
 	(wire
 		(pts
-			(xy 86.36 119.38) (xy 101.6 119.38)
-		)
-		(stroke
-			(width 0)
-			(type default)
-		)
-	)
-	(wire
-		(pts
 			(xy 55.88 96.52) (xy 86.36 96.52)
 		)
@@
 	(wire
 		(pts
-			(xy 86.36 88.9) (xy 101.6 88.9)
-		)
-		(stroke
-			(width 0)
-			(type default)
-		)
-	)
-	(wire
-		(pts
 			(xy 101.6 134.62) (xy 113.03 134.62)
 		)
@@
 	(wire
 		(pts
-			(xy 86.36 134.62) (xy 101.6 134.62)
-		)
-		(stroke
-			(width 0)
-			(type default)
-		)
-	)
-	(wire
-		(pts
 			(xy 219.71 125.73) (xy 219.71 124.46)
 		)
@@
 	(wire
 		(pts
-			(xy 86.36 111.76) (xy 101.6 111.76)
-		)
-		(stroke
-			(width 0)
-			(type default)
-		)
-	)
-	(wire
-		(pts
 			(xy 104.14 93.98) (xy 104.14 114.3)
 		)
@@
 	(wire
 		(pts
-			(xy 86.36 116.84) (xy 101.6 116.84)
-		)
-		(stroke
-			(width 0)
-			(type default)
-		)
-	)
-	(wire
-		(pts
 			(xy 35.56 116.84) (xy 62.23 116.84)
 		)
@@
 	(wire
 		(pts
-			(xy 86.36 99.06) (xy 101.6 99.06)
-		)
-		(stroke
-			(width 0)
-			(type default)
-		)
-	)
-	(wire
-		(pts
 			(xy 260.35 111.76) (xy 229.87 111.76)
 		)
@@
 		)
 		(stroke
-			(width 0)
-			(type default)
-		)
-	)
-	(wire
-		(pts
-			(xy 86.36 91.44) (xy 101.6 91.44)
-		)
-		(stroke

Commit message: new power rail YAY
Connections:
- net +VBUS renamed +5V
Other:
- note removed: "BOOST CONVERTER TO 5V??? JLC: "boost 5V", QX2303L50E maybe"
Changed lines of the file:
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@@
 	(generator_version "10.0")
 	(paper "A4")
-	(text "BOOST CONVERTER TO 5V??? JLC: \"boost 5V\", QX2303L50E maybe"
-		(exclude_from_sim no)
-		(at 124.206 36.576 0)
-		(effects
-			(font
-				(size 2.54 2.54)
-			)
-		)
-	)
 	(text "Current limit resistor!"
 		(exclude_from_sim no)
@@
 	)
 	(symbol
-		(lib_id "power:+1V0")
-		(at 260.35 93.98 0)
+		(lib_id "Device:C")
+		(at 236.22 101.6 0)
 		(unit 1)
 		(body_style 1)
@@
 		(dnp no)
 		(fields_autoplaced yes)
-		(property "Reference" "#PWR085"
-			(at 260.35 97.79 0)
-			(hide yes)
+		(property "Reference" "C122"
+			(at 240.03 100.3299 0)
 			(show_name no)
 			(do_not_autoplace no)
@@
 					(size 1.27 1.27)
 				)
+				(justify left)
 			)
 		)
-		(property "Value" "+VBUS"
-			(at 260.35 88.9 0)
+		(property "Value" "100n"
+			(at 240.03 102.8699 0)
 			(show_name no)
 			(do_not_autoplace no)
@@
 					(size 1.27 1.27)
 				)
+				(justify left)
 			)
 		)
-		(property "Footprint" ""
-			(at 260.35 93.98 0)
+		(property "Footprint" "Capacitor_SMD:C_0402_1005Metric"
+			(at 237.1852 105.41 0)
 			(hide yes)
 			(show_name no)
@@
 		)
 		(property "Datasheet" ""
-			(at 260.35 93.98 0)
+			(at 236.22 101.6 0)
 			(hide yes)
 			(show_name no)
@@
 			)
 		)
-		(property "Description" "Power symbol creates a global label with name \"+1V0\""
-			(at 260.35 93.98 0)
+		(property "Description" "Unpolarized capacitor"
+			(at 236.22 101.6 0)
 			(hide yes)
 			(show_name no)
@@
 			)
 		)
+		(pin "2"
+		)
 		(pin "1"
 		)
 		(instances
-			(project "PCB"
+			(project ""
 				(path "/ed0095eb-57a0-4856-9ac4-7b40bd214a3a/e0bb63a6-1743-4d45-83e3-83dd5e1cd35c"
-					(reference "#PWR085")
+					(reference "C122")
 					(unit 1)
 				)
@@
 	)
 	(symbol
-		(lib_id "Device:C")
-		(at 236.22 101.6 0)
+		(lib_id "power:+5V")
+		(at 123.19 53.34 0)
 		(unit 1)
 		(body_style 1)
@@
 		(dnp no)
 		(fields_autoplaced yes)
-		(property "Reference" "C122"
-			(at 240.03 100.3299 0)
+		(property "Reference" "#PWR0137"
+			(at 123.19 57.15 0)
+			(hide yes)
 			(show_name no)
 			(do_not_autoplace no)
@@
 					(size 1.27 1.27)
 				)
-				(justify left)
 			)
 		)
-		(property "Value" "100n"
-			(at 240.03 102.8699 0)
+		(property "Value" "+5V"
+			(at 123.19 48.26 0)
 			(show_name no)
 			(do_not_autoplace no)
@@
 					(size 1.27 1.27)
 				)
-				(justify left)
 			)
 		)
-		(property "Footprint" "Capacitor_SMD:C_0402_1005Metric"
-			(at 237.1852 105.41 0)
+		(property "Footprint" ""
+			(at 123.19 53.34 0)
 			(hide yes)
 			(show_name no)
@@
 		)
 		(property "Datasheet" ""
-			(at 236.22 101.6 0)
+			(at 123.19 53.34 0)
 			(hide yes)
 			(show_name no)
@@
 			)
 		)
-		(property "Description" "Unpolarized capacitor"
-			(at 236.22 101.6 0)
+		(property "Description" "Power symbol creates a global label with name \"+5V\""
+			(at 123.19 53.34 0)
 			(hide yes)
 			(show_name no)
@@
 			)
 		)
-		(pin "2"
-		)
 		(pin "1"
 		)
 		(instances
-			(project ""
+			(project "PCB"
 				(path "/ed0095eb-57a0-4856-9ac4-7b40bd214a3a/e0bb63a6-1743-4d45-83e3-83dd5e1cd35c"
-					(reference "C122")
+					(reference "#PWR0137")
 					(unit 1)
 				)
@@
 	)
 	(symbol
-		(lib_id "power:+1V0")
-		(at 123.19 53.34 0)
+		(lib_id "power:GND")
+		(at 219.71 125.73 0)
 		(unit 1)
 		(body_style 1)
@@
 		(dnp no)
 		(fields_autoplaced yes)
-		(property "Reference" "#PWR076"
-			(at 123.19 57.15 0)
+		(property "Reference" "#PWR078"
+			(at 219.71 132.08 0)
 			(hide yes)
 			(show_name no)
@@
 			)
 		)
-		(property "Value" "+VBUS"
-			(at 123.19 48.26 0)
+		(property "Value" "GND"
+			(at 219.71 130.81 0)
 			(show_name no)
 			(do_not_autoplace no)
@@
 		)
 		(property "Footprint" ""
-			(at 123.19 53.34 0)
+			(at 219.71 125.73 0)
 			(hide yes)
 			(show_name no)
@@
 		)
 		(property "Datasheet" ""
-			(at 123.19 53.34 0)
+			(at 219.71 125.73 0)
 			(hide yes)
 			(show_name no)
@@
 			)
 		)
-		(property "Description" "Power symbol creates a global label with name \"+1V0\""
-			(at 123.19 53.34 0)
+		(property "Description" "Power symbol creates a global label with name \"GND\" , ground"
+			(at 219.71 125.73 0)
 			(hide yes)
 			(show_name no)
@@
 		)
 		(instances
-			(project "PCB"
+			(project ""
 				(path "/ed0095eb-57a0-4856-9ac4-7b40bd214a3a/e0bb63a6-1743-4d45-83e3-83dd5e1cd35c"
-					(reference "#PWR076")
+					(reference "#PWR078")
 					(unit 1)
 				)
@@
 	)
 	(symbol
-		(lib_id "power:GND")
-		(at 219.71 125.73 0)
+		(lib_id "Device:C_Small")
+		(at 71.12 134.62 90)
 		(unit 1)
 		(body_style 1)
@@
 		(in_pos_files yes)
 		(dnp no)
-		(fields_autoplaced yes)
-		(property "Reference" "#PWR078"
-			(at 219.71 132.08 0)
-			(hide yes)
+		(property "Reference" "C14"
+			(at 73.66 133.604 90)
 			(show_name no)
 			(do_not_autoplace no)
 			(effects
 				(font
-					(size 1.27 1.27)
+					(size 1.016 1.016)
 				)
 			)
 		)
-		(property "Value" "GND"
-			(at 219.71 130.81 0)
+		(property "Value" "100n"
+			(at 68.072 133.604 90)
 			(show_name no)
 			(do_not_autoplace no)
 			(effects
 				(font
-					(size 1.27 1.27)
+					(size 1.016 1.016)
 				)
 			)
 		)
-		(property "Footprint" ""
-			(at 219.71 125.73 0)
+		(property "Footprint" "Capacitor_SMD:C_0402_1005Metric"
+			(at 71.12 134.62 0)
 			(hide yes)
 			(show_name no)
@@
 		)
 		(property "Datasheet" ""
-			(at 219.71 125.73 0)
+			(at 71.12 134.62 0)
 			(hide yes)
 			(show_name no)
@@
 			)
 		)
-		(property "Description" "Power symbol creates a global label with name \"GND\" , ground"
-			(at 219.71 125.73 0)
+		(property "Description" "Unpolarized capacitor, small symbol"
+			(at 71.12 134.62 0)
 			(hide yes)
 			(show_name no)
@@
 			)
 		)
+		(pin "2"
+		)
 		(pin "1"
 		)
 		(instances
-			(project ""
+			(project "PCB"
 				(path "/ed0095eb-57a0-4856-9ac4-7b40bd214a3a/e0bb63a6-1743-4d45-83e3-83dd5e1cd35c"
-					(reference "#PWR078")
+					(reference "C14")
 					(unit 1)
 				)
@@
 	)
 	(symbol
-		(lib_id "Device:C_Small")
-		(at 71.12 134.62 90)
+		(lib_id "power:+5V")
+		(at 260.35 93.98 0)
 		(unit 1)
 		(body_style 1)
@@
 		(in_pos_files yes)
 		(dnp no)
-		(property "Reference" "C14"
-			(at 73.66 133.604 90)
+		(fields_autoplaced yes)
+		(property "Reference" "#PWR0138"
+			(at 260.35 97.79 0)
+			(hide yes)
 			(show_name no)
 			(do_not_autoplace no)
 			(effects
 				(font
-					(size 1.016 1.016)
+					(size 1.27 1.27)
 				)
 			)
 		)
-		(property "Value" "100n"
-			(at 68.072 133.604 90)
+		(property "Value" "+5V"
+			(at 260.35 88.9 0)
 			(show_name no)
 			(do_not_autoplace no)
 			(effects
 				(font
-					(size 1.016 1.016)
+					(size 1.27 1.27)
 				)
 			)
 		)
-		(property "Footprint" "Capacitor_SMD:C_0402_1005Metric"
-			(at 71.12 134.62 0)
+		(property "Footprint" ""
+			(at 260.35 93.98 0)
 			(hide yes)
 			(show_name no)
@@
 		)
 		(property "Datasheet" ""
-			(at 71.12 134.62 0)
+			(at 260.35 93.98 0)
 			(hide yes)
 			(show_name no)
@@
 			)
 		)
-		(property "Description" "Unpolarized capacitor, small symbol"
-			(at 71.12 134.62 0)
+		(property "Description" "Power symbol creates a global label with name \"+5V\""
+			(at 260.35 93.98 0)
 			(hide yes)
 			(show_name no)
@@
 			)
 		)
-		(pin "2"
-		)
 		(pin "1"
 		)
@@
 			(project "PCB"
 				(path "/ed0095eb-57a0-4856-9ac4-7b40bd214a3a/e0bb63a6-1743-4d45-83e3-83dd5e1cd35c"
-					(reference "C14")
+					(reference "#PWR0138")
 					(unit 1)
 				)

Commit message: more HDMI routing
Parts:
- J7: footprint Connector_Video:HDMI_Micro-D_Molex_46765-1xxx -> FPGA:Kai's_HDMI_Micro-D_Molex_46765-1xxx
Connections:
- net HDMI_CONN_D0-: now reaches J7.11 (D0-), U16.9
- net HDMI_CONN_CLK+: now reaches J7.12 (CK+), U16.7
- net HDMI_CONN_CLK-: now reaches J7.14 (CK-), U16.6
- net HDMI_CONN_D2+: now reaches J7.3 (D2+), U15.10
- net HDMI_CONN_D2-: now reaches J7.5 (D2-), U15.9
- net HDMI_CONN_D1+: now reaches J7.6 (D1+), U15.7
- net HDMI_CONN_D1-: now reaches J7.8 (D1-), U15.6
- net HDMI_CONN_D0+: now reaches J7.9 (D0+), U16.10
Other:
- moved on the sheet: C113, C114, C115, C116, C117, C119, C120, C121, C122, C123, C14, C16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

Commit message: FIRE HDMI shenanigans
Connections:
- net HDMI_CEC: now also J7.15 (CEC), U14.7
- net HDMI_CONN_CLK+: now also C16.2, U16.4
- net HDMI_CONN_CLK-: now also C14.2, U16.5
- net HDMI_CONN_D0+: now also C116.2, U15.4, U15.7; no longer U16.10
- net HDMI_CONN_D0-: now also C115.2, U15.5, U15.6; no longer U16.9
- net HDMI_CONN_D1+: now also C114.2, U16.1, U16.10; no longer U15.7
- net HDMI_CONN_D1-: now also C113.2, U16.2, U16.9; no longer U15.6
- net HDMI_CONN_D2+: now also C119.2, U15.1
- net HDMI_CONN_D2-: now also C117.2, U15.2
- net HDMI_D0+: now also C116.1; no longer C114.1
- net HDMI_D0-: now also C115.1; no longer C113.1
- net HDMI_D1+: now also C114.1; no longer C116.1
- net HDMI_D1-: now also C113.1; no longer C115.1
- net HDMI_SCL_5V: now also J7.17 (SCL), U14.2, U14.9; no longer U14.1
- net HDMI_SDA_5V: now also J7.18 (SDA), U14.1, U14.10; no longer U14.2
- net at R57.2, U14.5: now also J7.1 (HPD/HEAC-), U14.6

Commit message: going more insane with HDMI routing
Connections:
- net HDMI_SCL: now also R62.2, U12.4 (SDA1); no longer R61.2, U12.3 (SCL1)
- net HDMI_SCL_5V: now also R59.2, U12.5 (SDA2); no longer R60.2, U12.6 (SCL2)
- net HDMI_SDA: now also R61.2, U12.3 (SCL1); no longer R62.2, U12.4 (SDA1)
- net HDMI_SDA_5V: now also R60.2, U12.6 (SCL2); no longer R59.2, U12.5 (SDA2)
Changed lines of the file:
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@@
+		)
+	)
+	(label "HDMI_SDA"
+		(at 236.22 153.67 0)
+		(effects
+			(font
+				(size 1.27 1.27)
+			)
+			(justify left bottom)
 		)
 	)
@@
 		)
 	)
-	(label "HDMI_SDA_5V"
-		(at 346.71 156.21 180)
-		(effects
-			(font
-				(size 1.27 1.27)
-			)
-			(justify right bottom)
-		)
-	)
 	(label "HDMI_CLK-"
 		(at 77.47 177.8 0)
@@
 		)
 	)
-	(label "HDMI_CONN_D2-"
-		(at 148.59 154.94 0)
+	(label "HDMI_SCL_5V"
+		(at 346.71 156.21 180)
 		(effects
 			(font
 				(size 1.27 1.27)
 			)
-			(justify left bottom)
+			(justify right bottom)
 		)
 	)
-	(label "HDMI_SDA"
-		(at 236.22 156.21 0)
+	(label "HDMI_CONN_D2-"
+		(at 148.59 154.94 0)
 		(effects
 			(font
@@
 	(label "HDMI_CONN_CLK+"
 		(at 148.59 175.26 0)
-		(effects
-			(font
-				(size 1.27 1.27)
-			)
-			(justify left bottom)
-		)
-	)
-	(label "HDMI_SCL"
-		(at 236.22 153.67 0)
 		(effects
 			(font
@@
 		)
 	)
+	(label "HDMI_SCL"
+		(at 236.22 156.21 0)
+		(effects
+			(font
+				(size 1.27 1.27)
+			)
+			(justify left bottom)
+		)
+	)
 	(label "HDMI_CONN_D0+"
 		(at 148.59 160.02 0)
@@
 		)
 	)
-	(label "HDMI_SCL_5V"
+	(label "HDMI_SDA_5V"
 		(at 346.71 153.67 180)
 		(effects
