File: PCB/ethernet.kicad_sch (KiCad schematic)
At the start: 0 parts

Commit message: chose some good ethernet IC's
Parts:
- added J5: RJ45_Hanrun_HR911105A_Horizontal, Connector_RJ:RJ45_Hanrun_HR911105A_Horizontal, symbol Connector:RJ45_Hanrun_HR911105A_Horizontal
- added U13: LAN8710A, Package_DFN_QFN:QFN-32-1EP_5x5mm_P0.5mm_EP3.3x3.3mm_ThermalVias, symbol Interface_Ethernet:LAN8710A
Other:
- note added: "look at the ethernet IP in vivado to see if they support the chip"
Changed lines of the file:
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@@
 		(members "JTAG_TCK" "JTAG_TDI" "JTAG_TDO" "JTAG_TMS")
 	)
+	(text "look at the ethernet IP in vivado to see if they support the chip"
+		(exclude_from_sim no)
+		(at 167.64 48.26 0)
+		(effects
+			(font
+				(size 1.27 1.27)
+			)
+		)
+	)
+	(symbol
+		(lib_id "Connector:RJ45_Hanrun_HR911105A_Horizontal")
+		(at 100.33 96.52 0)
+		(unit 1)
+		(exclude_from_sim no)
+		(in_bom yes)
+		(on_board yes)
+		(dnp no)
+		(fields_autoplaced yes)
+		(property "Reference" "J5"
+			(at 101.6 82.55 0)
+			(effects
+				(font
+					(size 1.27 1.27)
+				)
+			)
+		)
+		(property "Value" "RJ45_Hanrun_HR911105A_Horizontal"
+			(at 101.6 85.09 0)
+			(effects
+				(font
+					(size 1.27 1.27)
+				)
+			)
+		)
+		(property "Footprint" "Connector_RJ:RJ45_Hanrun_HR911105A_Horizontal"
+			(at 100.33 83.82 0)
+			(effects
+				(font
+					(size 1.27 1.27)
+				)
+				(hide yes)
+			)
+		)
+		(property "Datasheet" "https://datasheet.lcsc.com/lcsc/1811141815_HANRUN-Zhongshan-HanRun-Elec-HR911105A_C12074.pdf"
+			(at 100.33 81.28 0)
+			(effects
+				(font
+					(size 1.27 1.27)
+				)
+				(hide yes)
+			)
+		)
+		(property "Description" "1 Port RJ45 Magjack Connector Through Hole 10/100 Base-T, AutoMDIX"
+			(at 100.33 96.52 0)
+			(effects
+				(font
+					(size 1.27 1.27)
+				)
+				(hide yes)
+			)
+		)
+		(pin "5"
+		)
+		(pin "3"
+		)
+		(pin "2"
+		)
+		(pin "8"
+		)
+		(pin "1"
+		)
+		(pin "4"
+		)
+		(pin "6"
+		)
+		(pin "SH"
+		)
+		(pin "11"
+		)
+		(pin "9"
+		)
+		(pin "10"
+		)
+		(pin "12"
+		)
+		(pin "7"
+		)
+		(instances
+			(project ""
+				(path "/ed0095eb-57a0-4856-9ac4-7b40bd214a3a/09aa8758-c80d-4d7c-89ed-08037b84af81"
+					(reference "J5")
+					(unit 1)
+				)
+			)
+		)
+	)
+	(symbol
+		(lib_id "Interface_Ethernet:LAN8710A")
+		(at 172.72 96.52 0)
+		(unit 1)
+		(exclude_from_sim no)
+		(in_bom yes)
+		(on_board yes)
+		(dnp no)
+		(fields_autoplaced yes)
+		(property "Reference" "U13"
+			(at 174.8633 132.08 0)
+			(effects
+				(font
+					(size 1.27 1.27)
+				)
+				(justify left)
+			)
+		)
+		(property "Value" "LAN8710A"
+			(at 174.8633 134.62 0)
+			(effects
+				(font
+					(size 1.27 1.27)
+				)
+				(justify left)
+			)
+		)
+		(property "Footprint" "Package_DFN_QFN:QFN-32-1EP_5x5mm_P0.5mm_EP3.3x3.3mm_ThermalVias"
+			(at 176.53 130.81 0)
+			(effects
+				(font
+					(size 1.27 1.27)
+				)
+				(justify left)
+				(hide yes)
+			)
+		)
+		(property "Datasheet" "http://ww1.microchip.com/downloads/en/DeviceDoc/8710a.pdf"
+			(at 170.18 120.65 0)
+			(effects
+				(font
+					(size 1.27 1.27)
+				)
+				(hide yes)
+			)
+		)
+		(property "Description" "LAN8710 Ethernet PHY with MII/RMII interface, QFN-32"
+			(at 172.72 96.52 0)
+			(effects
+				(font
+					(size 1.27 1.27)
+				)
+				(hide yes)
+			)
+		)
+		(pin "11"
+		)
+		(pin "9"
+		)
+		(pin "13"
+		)
+		(pin "26"
+		)
+		(pin "16"
+		)
+		(pin "20"
+		)
+		(pin "25"
+		)
+		(pin "10"
+		)
+		(pin "22"
+		)
+		(pin "23"
+		)
+		(pin "21"
+		)
+		(pin "24"
+		)
+		(pin "8"
+		)
+		(pin "7"
+		)
+		(pin "15"
+		)
+		(pin "14"
+		)
+		(pin "6"
+		)
+		(pin "3"
+		)
+		(pin "4"
+		)
+		(pin "29"
+		)
+		(pin "12"
+		)
+		(pin "1"
+		)
+		(pin "28"
+		)
+		(pin "27"
+		)
+		(pin "2"
+		)
+		(pin "19"
+		)
+		(pin "32"
+		)
+		(pin "30"
+		)
+		(pin "17"
+		)
+		(pin "33"
+		)
+		(pin "5"
+		)
+		(pin "31"
+		)
+		(pin "18"
+		)
+		(instances
+			(project ""
+				(path "/ed0095eb-57a0-4856-9ac4-7b40bd214a3a/09aa8758-c80d-4d7c-89ed-08037b84af81"
+					(reference "U13")
+					(unit 1)
+				)
+			)
+		)
+	)
 )

Commit message: crystal/LAN MPN's and starting to wire ethernet
Parts:
- added Y1: 25MHz, symbol Device:Crystal_GND24
- U13: value LAN8710A -> LAN8710A-EZC-TR; LCSC (none) -> C46185; MPN (none) -> LAN8710A-EZC-TR
Connections:
- net RJ45_TX+: now reaches J5.1 (TD+)
- net RJ45_TX+: now also U13.29 (TXP)
- net RJ45_TX-: now reaches J5.2 (TD-)
- net RJ45_TX-: now also U13.28 (TXN)
- net RJ45_RX+: now reaches J5.3 (RD+)
- net RJ45_RX+: now also U13.31 (RXP)
- net RJ45_RX-: now reaches J5.6 (RD-)
- net RJ45_RX-: now also U13.30 (RXN)
- new net GND: Y1.2, Y1.4
Other:
- moved on the sheet: J5, U13

Commit message: some more ethernet wiring
Parts:
- removed Y1: 25MHz, symbol Device:Crystal_GND24
- added R63: 12.1k, symbol Device:R
Connections:
- net GND: now also U13.24 (TXD2), U13.25 (TXD3), R63.2
- net PHY_RXD1: now reaches U13.10 (RXD1/~{MODE1})
- net PHY_RXD0: now reaches U13.11 (RXD0/~{MODE0})
- net PHY_TXD0: now reaches U13.22 (TXD0)
- net PHY_TXD1: now reaches U13.23 (TXD1)
- net at U13.32 (RBIAS): now also R63.1
- net RJ45_RX+ renamed PHY_RX+
- net RJ45_RX- renamed PHY_RX-
- net RJ45_TX+ renamed PHY_TX+
- net RJ45_TX- renamed PHY_TX-
- no-connect marks 0 -> 3
Other:
- note added: "No connects to GND instead?"
- note added: "Using RMII >"

Commit message: wiring ethernet power and other pins
Parts:
- removed U13: LAN8710A-EZC-TR, Package_DFN_QFN:QFN-32-1EP_5x5mm_P0.5mm_EP3.3x3.3mm_ThermalVias, symbol Interface_Ethernet:LAN8710A
- added C124, C126, C130, C132: 1u, symbol Device:C
- added C125: 470p, Capacitor_SMD:C_0603_1608Metric, symbol Device:C
- added C127, C128, C129, C131, C133: 100n, symbol Device:C
- added FB4: 120@100MHz, symbol Device:FerriteBead_Small
- added U13: LAN8710A-EZC-TR, Package_DFN_QFN:QFN-32-1EP_5x5mm_P0.5mm_EP3.3x3.3mm_ThermalVias, symbol FPGA Accelerator:LAN8710A
Connections:
- net GND: now also C124.1, C125.1, C126.2, C127.2, C128.2, C129.2, C130.2, C131.1, C132.1, C133.1, U13.24 (TXD2), U13.25 (TXD3), U13.33 (VSS)
- net PHY_RX+: now also U13.31 (RXP)
- net PHY_RX-: now also U13.30 (RXN)
- net PHY_RXD0: now also U13.11 (RXD0/~{MODE0})
- net PHY_RXD1: now also U13.10 (RXD1/~{MODE1})
- net PHY_TX+: now also U13.29 (TXP)
- net PHY_TX-: now also U13.28 (TXN)
- net PHY_TXD0: now also U13.22 (TXD0)
- net PHY_TXD1: now also U13.23 (TXD1)
- net +3V3: now reaches J5.4 (TCT)
- net +3V3: now also J5.5 (RCT), C129.1, C130.1, C131.2, C132.2, C133.2, FB4.1, U13.12 (VDDIO)
- net at R63.1: now also U13.32 (RBIAS)
- new net: C126.1, C127.1, C128.1, FB4.2, U13.1 (VDD2A), U13.27 (VDD1A)
- new net: C124.2, C125.2, U13.6 (VDDCR)
Other:
- note added: "< Internal regulator"
- note added: "< Is this much decoupling necessary?"
- moved on the sheet: J5, R63

Commit message: hopping off for the night
Parts:
- removed C132: 1u, symbol Device:C
- removed C133: 100n, symbol Device:C
- added R64, R65: 4k7, symbol Device:R
- added R66, R67: 1k, symbol Device:R
Connections:
- net +3V3: no longer C131.2, J5.4 (TCT), J5.5 (RCT)
- net GND: now also C131.2, J5.8, J5.SH; no longer C131.1
- net +3V3A: now reaches C126.1, C127.1, C128.1, FB4.2, U13.1 (VDD2A), U13.27 (VDD1A)
- net +3V3A: now also C131.1, J5.4 (TCT), J5.5 (RCT), R64.1, R65.1, R66.2, R67.2
- net PHY_LED2: now reaches J5.10
- net PHY_LED2: now also U13.2 (LED2/~{INTSEL}), R64.2
- net PHY_LED1: now reaches J5.11
- net PHY_LED1: now also U13.3 (LED1/~{REGOFF}), R65.2
- net at J5.12: now also R67.1
- net at J5.9: now also R66.1
Other:
- note added: "< Driving the 3V3 analog rail"
- note added: "QUADRUPLE CHECK LED WIRING"
- note removed: "< Is this much decoupling necessary?"
- note removed: "look at the ethernet IP in vivado to see if they support the chip"
- moved on the sheet: J5

Commit message: almost done wiring ethernet transceiver
Parts:
- added R68: 10k, symbol Device:R
- added R69: 4k7, symbol Device:R
- R64, R65: value 4k7 -> 10k
Connections:
- net +3V3: now also R68.2, R69.1
- net PHY_RXER: now reaches U13.13 (RXER/RXD4/~{PHYAD0})
- net PHY_CRS-DV: now reaches U13.15 (COL/CRS_DV/~{MODE2})
- net PHY_MDIO: now reaches U13.16 (MDIO)
- net PHY_MDIO: now also R69.2
- net PHY_MDC: now reaches U13.17 (MDC)
- net at U13.18 (~{INT}/TXER/TXD4): now also R68.1
- net PHY_TXEN: now reaches U13.21 (TXEN)
- no-connect marks 3 -> 6
Other:
- note added: "< LED's are pulled high and become active-low"
- note added: "Optional >"
- note removed: "No connects to GND instead?"
- note removed: "QUADRUPLE CHECK LED WIRING"
- moved on the sheet: C124, C125, C126, C127, C128, C129, C130, C131, FB4, J5, R63, R64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

Commit message: adding the transceiver crystal
Parts:
- added C132, C133: 18p, symbol Device:C
- added R70: 1M, symbol Device:R
- added Y1: 50MHz, symbol Device:Crystal_GND24
Connections:
- net GND: now also C132.1, C133.1, Y1.2, Y1.4
- net PHY_XTAL2: now reaches U13.4 (XTAL2)
- net PHY_XTAL2: now also C133.2, R70.2, Y1.1
- net PHY_XTAL1: now reaches U13.5 (XTAL1/CLKIN)
- net PHY_XTAL1: now also C132.2, R70.1, Y1.3
Other:
- moved on the sheet: C131, J5, R66, R67
