File: PCB/ethernet.kicad_sch (KiCad schematic)
At the start: 22 parts, among them J5 RJ45_Hanrun_HR911105A_Horizon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, U13 LAN8710A-EZC-TR, Y1 50MHz

Commit message: finished wiring the actual EPHY
Parts:
- removed R64: 10k, symbol Device:R
Connections:
- net PHY_nRST: now reaches U13.19 (~{RST})
Other:
- note removed: "Optional >"
- note removed: "Using RMII >"
- moved on the sheet: R65, R69

Commit message: kind of finished wiring ethernet, cleaning stuff up
Parts:
- added C134: 100n, symbol Device:C
- added R64: 4k7, symbol Device:R
- added SW2: SW_Push, symbol Switch:SW_Push
Connections:
- net +3V3: now also R64.1
- net GND: now also C134.2, SW2.1
- net PHY_nRST: now also C134.1, R64.2, SW2.2
Other:
- moved on the sheet: C124, C125, C126, C127, C128, C129, C130, C131, C132, C133, FB4, J5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

Commit message: adding some termination resistors and DNP's to EPHY
Parts:
- added C135, C136, C137, C138: 10p, symbol Device:C
- added R71, R72, R73, R74: 49.9, symbol Device:R
Connections:
- net +3V3A: now also R71.1, R72.1, R73.1, R74.1
- net GND: now also C135.2, C136.2, C137.2, C138.2
- net PHY_RX+: now also C137.1, R73.2
- net PHY_RX-: now also C138.1, R74.2
- net PHY_TX+: now also C135.1, R71.2
- net PHY_TX-: now also C136.1, R72.2
Other:
- note added: "100 Mbps, RMII Ethernet!"
- note added: "100 ohm termination, and optional EMI shunts!"
- note added: "< Internal pullup!"
- moved on the sheet: C124, C125, C126, C127, C128, C129, C130, C131, C132, C133, C134, FB4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

Commit message: basic HDMI ESD protection I think
Other:
- moved on the sheet: R65
Changed lines of the file:
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@@
 	(text "< Internal pullup!"
 		(exclude_from_sim no)
-		(at 195.58 149.86 0)
+		(at 198.12 149.86 0)
 		(effects
 			(font
@@
 	)
 	(junction
-		(at 170.18 147.32)
+		(at 171.45 147.32)
 		(diameter 0)
 		(color 0 0 0 0)
@@
 	(wire
 		(pts
-			(xy 170.18 144.78) (xy 170.18 147.32)
+			(xy 171.45 144.78) (xy 171.45 147.32)
 		)
 		(stroke
@@
 	(wire
 		(pts
-			(xy 170.18 135.89) (xy 170.18 137.16)
+			(xy 171.45 135.89) (xy 171.45 137.16)
 		)
 		(stroke
@@
 	(wire
 		(pts
-			(xy 170.18 147.32) (xy 165.1 147.32)
+			(xy 171.45 147.32) (xy 165.1 147.32)
 		)
 		(stroke
@@
 	(wire
 		(pts
-			(xy 170.18 147.32) (xy 184.15 147.32)
+			(xy 171.45 147.32) (xy 186.69 147.32)
 		)
 		(stroke
@@
 	(wire
 		(pts
-			(xy 165.1 149.86) (xy 184.15 149.86)
+			(xy 165.1 149.86) (xy 186.69 149.86)
 		)
 		(stroke
@@
 	)
 	(label "PHY_LED1"
-		(at 184.15 147.32 180)
+		(at 186.69 147.32 180)
 		(effects
 			(font
@@
 	)
 	(label "PHY_LED2"
-		(at 184.15 149.86 180)
+		(at 186.69 149.86 180)
 		(effects
 			(font
@@
 	(symbol
 		(lib_id "Device:R")
-		(at 170.18 140.97 0)
+		(at 171.45 140.97 0)
 		(unit 1)
 		(exclude_from_sim no)
@@
 		(fields_autoplaced yes)
 		(property "Reference" "R65"
-			(at 172.72 139.6999 0)
+			(at 173.99 139.6999 0)
 			(effects
 				(font
@@
 		)
 		(property "Value" "10k"
-			(at 172.72 142.2399 0)
+			(at 173.99 142.2399 0)
 			(effects
 				(font
@@
 		)
 		(property "Footprint" ""
-			(at 168.402 140.97 90)
+			(at 169.672 140.97 90)
 			(effects
 				(font
@@
 		)
 		(property "Datasheet" "~"
-			(at 170.18 140.97 0)
+			(at 171.45 140.97 0)
 			(effects
 				(font
@@
 		)
 		(property "Description" "Resistor"
-			(at 170.18 140.97 0)
+			(at 171.45 140.97 0)
 			(effects
 				(font
@@
 	(symbol
 		(lib_id "power:+3V3")
-		(at 170.18 135.89 0)
+		(at 171.45 135.89 0)
 		(unit 1)
 		(exclude_from_sim no)
@@
 		(fields_autoplaced yes)
 		(property "Reference" "#PWR0132"
-			(at 170.18 139.7 0)
+			(at 171.45 139.7 0)
 			(effects
 				(font
@@
 		)
 		(property "Value" "+3V3A"
-			(at 170.18 130.81 0)
+			(at 171.45 130.81 0)
 			(effects
 				(font
@@
 		)
 		(property "Footprint" ""
-			(at 170.18 135.89 0)
+			(at 171.45 135.89 0)
 			(effects
 				(font
@@
 		)
 		(property "Datasheet" ""
-			(at 170.18 135.89 0)
+			(at 171.45 135.89 0)
 			(effects
 				(font
@@
 		)
 		(property "Description" "Power symbol creates a global label with name \"+3V3\""
-			(at 170.18 135.89 0)
+			(at 171.45 135.89 0)
 			(effects
 				(font

Commit message: cleaning  up the schematic some more before sharing
Parts:
- removed C124: 1u, symbol Device:C
- removed C125: 470p, Capacitor_SMD:C_0603_1608Metric, symbol Device:C
- added C140: 470p, symbol Device:C
- added C141: 1u, symbol Device:C
Connections:
- net GND: now also C140.2, C141.2
- net at U13.6 (VDDCR): now also C140.1, C141.1
Other:
- note removed: "< Internal regulator"

Commit message: added basic capacitor footprints
Parts:
- C127, C128, C129, C131, C134: footprint (none) -> Capacitor_SMD:C_0402_1005Metric
- C140: footprint (none) -> Capacitor_SMD:C_0603_1608Metric
Changed lines of the file:
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@@
 			)
 		)
-		(property "Footprint" ""
+		(property "Footprint" "Capacitor_SMD:C_0402_1005Metric"
 			(at 72.0852 175.26 0)
 			(effects
@@
 			)
 		)
-		(property "Footprint" ""
+		(property "Footprint" "Capacitor_SMD:C_0402_1005Metric"
 			(at 286.7152 161.29 0)
 			(effects
@@
 			)
 		)
-		(property "Footprint" ""
+		(property "Footprint" "Capacitor_SMD:C_0402_1005Metric"
 			(at 167.3352 71.12 0)
 			(effects
@@
 			)
 		)
-		(property "Footprint" ""
+		(property "Footprint" "Capacitor_SMD:C_0402_1005Metric"
 			(at 154.6352 71.12 0)
 			(effects
@@
 			)
 		)
-		(property "Footprint" ""
+		(property "Footprint" "Capacitor_SMD:C_0402_1005Metric"
 			(at 126.6952 71.12 0)
 			(effects
@@
 			)
 		)
-		(property "Footprint" ""
+		(property "Footprint" "Capacitor_SMD:C_0603_1608Metric"
 			(at 158.4452 96.52 0)
 			(effects

Commit message: cleaning up ethernet, added some dampening resistors
Parts:
- added R78, R79, R80, R81, R82, R83, R84: 22, symbol Device:R_Small
Connections:
- net PHY_CRS-DV: now also R81.1; no longer U13.15 (COL/CRS_DV/~{MODE2})
- net PHY_RXD0: now also R78.1; no longer U13.11 (RXD0/~{MODE0})
- net PHY_RXD1: now also R79.1; no longer U13.10 (RXD1/~{MODE1})
- net PHY_RXER: now also R80.1; no longer U13.13 (RXER/RXD4/~{PHYAD0})
- net PHY_TXD0: now also R84.1; no longer U13.22 (TXD0)
- net PHY_TXD1: now also R83.1; no longer U13.23 (TXD1)
- net PHY_TXEN: now also R82.1; no longer U13.21 (TXEN)
- new net: R79.2, U13.10 (RXD1/~{MODE1})
- new net: R81.2, U13.15 (COL/CRS_DV/~{MODE2})
- new net: R83.2, U13.23 (TXD1)
- new net: R82.2, U13.21 (TXEN)
- new net: R84.2, U13.22 (TXD0)
- new net: R78.2, U13.11 (RXD0/~{MODE0})
- new net: R80.2, U13.13 (RXER/RXD4/~{PHYAD0})
Other:
- moved on the sheet: C134, R64, R69, SW2
