File: PCB/banks.kicad_sch (KiCad schematic)
At the start: 1 part, among them U1 XC7A50T-FGG484

Commit message: working on bank 13/14 configs
Parts:
- added R43, R44: 1k, symbol Device:R
Connections:
- net +3V3: now also U1.AA17 (VCCO_13), U1.AB14 (VCCO_13), U1.V16 (VCCO_13), U1.W13 (VCCO_13), U1.Y10 (VCCO_13), R43.1
- net at U1.U22 (IO_L3P_T0_DQS_PUDC_B_14): now also R43.2, R44.1
- new net GND: R44.2
- no-connect marks 0 -> 5
Other:
- note added: "Pull HIGH = disable internal I/O pullups Pull LOW = enable internal I/O pullups"
- moved on the sheet: U1B, U1C

Commit message: cleaninng up the board, fixing some pullups, PCIe command pins
Parts:
- added R45, R46: 10k, symbol Device:R
Connections:
- net +3V3: now also U1.G19 (VCCO_15), U1.H16 (VCCO_15), U1.J13 (VCCO_15), U1.K20 (VCCO_15), U1.L17 (VCCO_15), U1.N21 (VCCO_15), R45.1, R46.1; no longer U1.AA17 (VCCO_13), U1.AB14 (VCCO_13), U1.V16 (VCCO_13), U1.W13 (VCCO_13), U1.Y10 (VCCO_13)
- net ~{PCIe_CLKREQ}: now reaches U1.AA19 (IO_L15P_T2_DQS_RDWR_B_14)
- net ~{PCIe_CLKREQ}: now also R46.2
- net ~{PCIe_PERST}: now reaches U1.AB20 (IO_L15N_T2_DQS_DOUT_CSO_B_14)
- net ~{PCIe_PEWAKE}: now reaches U1.V17 (IO_L16P_T2_CSI_B_14)
- net ~{PCIe_PEWAKE}: now also R45.2
Other:
- note added: "< Can change to different pins if needed, just pin optimizing"
- note added: "No pullup on PERST for BOM optimizing! (very low leakage)"

Commit message: finished mid-difficulty configuration
Connections:
- no-connect marks 5 -> 10
Other:
- note added: "No weak pullup on PERST for BOM optimizing! (very low leakage)"
- note removed: "No pullup on PERST for BOM optimizing! (very low leakage)"
- moved on the sheet: U1B, U1C
Changed lines of the file:
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@@
 		(members "QSPI_DQ[0..3]" "QSPI_CS")
 	)
-	(text "No pullup on PERST for BOM optimizing! (very low leakage)"
+	(text "No weak pullup on PERST for BOM optimizing! (very low leakage)"
 		(exclude_from_sim no)
-		(at 160.274 172.72 0)
+		(at 161.544 172.72 0)
 		(effects
 			(font
@@
 	)
 	(junction
-		(at 463.55 68.58)
+		(at 294.64 68.58)
 		(diameter 0)
 		(color 0 0 0 0)
@@
 	)
 	(junction
-		(at 455.93 68.58)
+		(at 287.02 68.58)
 		(diameter 0)
 		(color 0 0 0 0)
 	)
 	(junction
-		(at 453.39 68.58)
+		(at 284.48 68.58)
 		(diameter 0)
 		(color 0 0 0 0)
@@
 	)
 	(junction
-		(at 458.47 68.58)
+		(at 289.56 68.58)
 		(diameter 0)
 		(color 0 0 0 0)
 	)
 	(junction
-		(at 461.01 68.58)
+		(at 292.1 68.58)
 		(diameter 0)
 		(color 0 0 0 0)
 	)
 	(no_connect
+		(at 271.78 166.37)
+	)
+	(no_connect
+		(at 271.78 204.47)
+	)
+	(no_connect
+		(at 271.78 209.55)
+	)
+	(no_connect
 		(at 127 115.57)
 	)
 	(no_connect
+		(at 271.78 212.09)
+	)
+	(no_connect
 		(at 127 105.41)
 	)
 	(no_connect
+		(at 271.78 207.01)
+	)
+	(no_connect
 		(at 127 107.95)
 	)
@@
 	(wire
 		(pts
-			(xy 453.39 68.58) (xy 453.39 69.85)
+			(xy 284.48 68.58) (xy 284.48 69.85)
 		)
 		(stroke
@@
 	(wire
 		(pts
-			(xy 463.55 66.04) (xy 463.55 68.58)
+			(xy 294.64 66.04) (xy 294.64 68.58)
 		)
 		(stroke
@@
 	(wire
 		(pts
-			(xy 461.01 68.58) (xy 463.55 68.58)
+			(xy 292.1 68.58) (xy 294.64 68.58)
 		)
 		(stroke
@@
 	(wire
 		(pts
-			(xy 458.47 68.58) (xy 458.47 69.85)
+			(xy 289.56 68.58) (xy 289.56 69.85)
 		)
 		(stroke
@@
 	(wire
 		(pts
-			(xy 463.55 68.58) (xy 463.55 69.85)
+			(xy 294.64 68.58) (xy 294.64 69.85)
 		)
 		(stroke
@@
 	(wire
 		(pts
-			(xy 455.93 68.58) (xy 455.93 69.85)
+			(xy 287.02 68.58) (xy 287.02 69.85)
 		)
 		(stroke
@@
 	(wire
 		(pts
-			(xy 450.85 68.58) (xy 450.85 69.85)
+			(xy 281.94 68.58) (xy 281.94 69.85)
 		)
 		(stroke
@@
 	(wire
 		(pts
-			(xy 455.93 68.58) (xy 458.47 68.58)
+			(xy 287.02 68.58) (xy 289.56 68.58)
 		)
 		(stroke
@@
 	(wire
 		(pts
-			(xy 458.47 68.58) (xy 461.01 68.58)
+			(xy 289.56 68.58) (xy 292.1 68.58)
 		)
 		(stroke
@@
 	(wire
 		(pts
-			(xy 461.01 68.58) (xy 461.01 69.85)
+			(xy 292.1 68.58) (xy 292.1 69.85)
 		)
 		(stroke
@@
 	(wire
 		(pts
-			(xy 450.85 68.58) (xy 453.39 68.58)
+			(xy 281.94 68.58) (xy 284.48 68.58)
 		)
 		(stroke
@@
 	(wire
 		(pts
-			(xy 453.39 68.58) (xy 455.93 68.58)
+			(xy 284.48 68.58) (xy 287.02 68.58)
 		)
 		(stroke
@@
 	(symbol
 		(lib_id "power:+3V3")
-		(at 463.55 66.04 0)
+		(at 294.64 66.04 0)
 		(unit 1)
 		(exclude_from_sim no)
@@
 		(fields_autoplaced yes)
 		(property "Reference" "#PWR063"
-			(at 463.55 69.85 0)
+			(at 294.64 69.85 0)
 			(effects
 				(font
@@
 		)
 		(property "Value" "+3V3"
-			(at 463.55 60.96 0)
+			(at 294.64 60.96 0)
 			(effects
 				(font
@@
 		)
 		(property "Footprint" ""
-			(at 463.55 66.04 0)
+			(at 294.64 66.04 0)
 			(effects
 				(font
@@
 		)
 		(property "Datasheet" ""
-			(at 463.55 66.04 0)
+			(at 294.64 66.04 0)
 			(effects
 				(font
@@
 		)
 		(property "Description" "Power symbol creates a global label with name \"+3V3\""
-			(at 463.55 66.04 0)
+			(at 294.64 66.04 0)
 			(effects
 				(font
@@
 	(symbol
 		(lib_id "FPGA Accelerator:XC7A50T-FGG484")
-		(at 491.49 143.51 0)
+		(at 322.58 143.51 0)
 		(unit 2)
 		(exclude_from_sim no)
@@
 		(fields_autoplaced yes)
 		(property "Reference" "U1"
-			(at 491.49 219.71 0)
+			(at 322.58 219.71 0)
 			(effects
 				(font
@@
 		)
 		(property "Value" "XC7A50T-FGG484"
-			(at 491.49 222.25 0)
+			(at 322.58 222.25 0)
 			(effects
 				(font
@@
 		)
 		(property "Footprint" "Package_BGA:Xilinx_FGG484"
-			(at 491.49 143.51 0)
+			(at 322.58 143.51 0)
 			(effects
 				(font
@@
 		)
 		(property "Datasheet" ""
-			(at 491.49 143.51 0)
+			(at 322.58 143.51 0)
 			(effects
 				(font
@@
 		)
 		(property "Description" "Artix 7 T 50 XC7A50T-FGG484"
-			(at 491.49 143.51 0)
+			(at 322.58 143.51 0)
 			(effects
 				(font
@@
 	(symbol
 		(lib_id "FPGA Accelerator:XC7A50T-FGG484")
-		(at 297.18 143.51 0)
+		(at 499.11 143.51 0)
 		(unit 3)
 		(exclude_from_sim no)
@@
 		(fields_autoplaced yes)
 		(property "Reference" "U1"
-			(at 297.18 219.71 0)
+			(at 499.11 219.71 0)
 			(effects
 				(font
@@
 		)
 		(property "Value" "XC7A50T-FGG484"
-			(at 297.18 222.25 0)
+			(at 499.11 222.25 0)
 			(effects
 				(font
@@
 		)
 		(property "Footprint" "Package_BGA:Xilinx_FGG484"
-			(at 297.18 143.51 0)
+			(at 499.11 143.51 0)
 			(effects
 				(font
@@
 		)
 		(property "Datasheet" ""
-			(at 297.18 143.51 0)
+			(at 499.11 143.51 0)
 			(effects
 				(font
@@
 		)
 		(property "Description" "Artix 7 T 50 XC7A50T-FGG484"
-			(at 297.18 143.51 0)
+			(at 499.11 143.51 0)
 			(effects
 				(font

Commit message: cleaning up the schematic some more, getting ready to wire the clocks, HDMI and ethernet!
Other:
- note added: "Most of the NC's are usable as I/O's too, even if they're configurations ;)"
- note removed: "No weak pullup on PERST for BOM optimizing! (very low leakage)"
Changed lines of the file:
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@@
 		(members "QSPI_DQ[0..3]" "QSPI_CS")
 	)
-	(text "No weak pullup on PERST for BOM optimizing! (very low leakage)"
+	(text "Most of the NC's are usable as I/O's too,\neven if they're configurations ;) "
 		(exclude_from_sim no)
-		(at 161.544 172.72 0)
+		(at 23.368 23.876 0)
 		(effects
 			(font
 				(size 1.27 1.27)
 			)
+			(justify left)
 		)
 	)

Commit message: cleaning up the schematic even more, it looks sick now
Changed lines of the file:
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@@
+		)
+	)
+	(hierarchical_label "{DDR_CLK}"
+		(shape output)
+		(at 400.05 54.61 0)
+		(effects
+			(font
+				(size 1.27 1.27)
+			)
+			(justify left)
 		)
 	)
@@
 		(effects
 			(font
+				(size 1.27 1.27)
+			)
+			(justify left)
+		)
+	)
+	(hierarchical_label "{DDR_ADDRESS}"
+		(shape bidirectional)
+		(at 400.05 46.99 0)
+		(effects
+			(font
+				(size 1.27 1.27)
+			)
+			(justify left)
+		)
+	)
+	(hierarchical_label "{DDR_COMMAND}"
+		(shape output)
+		(at 400.05 50.8 0)
+		(effects
+			(font
+				(size 1.27 1.27)
+			)
+			(justify left)
+		)
+	)
+	(hierarchical_label "{DDR_DATA}"
+		(shape bidirectional)
+		(at 400.05 58.42 0)
+		(effects
+			(font

Commit message: almost done wiring HDMI
Changed lines of the file:
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@@
+		)
+	)
+	(hierarchical_label "{HDMI}"
+		(shape bidirectional)
+		(at 400.05 66.04 0)
+		(effects
+			(font
+				(size 1.27 1.27)
+			)
+			(justify left)
 		)
 	)

Commit message: kind of finished wiring ethernet, cleaning stuff up
Changed lines of the file:
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@@
+		)
+	)
+	(hierarchical_label "{EPHY}"
+		(shape bidirectional)
+		(at 400.05 71.12 0)
+		(effects
+			(font
+				(size 1.27 1.27)
+			)
+			(justify left)
 		)
 	)

Commit message: wired the 100MHz clock for PLL's
Parts:
- added C139: 100n, symbol Device:C
- added R75: 22, symbol Device:R
- added Y3: 100MHz, Oscillator:Oscillator_SMD_SiT_PQFN-4Pin_5.0x3.2mm, symbol Oscillator:SiT8008xx-3x-xxE
Connections:
- net +3V3: now also C139.1, Y3.4 (Vdd)
- net GND: now also C139.2, Y3.2 (GND)
- new net: R75.1, Y3.3 (OUT)
- new net BUCK_PG4: Y3.1 (OE)
- new net CLK_100MHz: R75.2
Other:
- note added: "Wait for rails before starting the crystal! >"
