File: PCB/banks.kicad_sch (KiCad schematic)
At the start: 8 parts, among them U1 XC7A50T-FGG484, Y3 100MHz

Commit message: completely finished the clock, cleaned up the schematic
Connections:
- net +3V3: now also U1.AA17 (VCCO_13), U1.AB14 (VCCO_13), U1.V16 (VCCO_13), U1.W13 (VCCO_13), U1.Y10 (VCCO_13)
- net CLK_100MHz: now also U1.W19 (IO_L12P_T1_MRCC_14)
Other:
- note added: "Move if needed"
- moved on the sheet: R45, R46

Commit message: added UART debugging
Changed lines of the file:
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@@
+		)
+	)
+	(hierarchical_label "{UART}"
+		(shape bidirectional)
+		(at 400.05 77.47 0)
+		(effects
+			(font
+				(size 1.27 1.27)
+			)
+			(justify left)
 		)
 	)

Commit message: added basic capacitor footprints
Parts:
- C139: footprint (none) -> Capacitor_SMD:C_0402_1005Metric
Changed lines of the file:
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@@
 			)
 		)
-		(property "Footprint" ""
+		(property "Footprint" "Capacitor_SMD:C_0402_1005Metric"
 			(at 105.41 249.2248 0)
 			(effects

Commit message: buttons, more footprints, some other stuff
Parts:
- R75: footprint (none) -> Resistor_SMD:R_0402_1005Metric
Changed lines of the file:
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@@
 			)
 		)
-		(property "Footprint" ""
+		(property "Footprint" "Resistor_SMD:R_0402_1005Metric"
 			(at 114.3 264.668 90)
 			(effects

Commit message: adding most of the resistor footprints
Parts:
- R45, R46: footprint (none) -> Resistor_SMD:R_0402_1005Metric
Changed lines of the file:
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@@
 			)
 		)
-		(property "Footprint" ""
+		(property "Footprint" "Resistor_SMD:R_0402_1005Metric"
 			(at 144.272 154.94 90)
 			(effects
@@
 			)
 		)
-		(property "Footprint" ""
+		(property "Footprint" "Resistor_SMD:R_0402_1005Metric"
 			(at 153.162 154.94 90)
 			(effects

Commit message: finisehed upassigning resistor footprints
Parts:
- R43, R44: footprint (none) -> Resistor_SMD:R_0402_1005Metric
Changed lines of the file:
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@@
 			)
 		)
-		(property "Footprint" ""
+		(property "Footprint" "Resistor_SMD:R_0402_1005Metric"
 			(at 153.162 107.95 90)
 			(effects
@@
 			)
 		)
-		(property "Footprint" ""
+		(property "Footprint" "Resistor_SMD:R_0402_1005Metric"
 			(at 153.162 97.79 90)
 			(effects
