File: PCB/banks.kicad_sch (KiCad schematic)
At the start: 50 parts, among them U1 XC7A50T-FGG484, Y3 100MHz

Commit message: working on adding in the pin header
Connections:
- net HDMI_CEC: now also U1.A18 (IO_L17P_T2_16); no longer U1.A19 (IO_L17N_T2_16)
- net HDMI_HPD: now also U1.A19 (IO_L17N_T2_16); no longer U1.A18 (IO_L17P_T2_16)
Changed lines of the file:
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@@
+		)
+	)
+	(label "HDMI_HPD"
+		(at 377.19 176.53 180)
+		(effects
+			(font
+				(size 1.27 1.27)
+			)
+			(justify right bottom)
 		)
 	)
@@
 		)
 	)
-	(label "HDMI_HPD"
-		(at 377.19 173.99 180)
-		(effects
-			(font
-				(size 1.27 1.27)
-			)
-			(justify right bottom)
-		)
-	)
 	(label "HDMI_D0+"
 		(at 377.19 133.35 180)
@@
 		)
 	)
+	(label "HDMI_CEC"
+		(at 377.19 173.99 180)
+		(effects
+			(font
+				(size 1.27 1.27)
+			)
+			(justify right bottom)
+		)
+	)
 	(label "~{PCIe_PERST}"
 		(at 184.15 209.55 180)
@@
 		(effects
 			(font
-				(size 1.27 1.27)
-			)
-			(justify right bottom)
-		)
-	)
-	(label "HDMI_CEC"
-		(at 377.19 176.53 180)
-		(effects
-			(font

Commit message: routed a bunch of GPIO's, tuning up the USB 3V3 fill
Parts:
- added J5: Conn_02x05_Odd_Even, FPGA:PinHeader_2x05_P1.27mm_Vertical_SMD, symbol Connector_Generic:Conn_02x05_Odd_Even
Connections:
- net +3V3: now also J5.9 (Pin_9)
- net GND: now also J5.7 (Pin_7)
- net GPIO_0: now reaches U1.B22 (IO_L20N_T3_16)
- net GPIO_0: now also J5.10 (Pin_10)
- net GPIO_3: now reaches U1.C20 (IO_L19N_T3_VREF_16)
- net GPIO_3: now also J5.6 (Pin_6)
- net GPIO_4: now reaches U1.C22 (IO_L20P_T3_16)
- net GPIO_4: now also J5.4 (Pin_4)
- net GPIO_2: now reaches U1.D21 (IO_L23N_T3_16)
- net GPIO_2: now also J5.2 (Pin_2)
- net GPIO_1: now reaches U1.D22 (IO_L22N_T3_16)
- net GPIO_1: now also J5.8 (Pin_8)
- new net +5V: J5.1 (Pin_1)
- no-connect marks 179 -> 174

Commit message: All GPIO's routed!
Connections:
- net GPIO_6: now reaches J5.3 (Pin_3)
- net GPIO_6: now also U1.F15 (IO_0_16)
- net GPIO_5: now reaches J5.5 (Pin_5)
- net GPIO_5: now also U1.F16 (IO_L2P_T0_16)
- no-connect marks 174 -> 172
Changed lines of the file:
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@@
 	)
 	(no_connect
-		(at 363.22 90.17)
-	)
-	(no_connect
 		(at 654.05 107.95)
 	)
@@
 	)
 	(no_connect
-		(at 363.22 97.79)
-	)
-	(no_connect
 		(at 363.22 153.67)
 	)
@@
 	(wire
 		(pts
+			(xy 377.19 90.17) (xy 363.22 90.17)
+		)
+		(stroke
+			(width 0)
+			(type default)
+		)
+	)
+	(wire
+		(pts
 			(xy 384.81 49.53) (xy 392.43 49.53)
 		)
@@
 		)
 	)
+	(wire
+		(pts
+			(xy 193.04 259.08) (xy 208.28 259.08)
+		)
+		(stroke
+			(width 0)
+			(type default)
+		)
+	)
 	(bus
 		(pts
@@
 	(wire
 		(pts
+			(xy 377.19 97.79) (xy 363.22 97.79)
+		)
+		(stroke
+			(width 0)
+			(type default)
+		)
+	)
+	(wire
+		(pts
 			(xy 384.81 62.23) (xy 384.81 59.69)
 		)
@@
 	(wire
 		(pts
+			(xy 193.04 261.62) (xy 208.28 261.62)
+		)
+		(stroke
+			(width 0)
+			(type default)
+		)
+	)
+	(wire
+		(pts
 			(xy 474.98 204.47) (xy 552.45 204.47)
 		)
@@
 		)
 	)
+	(label "GPIO_6"
+		(at 377.19 90.17 180)
+		(effects
+			(font
+				(size 1.27 1.27)
+			)
+			(justify right bottom)
+		)
+	)
 	(label "DDR_A1"
 		(at 552.45 115.57 180)
@@
 		)
 	)
+	(label "GPIO_5"
+		(at 377.19 97.79 180)
+		(effects
+			(font
+				(size 1.27 1.27)
+			)
+			(justify right bottom)
+		)
+	)
 	(label "HDMI_D2+"
 		(at 377.19 138.43 180)
@@
 		)
 	)
+	(label "GPIO_6"
+		(at 193.04 259.08 0)
+		(effects
+			(font
+				(size 1.27 1.27)
+			)
+			(justify left bottom)
+		)
+	)
 	(label "HDMI_D1+"
 		(at 377.19 123.19 180)
@@
 		)
 	)
+	(label "GPIO_5"
+		(at 193.04 261.62 0)
+		(effects
+			(font
+				(size 1.27 1.27)
+			)
+			(justify left bottom)
+		)
+	)

Commit message: tuning stuff up, and fixing DRC!
Connections:
- net GPIO_0: now also J5.2 (Pin_2), U1.D21 (IO_L23N_T3_16); no longer J5.10 (Pin_10), U1.B22 (IO_L20N_T3_16)
- net GPIO_1: now also J5.3 (Pin_3), U1.F15 (IO_0_16); no longer J5.8 (Pin_8), U1.D22 (IO_L22N_T3_16)
- net GPIO_2: now also J5.4 (Pin_4), U1.C22 (IO_L20P_T3_16); no longer J5.2 (Pin_2), U1.D21 (IO_L23N_T3_16)
- net GPIO_3: now also J5.5 (Pin_5), U1.F16 (IO_L2P_T0_16); no longer J5.6 (Pin_6), U1.C20 (IO_L19N_T3_VREF_16)
- net GPIO_4: now also J5.6 (Pin_6), U1.C20 (IO_L19N_T3_VREF_16); no longer J5.4 (Pin_4), U1.C22 (IO_L20P_T3_16)
- net GPIO_5: now also J5.8 (Pin_8), U1.D22 (IO_L22N_T3_16); no longer J5.5 (Pin_5), U1.F16 (IO_L2P_T0_16)
- net GPIO_6: now also J5.10 (Pin_10), U1.B22 (IO_L20N_T3_16); no longer J5.3 (Pin_3), U1.F15 (IO_0_16)
Changed lines of the file:
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@@
+		)
+	)
+	(label "GPIO_3"
+		(at 193.04 261.62 0)
+		(effects
+			(font
+				(size 1.27 1.27)
+			)
+			(justify left bottom)
 		)
 	)
@@
 		)
 	)
-	(label "GPIO_1"
-		(at 377.19 201.93 180)
-		(effects
-			(font
-				(size 1.27 1.27)
-			)
-			(justify right bottom)
-		)
-	)
 	(label "DDR_BA0"
 		(at 552.45 138.43 180)
@@
 		)
 	)
-	(label "GPIO_0"
-		(at 377.19 191.77 180)
-		(effects
-			(font
-				(size 1.27 1.27)
-			)
-			(justify right bottom)
-		)
-	)
 	(label "DDR_DQ11"
 		(at 552.45 209.55 180)
@@
 		)
 	)
+	(label "GPIO_1"
+		(at 377.19 90.17 180)
+		(effects
+			(font
+				(size 1.27 1.27)
+			)
+			(justify right bottom)
+		)
+	)
 	(label "DDR_DQS1+"
 		(at 552.45 194.31 180)
@@
 		)
 	)
-	(label "GPIO_6"
-		(at 377.19 90.17 180)
-		(effects
-			(font
-				(size 1.27 1.27)
-			)
-			(justify right bottom)
-		)
-	)
 	(label "DDR_A1"
 		(at 552.45 115.57 180)
@@
 		)
 	)
-	(label "GPIO_2"
-		(at 232.41 256.54 180)
-		(effects
-			(font
-				(size 1.27 1.27)
-			)
-			(justify right bottom)
-		)
-	)
 	(label "~{PCIe_PEWAKE}"
 		(at 184.15 194.31 180)
@@
 		)
 	)
-	(label "GPIO_2"
-		(at 377.19 207.01 180)
-		(effects
-			(font
-				(size 1.27 1.27)
-			)
-			(justify right bottom)
-		)
-	)
 	(label "HDMI_D0+"
 		(at 377.19 133.35 180)
@@
 		)
 	)
-	(label "GPIO_3"
-		(at 232.41 261.62 180)
-		(effects
-			(font
-				(size 1.27 1.27)
-			)
-			(justify right bottom)
-		)
-	)
-	(label "GPIO_1"
-		(at 232.41 264.16 180)
-		(effects
-			(font
-				(size 1.27 1.27)
-			)
-			(justify right bottom)
-		)
-	)
 	(label "DDR_DQ10"
 		(at 552.45 204.47 180)
@@
 		)
 	)
+	(label "GPIO_2"
+		(at 377.19 189.23 180)
+		(effects
+			(font
+				(size 1.27 1.27)
+			)
+			(justify right bottom)
+		)
+	)
+	(label "GPIO_5"
+		(at 232.41 264.16 180)
+		(effects
+			(font
+				(size 1.27 1.27)
+			)
+			(justify right bottom)
+		)
+	)
 	(label "HDMI_CLK+"
 		(at 377.19 125.73 180)
@@
 		)
 	)
-	(label "GPIO_5"
-		(at 377.19 97.79 180)
-		(effects
-			(font
-				(size 1.27 1.27)
-			)
-			(justify right bottom)
-		)
-	)
 	(label "HDMI_D2+"
 		(at 377.19 138.43 180)
@@
 	)
 	(label "GPIO_0"
-		(at 232.41 266.7 180)
+		(at 232.41 256.54 180)
+		(effects
+			(font
+				(size 1.27 1.27)
+			)
+			(justify right bottom)
+		)
+	)
+	(label "GPIO_6"
+		(at 377.19 191.77 180)
+		(effects
+			(font
+				(size 1.27 1.27)
+			)
+			(justify right bottom)
+		)
+	)
+	(label "GPIO_4"
+		(at 232.41 261.62 180)
 		(effects
 			(font
@@
 		)
 	)
+	(label "GPIO_2"
+		(at 232.41 259.08 180)
+		(effects
+			(font
+				(size 1.27 1.27)
+			)
+			(justify right bottom)
+		)
+	)
+	(label "GPIO_0"
+		(at 377.19 207.01 180)
+		(effects
+			(font
+				(size 1.27 1.27)
+			)
+			(justify right bottom)
+		)
+	)
 	(label "~{DDR_CAS}"
 		(at 552.45 143.51 180)
@@
 		)
 	)
+	(label "GPIO_6"
+		(at 232.41 266.7 180)
+		(effects
+			(font
+				(size 1.27 1.27)
+			)
+			(justify right bottom)
+		)
+	)
 	(label "DDR_A4"
 		(at 552.45 105.41 180)
@@
 		)
 	)
-	(label "GPIO_3"
-		(at 377.19 186.69 180)
-		(effects
-			(font
-				(size 1.27 1.27)
-			)
-			(justify right bottom)
-		)
-	)
 	(label "DDR_A13"
 		(at 552.45 123.19 180)
@@
 		)
 	)
-	(label "GPIO_6"
-		(at 193.04 259.08 0)
-		(effects
-			(font
-				(size 1.27 1.27)
-			)
-			(justify left bottom)
+	(label "GPIO_4"
+		(at 377.19 186.69 180)
+		(effects
+			(font
+				(size 1.27 1.27)
+			)
+			(justify right bottom)
 		)
 	)
@@
 		)
 	)
+	(label "GPIO_1"
+		(at 193.04 259.08 0)
+		(effects
+			(font
+				(size 1.27 1.27)
+			)
+			(justify left bottom)
+		)
+	)
 	(label "DDR_DQ13"
 		(at 552.45 189.23 180)
@@
 		)
 	)
+	(label "GPIO_5"
+		(at 377.19 201.93 180)
+		(effects
+			(font
+				(size 1.27 1.27)
+			)
+			(justify right bottom)
+		)
+	)
 	(label "DDR_DQ4"
 		(at 552.45 156.21 180)
@@
 		)
 	)
-	(label "GPIO_5"
-		(at 193.04 261.62 0)
-		(effects
-			(font
-				(size 1.27 1.27)
-			)
-			(justify left bottom)
-		)
-	)
 	(label "DDR_A7"
 		(at 552.45 107.95 180)
@@
 		)
 	)
-	(label "GPIO_4"
-		(at 232.41 259.08 180)
+	(label "GPIO_3"
+		(at 377.19 97.79 180)
 		(effects
 			(font
@@
 		(effects
 			(font
-				(size 1.27 1.27)
-			)
-			(justify right bottom)
-		)
-	)
-	(label "GPIO_4"
-		(at 377.19 189.23 180)
-		(effects
-			(font

Commit message: working on programmable LED's
Parts:
- added D5, D6, D7: KT-0603G, LED_SMD:LED_0603_1608Metric, symbol Device:LED
- added R78, R79, R80: 1k, Resistor_SMD:R_0402_1005Metric, symbol Device:R
Connections:
- net GND: now also R78.2, R79.2, R80.2
- new net: D7.1 (K), R80.1
- new net: D5.1 (K), R78.1
- new net: D6.1 (K), R79.1

Commit message: routed all the programmable LED's
Connections:
- net GND: now also D5.1 (K), D6.1 (K), D7.1 (K); no longer R78.2, R79.2, R80.2
- net USER_LED_3: now reaches R80.1
- net USER_LED_3: now also U1.C13 (IO_L8P_T1_16); no longer D7.1 (K)
- net at D7.2 (A): now also R80.2
- net USER_LED_1: now reaches R78.1
- net USER_LED_1: now also U1.C19 (IO_L13N_T2_MRCC_16); no longer D5.1 (K)
- net at D5.2 (A): now also R78.2
- net USER_LED_2: now reaches R79.1
- net USER_LED_2: now also U1.F13 (IO_L1P_T0_16); no longer D6.1 (K)
- net at D6.2 (A): now also R79.2
- no-connect marks 172 -> 169
