File: PCB/usb.kicad_sch (KiCad schematic)
At the start: 40 parts, among them J4 USB_C_Receptacle_USB2.0_16P, J5 Conn_ARM_SWD_TagConnect_TC2030, U10 FT2232HQ, U3 TPD2EUSB30, U8 TPS62132, U9 M93C56-WMN6TP, Y2 12MHz

Commit message: created a JTAG bus
Parts:
- added R29, R32, R36, R37: 22, symbol Device:R
- added R38, R39, R40, R41: 10k, symbol Device:R
- added U4, U6: TPD2EUSB30, Package_TO_SOT_SMD:Texas_DRT-3, symbol Power_Protection:TPD2EUSB30
- J5: Alt_Value (none) -> TC2030 JTAG
Connections:
- net +3V3: now also R38.1, R39.1, R40.1, R41.1
- net GND: now also U4.3 (GND), U6.3 (GND)
- net 1V8_INTERNAL_LDO: now reaches C100.1, C102.1, C98.1, C99.1, U10.12 (VCORE), U10.37 (VCORE), U10.49 (VREGOUT), U10.64 (VCORE)
- net TCK: no longer names the net of J5.4 (SWCLK), U10.16 (ADBUS0)
- net TCK: now also R29.1, U6.2 (D-)
- net TDI: no longer names the net of J5.3 (~{RESET}), U10.17 (ADBUS1)
- net TDI: now also R32.1, U6.1 (D+)
- net TDO: no longer names the net of J5.6 (SWO), U10.18 (ADBUS2)
- net TDO: now also R36.1, U4.2 (D-)
- net TMS: no longer names the net of J5.2 (SWDIO), U10.19 (ADBUS3)
- net TMS: now also R37.1, U4.1 (D+)
- new net JTAG_TCK: R29.2, R38.2
- new net JTAG_TDI: R32.2, R39.2
- new net JTAG_TDO: R36.2, R40.2
- new net JTAG_TMS: R37.2, R41.2
Other:
- moved on the sheet: C100, C101, C102, C103, C104, C105, C106, C107, C108, C109, C87, C88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

Commit message: improving clarity, +JTAG ESD protection
Parts:
- removed J5: Conn_ARM_SWD_TagConnect_TC2030, Connector:Tag-Connect_TC2030-IDC-FP_2x03_P1.27mm_Vertical, symbol Connector:Conn_ARM_SWD_TagConnect_TC2030
- added J2: Conn_ARM_SWD_TagConnect_TC2030, Connector:Tag-Connect_TC2030-IDC-FP_2x03_P1.27mm_Vertical, symbol FPGA Accelerator:Conn_ARM_SWD_TagConnect_TC2030
Connections:
- net +3V3: now also J2.1 (VCC)
- net GND: now also J2.5 (GND)
- net at R36.1, U10.18 (ADBUS2), U4.2 (D-): now also J2.6 (SWO/TDO)
- net at R29.1, U10.16 (ADBUS0), U6.2 (D-): now also J2.4 (SWCLK/TCK)
- net at R32.1, U10.17 (ADBUS1), U6.1 (D+): now also J2.3 (~{RESET})
- net at R37.1, U10.19 (ADBUS3), U4.1 (D+): now also J2.2 (SWDIO/TMS)
Other:
- moved on the sheet: C100, C101, C102, C103, C104, C105, C106, C107, C108, C109, C93, C94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

Commit message: wired JTAG bus
Other:
- moved on the sheet: C100, C101, C102, C103, C104, C105, C106, C107, C108, C109, C87, C88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

Commit message: added the SPI net labels!
Other:
- note added: "UART and other pins on FT2232H"
Changed lines of the file:
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@@
+		)
+	)
+	(text "UART and other pins on FT2232H"
+		(exclude_from_sim no)
+		(at 281.94 224.79 0)
+		(effects
+			(font
+				(size 2.54 2.54)
+			)
 		)
 	)

Commit message: cleaning the schematic up
Changed lines of the file:
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@@
 	)
 	(hierarchical_label "{JTAG}"
-		(shape output)
+		(shape bidirectional)
 		(at 361.95 152.4 0)
 		(effects

Commit message: cleaning up the schematic even more, it looks sick now
Parts:
- J4: value USB_C_Receptacle_USB2.0_16P -> TYPE-C-31-M-12; LCSC (none) -> C165948; MPN (none) -> TYPE-C-31-M-12
Changed lines of the file:
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@@
 	(generator_version "9.0")
 	(paper "A3")
-	(bus_alias "JTAG"
-		(members "JTAG_TCK" "JTAG_TDI" "JTAG_TDO" "JTAG_TMS")
-	)
 	(text "1.5uH & 47uF for BOM optimization"
 		(exclude_from_sim no)
@@
 			)
 		)
-		(property "Value" "USB_C_Receptacle_USB2.0_16P"
+		(property "Value" "TYPE-C-31-M-12"
 			(at 35.56 22.86 0)
 			(effects
@@
 			(at 35.56 43.18 0)
 			(effects
+				(font
+					(size 1.27 1.27)
+				)
+				(hide yes)
+			)
+		)
+		(property "MPN" "TYPE-C-31-M-12"
+			(at 35.56 43.18 0)
+			(effects
+				(font
+					(size 1.27 1.27)
+				)
+				(hide yes)
+			)
+		)
+		(property "LCSC" "C165948"
+			(at 35.56 43.18 0)
+			(effects

Commit message: wired the 100MHz clock for PLL's
Other:
- note added: "USB + UART??"
Changed lines of the file:
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@@
+		)
+	)
+	(text "USB + UART??"
+		(exclude_from_sim no)
+		(at 276.86 55.118 0)
+		(effects
+			(font
+				(size 2.54 2.54)
+			)
 		)
 	)
