File: PCB/usb.kicad_sch (KiCad schematic)
At the start: 50 parts, among them J2 Conn_ARM_SWD_TagConnect_TC2030, J4 TYPE-C-31-M-12, U10 FT2232HQ, U3 TPD2EUSB30, U4 TPD2EUSB30, U6 TPD2EUSB30, U8 TPS62132, U9 M93C56-WMN6TP, Y2 12MHz

Commit message: added UART debugging
Parts:
- added D2: LED, symbol Device:LED
- added R76: 1k, symbol Device:R
Connections:
- net +3V3: now also D2.2 (A)
- net GND: now also U10.13 (TEST)
- net at J2.6 (SWO/TDO), R36.1, U10.18 (ADBUS2): now also U4.1 (D+); no longer U4.2 (D-)
- net at J2.4 (SWCLK/TCK), R29.1, U10.16 (ADBUS0): now also U6.1 (D+); no longer U6.2 (D-)
- net at J2.3 (~{RESET}), R32.1, U10.17 (ADBUS1): now also U6.2 (D-); no longer U6.1 (D+)
- net at J2.2 (SWDIO/TMS), R37.1, U10.19 (ADBUS3): now also U4.2 (D-); no longer U4.1 (D+)
- net UART_TXD: now reaches U10.38 (BDBUS0)
- net UART_RXD: now reaches U10.39 (BDBUS1)
- net at U10.54 (BCBUS3): now also U10.55 (BCBUS4), R76.1
- new net: D2.1 (K), R76.2
- no-connect marks 2 -> 25
Other:
- note added: "< SELF POWERED?? Page 52"
- moved on the sheet: J2, U4, U6

Commit message: cleaned up the schematic, I think it just needs a couple of reviews now!
Connections:
- no-connect marks 25 -> 28
Other:
- note added: "Only have one plugged in at once!"
- note removed: "< SELF POWERED?? Page 52"
- note removed: "LCFilter?, Pg.10 >"
- note removed: "UART and other pins on FT2232H"
- note removed: "USB + UART??"
Changed lines of the file:
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@@
 		)
 	)
-	(text "< SELF POWERED?? Page 52 "
+	(text "Only have one plugged in at once!"
 		(exclude_from_sim no)
-		(at 219.964 246.888 0)
+		(at 244.094 173.99 0)
 		(effects
 			(font
 				(size 1.27 1.27)
-			)
-		)
-	)
-	(text "UART and other pins on FT2232H"
-		(exclude_from_sim no)
-		(at 516.636 170.18 0)
-		(effects
-			(font
-				(size 2.54 2.54)
-			)
-		)
-	)
-	(text "LCFilter?, Pg.10 >"
-		(exclude_from_sim no)
-		(at 111.252 115.57 0)
-		(effects
-			(font
-				(size 1.27 1.27)
+				(italic yes)
 			)
 		)
@@
 		)
 	)
-	(text "USB + UART??"
-		(exclude_from_sim no)
-		(at 276.86 55.118 0)
-		(effects
-			(font
-				(size 2.54 2.54)
-			)
-		)
-	)
 	(junction
 		(at 184.15 38.1)
@@
 	)
 	(no_connect
+		(at 199.39 254)
+	)
+	(no_connect
 		(at 199.39 190.5)
 	)
@@
 	)
 	(no_connect
+		(at 199.39 177.8)
+	)
+	(no_connect
+		(at 199.39 251.46)
+	)
+	(no_connect

Commit message: added basic capacitor footprints
Parts:
- C100, C101, C102, C103, C104, C105, C106, C107, C108, C109, C88, C90, C95, C99: footprint (none) -> Capacitor_SMD:C_0201_0603Metric
- C91, C94, C98: footprint (none) -> Capacitor_SMD:C_0603_1608Metric
- C93: footprint (none) -> Capacitor_SMD:C_0402_1005Metric
Changed lines of the file:
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@@
 			)
 		)
-		(property "Footprint" ""
+		(property "Footprint" "Capacitor_SMD:C_0201_0603Metric"
 			(at 120.3452 173.99 0)
 			(effects
@@
 			)
 		)
-		(property "Footprint" ""
+		(property "Footprint" "Capacitor_SMD:C_0201_0603Metric"
 			(at 149.5552 106.68 0)
 			(effects
@@
 			)
 		)
-		(property "Footprint" ""
+		(property "Footprint" "Capacitor_SMD:C_0603_1608Metric"
 			(at 177.4952 48.26 0)
 			(effects
@@
 			)
 		)
-		(property "Footprint" ""
+		(property "Footprint" "Capacitor_SMD:C_0402_1005Metric"
 			(at 63.5 212.3948 0)
 			(effects
@@
 			)
 		)
-		(property "Footprint" ""
+		(property "Footprint" "Capacitor_SMD:C_0201_0603Metric"
 			(at 93.6752 38.1 0)
 			(effects
@@
 			)
 		)
-		(property "Footprint" ""
+		(property "Footprint" "Capacitor_SMD:C_0201_0603Metric"
 			(at 169.8752 48.26 0)
 			(effects
@@
 			)
 		)
-		(property "Footprint" ""
+		(property "Footprint" "Capacitor_SMD:C_0201_0603Metric"
 			(at 131.7752 130.81 0)
 			(effects
@@
 			)
 		)
-		(property "Footprint" ""
+		(property "Footprint" "Capacitor_SMD:C_0201_0603Metric"
 			(at 140.6652 130.81 0)
 			(effects
@@
 			)
 		)
-		(property "Footprint" ""
+		(property "Footprint" "Capacitor_SMD:C_0201_0603Metric"
 			(at 140.6652 106.68 0)
 			(effects
@@
 			)
 		)
-		(property "Footprint" ""
+		(property "Footprint" "Capacitor_SMD:C_0201_0603Metric"
 			(at 127.9652 173.99 0)
 			(effects
@@
 			)
 		)
-		(property "Footprint" ""
+		(property "Footprint" "Capacitor_SMD:C_0201_0603Metric"
 			(at 190.1952 132.08 0)
 			(effects
@@
 			)
 		)
-		(property "Footprint" ""
+		(property "Footprint" "Capacitor_SMD:C_0201_0603Metric"
 			(at 101.2952 168.91 0)
 			(effects
@@
 			)
 		)
-		(property "Footprint" ""
+		(property "Footprint" "Capacitor_SMD:C_0603_1608Metric"
 			(at 112.7252 173.99 0)
 			(effects
@@
 			)
 		)
-		(property "Footprint" ""
+		(property "Footprint" "Capacitor_SMD:C_0201_0603Metric"
 			(at 199.0852 132.08 0)
 			(effects
@@
 			)
 		)
-		(property "Footprint" ""
+		(property "Footprint" "Capacitor_SMD:C_0201_0603Metric"
 			(at 207.9752 132.08 0)
 			(effects
@@
 			)
 		)
-		(property "Footprint" ""
+		(property "Footprint" "Capacitor_SMD:C_0201_0603Metric"
 			(at 135.5852 173.99 0)
 			(effects
@@
 			)
 		)
-		(property "Footprint" ""
+		(property "Footprint" "Capacitor_SMD:C_0201_0603Metric"
 			(at 216.8652 132.08 0)
 			(effects
@@
 			)
 		)
-		(property "Footprint" ""
+		(property "Footprint" "Capacitor_SMD:C_0603_1608Metric"
 			(at 93.6752 168.91 0)
 			(effects

Commit message: LED parts and inductor footprints
Parts:
- removed L6: 1.5u, symbol Device:L
- added L5: 1u5, Inductor_SMD:L_Sunlord_SWPA4030S, symbol Device:L
- D2: value LED -> KT-0805Y; footprint (none) -> LED_SMD:LED_0805_2012Metric; LCSC (none) -> C2296; MPN (none) -> KT-0805Y
Connections:
- net +VBUS_3V3: now also L5.2
- net at U8.1 (SW), U8.2 (SW), U8.3 (SW): now also L5.1
Other:
- moved on the sheet: R76

Commit message: buttons, more footprints, some other stuff
Parts:
- R29, R32, R36, R37: footprint (none) -> Resistor_SMD:R_0402_1005Metric
- Y2: footprint (none) -> Crystal:Crystal_SMD_3225-4Pin_3.2x2.5mm
Changed lines of the file:
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@@
 			)
 		)
-		(property "Footprint" ""
+		(property "Footprint" "Crystal:Crystal_SMD_3225-4Pin_3.2x2.5mm"
 			(at 125.73 243.84 0)
 			(effects
@@
 			)
 		)
-		(property "Footprint" ""
+		(property "Footprint" "Resistor_SMD:R_0402_1005Metric"
 			(at 293.37 166.878 90)
 			(effects
@@
 			)
 		)
-		(property "Footprint" ""
+		(property "Footprint" "Resistor_SMD:R_0402_1005Metric"
 			(at 293.37 169.418 90)
 			(effects
@@
 			)
 		)
-		(property "Footprint" ""
+		(property "Footprint" "Resistor_SMD:R_0402_1005Metric"
 			(at 293.37 161.798 90)
 			(effects
@@
 			)
 		)
-		(property "Footprint" ""
+		(property "Footprint" "Resistor_SMD:R_0402_1005Metric"
 			(at 293.37 164.338 90)
 			(effects

Commit message: adding most of the resistor footprints
Parts:
- R38, R39, R40, R41, R51, R53, R54: footprint (none) -> Resistor_SMD:R_0402_1005Metric
- R48, R49: value 5.1k -> 5k1
Changed lines of the file:
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@@
 			)
 		)
-		(property "Footprint" ""
+		(property "Footprint" "Resistor_SMD:R_0402_1005Metric"
 			(at 94.742 217.17 90)
 			(effects
@@
 	)
 	(symbol
+		(lib_id "Device:R")
+		(at 59.69 35.56 90)
+		(mirror x)
+		(unit 1)
+		(exclude_from_sim no)
+		(in_bom yes)
+		(on_board yes)
+		(dnp no)
+		(property "Reference" "R49"
+			(at 64.77 34.29 90)
+			(effects
+				(font
+					(size 1.27 1.27)
+				)
+			)
+		)
+		(property "Value" "5k1"
+			(at 54.356 34.29 90)
+			(effects
+				(font
+					(size 1.27 1.27)
+				)
+			)
+		)
+		(property "Footprint" ""
+			(at 59.69 33.782 90)
+			(effects
+				(font
+					(size 1.27 1.27)
+				)
+				(hide yes)
+			)
+		)
+		(property "Datasheet" "~"
+			(at 59.69 35.56 0)
+			(effects
+				(font
+					(size 1.27 1.27)
+				)
+				(hide yes)
+			)
+		)
+		(property "Description" "Resistor"
+			(at 59.69 35.56 0)
+			(effects
+				(font
+					(size 1.27 1.27)
+				)
+				(hide yes)
+			)
+		)
+		(pin "2"
+		)
+		(pin "1"
+		)
+		(instances
+			(project "PCB"
+				(path "/ed0095eb-57a0-4856-9ac4-7b40bd214a3a/b3feae67-f5ac-44a3-90a4-88fd0a4da47c"
+					(reference "R49")
+					(unit 1)
+				)
+			)
+		)
+	)
+	(symbol
 		(lib_id "Device:C")
 		(at 119.38 170.18 0)
@@
 			)
 		)
-		(property "Footprint" ""
+		(property "Footprint" "Resistor_SMD:R_0402_1005Metric"
 			(at 304.292 151.13 90)
 			(effects
@@
 	)
 	(symbol
-		(lib_id "Device:R")
-		(at 59.69 35.56 90)
-		(unit 1)
-		(exclude_from_sim no)
-		(in_bom yes)
-		(on_board yes)
-		(dnp no)
-		(property "Reference" "R49"
-			(at 64.77 37.084 90)
-			(effects
-				(font
-					(size 1.27 1.27)
-				)
-			)
-		)
-		(property "Value" "5.1k"
-			(at 54.356 37.084 90)
-			(effects
-				(font
-					(size 1.27 1.27)
-				)
-			)
-		)
-		(property "Footprint" ""
-			(at 59.69 37.338 90)
-			(effects
-				(font
-					(size 1.27 1.27)
-				)
-				(hide yes)
-			)
-		)
-		(property "Datasheet" "~"
-			(at 59.69 35.56 0)
-			(effects
-				(font
-					(size 1.27 1.27)
-				)
-				(hide yes)
-			)
-		)
-		(property "Description" "Resistor"
-			(at 59.69 35.56 0)
-			(effects
-				(font
-					(size 1.27 1.27)
-				)
-				(hide yes)
-			)
-		)
-		(pin "2"
-		)
-		(pin "1"
-		)
-		(instances
-			(project "PCB"
-				(path "/ed0095eb-57a0-4856-9ac4-7b40bd214a3a/b3feae67-f5ac-44a3-90a4-88fd0a4da47c"
-					(reference "R49")
-					(unit 1)
-				)
-			)
-		)
-	)
-	(symbol
 		(lib_id "Power_Protection:TPD2EUSB30")
 		(at 261.62 204.47 0)
@@
 			)
 		)
-		(property "Footprint" ""
+		(property "Footprint" "Resistor_SMD:R_0402_1005Metric"
 			(at 330.962 151.13 90)
 			(effects
@@
 			)
 		)
-		(property "Footprint" ""
+		(property "Footprint" "Resistor_SMD:R_0402_1005Metric"
 			(at 76.962 217.17 90)
 			(effects
@@
 			)
 		)
-		(property "Footprint" ""
+		(property "Footprint" "Resistor_SMD:R_0402_1005Metric"
 			(at 322.072 151.13 90)
 			(effects
@@
 		(dnp no)
 		(property "Reference" "R48"
-			(at 64.77 31.496 90)
+			(at 64.77 31.75 90)
 			(effects
 				(font
@@
 			)
 		)
-		(property "Value" "5.1k"
-			(at 54.356 31.496 90)
+		(property "Value" "5k1"
+			(at 54.356 31.75 90)
 			(effects
 				(font
@@
 			)
 		)
-		(property "Footprint" ""
+		(property "Footprint" "Resistor_SMD:R_0402_1005Metric"
 			(at 85.852 217.17 90)
 			(effects
@@
 			)
 		)
-		(property "Footprint" ""
+		(property "Footprint" "Resistor_SMD:R_0402_1005Metric"
 			(at 313.182 151.13 90)
 			(effects

Commit message: finisehed upassigning resistor footprints
Parts:
- C89: footprint (none) -> Capacitor_SMD:C_0603_1608Metric
- R48, R49, R50, R52, R55, R56, R76: footprint (none) -> Resistor_SMD:R_0402_1005Metric
Changed lines of the file:
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@@
 			)
 		)
-		(property "Footprint" ""
+		(property "Footprint" "Capacitor_SMD:C_0603_1608Metric"
 			(at 106.3752 49.53 0)
 			(effects
@@
 			)
 		)
-		(property "Footprint" ""
+		(property "Footprint" "Resistor_SMD:R_0402_1005Metric"
 			(at 59.69 33.782 90)
 			(effects
@@
 			)
 		)
-		(property "Footprint" ""
+		(property "Footprint" "Resistor_SMD:R_0402_1005Metric"
 			(at 130.81 199.898 90)
 			(effects
@@
 			)
 		)
-		(property "Footprint" ""
+		(property "Footprint" "Resistor_SMD:R_0402_1005Metric"
 			(at 209.55 240.538 90)
 			(effects
@@
 			)
 		)
-		(property "Footprint" ""
+		(property "Footprint" "Resistor_SMD:R_0402_1005Metric"
 			(at 130.81 194.818 90)
 			(effects
@@
 			)
 		)
-		(property "Footprint" ""
+		(property "Footprint" "Resistor_SMD:R_0402_1005Metric"
 			(at 59.69 31.242 90)
 			(effects
@@
 			)
 		)
-		(property "Footprint" ""
+		(property "Footprint" "Resistor_SMD:R_0402_1005Metric"
 			(at 153.162 41.91 90)
 			(effects
@@
 			)
 		)
-		(property "Footprint" ""
+		(property "Footprint" "Resistor_SMD:R_0402_1005Metric"
 			(at 85.09 235.458 90)
 			(effects
