File: PCB/usb.kicad_sch (KiCad schematic)
At the start: 39 parts, among them J2 Conn_ARM_SWD_TagConnect_TC2030, U10 FT2232HQ, U4 TPD2EUSB30, U6 TPD2EUSB30, U9 M93C56-WMN6TP, Y2 12MHz

Commit message: some JTAG shenanigans
Connections:
- net at J2.6 (SWO/TDO), R36.1, U10.18 (ADBUS2): now also U6.1 (D+); no longer U4.1 (D+)
- net at J2.4 (SWCLK/TCK), R29.1, U10.16 (ADBUS0): now also U4.2 (D-); no longer U6.1 (D+)
- net at J2.2 (SWDIO/TMS), R37.1, U10.19 (ADBUS3): now also U4.1 (D+); no longer U4.2 (D-)

Commit message: JTAG breakout
Connections:
- net at J2.6 (SWO/TDO), R36.1, U10.18 (ADBUS2): now also U6.2 (D-); no longer U6.1 (D+)
- net at J2.3 (~{RESET}), R32.1, U10.17 (ADBUS1): now also U6.1 (D+); no longer U6.2 (D-)
Changed lines of the file:
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@@
+	)
+	(junction
+		(at 281.94 153.67)
+		(diameter 0)
+		(color 0 0 0 0)
 	)
 	(junction
@@
 	)
 	(junction
+		(at 261.62 143.51)
+		(diameter 0)
+		(color 0 0 0 0)
+	)
+	(junction
 		(at 106.68 175.26)
 		(diameter 0)
@@
 	)
 	(junction
-		(at 281.94 143.51)
-		(diameter 0)
-		(color 0 0 0 0)
-	)
-	(junction
 		(at 342.9 109.22)
-		(diameter 0)
-		(color 0 0 0 0)
-	)
-	(junction
-		(at 261.62 153.67)
 		(diameter 0)
 		(color 0 0 0 0)
@@
 	(wire
 		(pts
-			(xy 281.94 143.51) (xy 281.94 167.64)
-		)
-		(stroke
-			(width 0)
-			(type default)
-		)
-	)
-	(wire
-		(pts
 			(xy 149.86 62.23) (xy 149.86 59.69)
 		)
@@
 	(wire
 		(pts
+			(xy 281.94 153.67) (xy 292.1 153.67)
+		)
+		(stroke
+			(width 0)
+			(type default)
+		)
+	)
+	(wire
+		(pts
 			(xy 184.15 228.6) (xy 186.69 228.6)
 		)
@@
 		)
 	)
-	(wire
-		(pts
-			(xy 281.94 143.51) (xy 284.48 143.51)
-		)
-		(stroke
-			(width 0)
-			(type default)
-		)
-	)
 	(bus
 		(pts
@@
 	(wire
 		(pts
-			(xy 236.22 153.67) (xy 261.62 153.67)
+			(xy 236.22 153.67) (xy 281.94 153.67)
 		)
 		(stroke
@@
 	(wire
 		(pts
+			(xy 281.94 153.67) (xy 281.94 167.64)
+		)
+		(stroke
+			(width 0)
+			(type default)
+		)
+	)
+	(wire
+		(pts
 			(xy 76.2 203.2) (xy 76.2 201.93)
 		)
@@
 	(wire
 		(pts
+			(xy 261.62 143.51) (xy 284.48 143.51)
+		)
+		(stroke
+			(width 0)
+			(type default)
+		)
+	)
+	(wire
+		(pts
 			(xy 140.97 96.52) (xy 149.86 96.52)
 		)
@@
 	(wire
 		(pts
-			(xy 261.62 153.67) (xy 292.1 153.67)
-		)
-		(stroke
-			(width 0)
-			(type default)
-		)
-	)
-	(wire
-		(pts
 			(xy 334.01 109.22) (xy 334.01 110.49)
 		)
@@
 	(wire
 		(pts
+			(xy 261.62 143.51) (xy 261.62 167.64)
+		)
+		(stroke
+			(width 0)
+			(type default)
+		)
+	)
+	(wire
+		(pts
 			(xy 217.17 97.79) (xy 217.17 95.25)
 		)
@@
 	(wire
 		(pts
-			(xy 236.22 143.51) (xy 281.94 143.51)
+			(xy 236.22 143.51) (xy 261.62 143.51)
 		)
 		(stroke
@@
 		)
 		(stroke
-			(width 0)
-			(type default)
-		)
-	)
-	(wire
-		(pts
-			(xy 261.62 153.67) (xy 261.62 167.64)
-		)
-		(stroke
