File: PCB/PCB.kicad_pcb (KiCad board)
At the start: 6 copper layers, 22 x 80 mm, 268 parts, among them J1 Bus_M.2_Edge_M, J2 Conn_ARM_SWD_TagConnect_TC2030, J4 TYPE-C-31-M-12, J7 HDMI_D_1.4, SW1 SW_Push, U1 XC7A50T-FGG484, U10 FT2232HQ, U11 MT41J128M16JT-125:K, U12 PCA9306DC1, U14 UCL0524P, U15 UCL0524P, U16 UCL0524P, U17 TPS62132, U2 MAX20029ATIA/V+, U3 TPD2EUSB30, U4 TPD2EUSB30, U5 TPS2121RUXR, U6 TPD2EUSB30, U7 MT25QL128ABA1EW7-0SIT, U9 M93C56-WMN6TP, Y2 12MHz, Y3 100MHz

Commit message: some huge layout improvements!
Parts:
- moved C132 31.6 mm to (136.2, 88.3)
- moved C88 26.8 mm to (134.4, 101.0), turned to -90 degrees
- moved C165 26.0 mm to (136.3, 109.7)
- moved C26 25.4 mm to (138.4, 98.0), turned to -90 degrees
- moved C140 24.4 mm to (143.0, 109.7)
- moved C34 23.1 mm to (138.2, 103.9)
- moved C167 1.88 mm to (138.1, 106.4)
- moved C166 1.86 mm to (135.1, 107.3)
- moved C169 1.41 mm to (140.3, 107.1)
- moved C141 1.39 mm to (140.6, 99.0), turned to 90 degrees
- moved C168 1.33 mm to (137.3, 108.1)
- moved C40 0.40 mm to (141.9, 107.0), turned to 90 degrees
- moved C138 0.12 mm to (140.2, 97.1)
- moved C144 0.10 mm to (140.2, 100.9)
- moved C31 0.09 mm to (143.1, 97.0)
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Routing:
- net +1V2: track 6.43 -> 7.74 mm
- net +3V3: track 42.3 -> 41.9 mm, vias 27 -> 37
- net GND: track 168.7 -> 168.8 mm, vias 153 -> 180
- net +1V8: track 13.3 -> 13.2 mm, vias 7 -> 13
- net +1V5: vias 44 -> 45
- net +1V0: vias 10 -> 17
- added copper zone on B.Cu, net +1V0
- added copper zone on B.Cu, net +1V8
- added copper zone on B.Cu, net +3V3

Commit message: all the FPGA decoupling layout and routing :D
Routing:
- net +3V3: vias 37 -> 43
- net GND: track 168.8 -> 168.9 mm, vias 180 -> 186
Changed lines of the file:
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@@
 	(footprint "Capacitor_SMD:C_0603_1608Metric"
 		(layer "B.Cu")
-		(at 139.1 90.2)
+		(at 139.1 90.25)
 		(descr "Capacitor SMD 0603 (1608 Metric), square (rectangular) end terminal, IPC-7351 nominal, (Body size source: IPC-SM-782 page 76, https://www.pcb-3d.com/wordpress/wp-content/uploads/ipc-sm-782a_amendment_1_and_2.pdf), generated with kicad-footprint-generator")
 		(tags "capacitor")
@@
 	)
 	(via
+		(at 135.75 100.45)
+		(size 0.45)
+		(drill 0.2)
+		(layers "F.Cu" "B.Cu")
+		(free yes)
+		(net "+3V3")
+	)
+	(via
 		(at 135.75 99.5)
 		(size 0.6)
@@
 	)
 	(via
+		(at 133.75 100.5)
+		(size 0.45)
+		(drill 0.2)
+		(layers "F.Cu" "B.Cu")
+		(free yes)
+		(net "+3V3")
+	)
+	(via
 		(at 137.75 107.5)
 		(size 0.6)
@@
 	)
 	(via
+		(at 138.75 87.55)
+		(size 0.45)
+		(drill 0.2)
+		(layers "F.Cu" "B.Cu")
+		(free yes)
+		(net "+3V3")
+	)
+	(via
+		(at 134.75 98.5)
+		(size 0.45)
+		(drill 0.2)
+		(layers "F.Cu" "B.Cu")
+		(free yes)
+		(net "+3V3")
+	)
+	(via
 		(at 141.834666 87.499999)
 		(size 0.6)
@@
 	)
 	(via
+		(at 134.75 100.45)
+		(size 0.45)
+		(drill 0.2)
+		(layers "F.Cu" "B.Cu")
+		(free yes)
+		(net "+3V3")
+	)
+	(via
 		(at 140.725 104.475)
 		(size 0.6)
@@
 	)
 	(via
+		(at 137.75 89.55)
+		(size 0.45)
+		(drill 0.2)
+		(layers "F.Cu" "B.Cu")
+		(free yes)
+		(net "+3V3")
+	)
+	(via
 		(at 136.9 110.7)
 		(size 0.45)
@@
 	)
 	(segment
-		(start 138.93 89.1)
-		(end 138.93 89.595)
-		(width 0.5)
-		(layer "B.Cu")
-		(net "+3V3")
-	)
-	(segment
 		(start 134.75 96.5)
 		(end 134.75 97.175)
@@
 	)
 	(segment
-		(start 138.93 89.595)
-		(end 138.325 90.2)
-		(width 0.5)
-		(layer "B.Cu")
-		(net "+3V3")
-	)
-	(segment
 		(start 135.75 91.5)
 		(end 135.75 92.225)
@@
 	)
 	(segment
+		(start 138.93 89.1)
+		(end 138.93 89.645)
+		(width 0.5)
+		(layer "B.Cu")
+		(net "+3V3")
+	)
+	(segment
 		(start 140.67 107.1)
 		(end 140.67 106.58)
@@
 	)
 	(segment
+		(start 138.93 89.645)
+		(end 138.325 90.25)
+		(width 0.5)
+		(layer "B.Cu")
+		(net "+3V3")
+	)
+	(segment
 		(start 140.93 105.2)
 		(end 140.93 104.68)
@@
 	)
 	(via
+		(at 133.75 87.5)
+		(size 0.45)
+		(drill 0.2)
+		(layers "F.Cu" "B.Cu")
+		(free yes)
+		(net "GND")
+	)
+	(via
 		(at 139.75 98.5)
 		(size 0.6)
@@
 	)
 	(via
+		(at 133.75 101.5)
+		(size 0.45)
+		(drill 0.2)
+		(layers "F.Cu" "B.Cu")
+		(free yes)
+		(net "GND")
+	)
+	(via
 		(at 136.05 66.7)
 		(size 0.45)
@@
 	)
 	(via
+		(at 133.75 89.5)
+		(size 0.45)
+		(drill 0.2)
+		(layers "F.Cu" "B.Cu")
+		(free yes)
+		(net "GND")
+	)
+	(via
 		(at 140.375 123.8)
 		(size 0.6)
@@
 	)
 	(via
+		(at 135.75 88.5)
+		(size 0.45)
+		(drill 0.2)
+		(layers "F.Cu" "B.Cu")
+		(free yes)
+		(net "GND")
+	)
+	(via
 		(at 144.7 75.05)
 		(size 0.45)
@@
 	)
 	(via
+		(at 134.75 89.5)
+		(size 0.45)
+		(drill 0.2)
+		(layers "F.Cu" "B.Cu")
+		(free yes)
+		(net "GND")
+	)
+	(via
 		(at 151.9 75.05)
 		(size 0.45)
@@
 	)
 	(via
+		(at 135.75 101.5)
+		(size 0.45)
+		(drill 0.2)
+		(layers "F.Cu" "B.Cu")
+		(free yes)
+		(net "GND")
+	)
+	(via
 		(at 135.02 76.79)
 		(size 0.45)
@@
 	)
 	(segment
+		(start 139.57 89.945)
+		(end 139.875 90.25)
+		(width 0.5)
+		(layer "B.Cu")
+		(net "GND")
+	)
+	(segment
 		(start 147.305 80.445)
 		(end 147.1 80.65)
@@
 	)
 	(segment
-		(start 139.57 89.895)
-		(end 139.875 90.2)
-		(width 0.5)
-		(layer "B.Cu")
-		(net "GND")
-	)
-	(segment
 		(start 142.3 79.85)
 		(end 141.68 79.85)
@@
 	)
 	(segment
+		(start 139.57 89.1)
+		(end 139.57 89.945)
+		(width 0.5)
+		(layer "B.Cu")
+		(net "GND")
+	)
+	(segment
 		(start 147.305 79.925)
 		(end 147.305 80.445)
@@
 	)
 	(segment
-		(start 139.57 89.1)
-		(end 139.57 89.895)
-		(width 0.5)
-		(layer "B.Cu")
-		(net "GND")
-	)
-	(segment
 		(start 148.6 96.3)
 		(end 148.775 96.475)
@@
 		(name "3V3")
 		(hatch edge 0.5)
+		(priority 9)
+		(connect_pads
+			(clearance 0.1)
+		)
+		(min_thickness 0.1)
+		(fill yes
+			(thermal_gap 0.1)
+			(thermal_bridge_width 0.5)
+			(island_removal_mode 0)
+		)
+		(polygon
+			(pts
+				(xy 137.05 90) (xy 139.25 90) (xy 139.25 88) (xy 138.35 87) (xy 137.05 87)
+			)
+		)
+	)
+	(zone
+		(net "+3V3")
+		(layer "B.Cu")
+		(name "3V3")
+		(hatch edge 0.5)
 		(priority 6)
 		(connect_pads
@@
 			)
 		)
+	)
+	(zone
+		(net "+3V3")
+		(layer "B.Cu")
+		(name "3V3")
+		(hatch edge 0.5)
+		(priority 8)
+		(connect_pads
+			(clearance 0.1)
+		)
+		(min_thickness 0.1)
+		(fill yes
+			(thermal_gap 0.1)
+			(thermal_bridge_width 0.5)
+			(island_removal_mode 0)
+		)
+		(polygon
+			(pts
+				(xy 133.25 101) (xy 136.25 101) (xy 136.25 98) (xy 133.25 98)
+			)
+		)
