File: PCB/PCB.kicad_pcb (KiCad board)
At the start: 6 copper layers, 22 x 80 mm, 266 parts, among them J1 Bus_M.2_Edge_M, J2 Conn_ARM_SWD_TagConnect_TC2030, J4 TYPE-C-31-M-12, J7 HDMI_D_1.4, SW1 SW_Push, U1 XC7A50T-FGG484, U10 FT2232HQ, U11 MT41J128M16JT-125:K, U12 PCA9306DC1, U14 UCL0524P, U15 UCL0524P, U16 UCL0524P, U17 TPS62132, U2 MAX20029ATIA/V+, U3 TPD2EUSB30, U4 TPD2EUSB30, U5 TPS2121RUXR, U6 TPD2EUSB30, U7 MT25QL128ABA1EW7-0SIT, U9 M93C56-WMN6TP, Y2 12MHz, Y3 100MHz

Commit message: removing the TC2030, doesn't make sense :/
Parts:
- removed J2: Conn_ARM_SWD_TagConnect_TC2030, Connector:Tag-Connect_TC2030-IDC-FP_2x03_P1.27mm_Vertical
- removed U4, U6: TPD2EUSB30, Package_TO_SOT_SMD:Texas_DRT-3
- moved C87 3.41 mm to (148.5, 67.0)
Routing:
- net GND: track 179.0 -> 173.9 mm, vias 205 -> 199
- net +VBUS: track 5.13 -> 0.00 mm, vias 6 -> 0
- net /USB to JTAG/USB_D+: track 5.03 -> 0.00 mm
- net /USB to JTAG/USB_D-: track 5.01 -> 0.00 mm
- net Net-(J4-CC1): track 2.69 -> 0.00 mm
- net Net-(J4-CC2): track 1.82 -> 0.00 mm
- net /Artix 7 Configurations and Flash/JTAG_TDO: track 3.51 -> 1.71 mm, vias 2 -> 1
- net Net-(U10-REF): track 1.21 -> 0.00 mm
- net Net-(U10-~{RESET}): track 1.10 -> 0.00 mm
- net +3V3: track 55.4 -> 54.3 mm
- net /Artix 7 Configurations and Flash/JTAG_TCK: track 4.03 -> 3.27 mm, vias 2 -> 1
- net /Artix 7 Configurations and Flash/JTAG_TDI: track 1.41 -> 0.71 mm, vias 2 -> 1

Commit message: nevermind, tc2030 is a good idea for a fallback breakout
Parts:
- added J2: Conn_ARM_SWD_TagConnect_TC2030, Connector:Tag-Connect_TC2030-IDC-FP_2x03_P1.27mm_Vertical, B.Cu at (150.8, 67.0)
- added U4: TPD2EUSB30, Package_TO_SOT_SMD:Texas_DRT-3, B.Cu at (146.3, 65.6)
- added U6: TPD2EUSB30, Package_TO_SOT_SMD:Texas_DRT-3, B.Cu at (146.3, 67.2)
- moved C87 3.41 mm to (146.3, 69.5)
Routing:
- net GND: track 173.9 -> 179.7 mm, vias 199 -> 206
- net +VBUS: track 0.00 -> 5.13 mm, vias 0 -> 6
- net /USB to JTAG/USB_D+: track 0.00 -> 5.03 mm
- net /USB to JTAG/USB_D-: track 0.00 -> 5.01 mm
- net Net-(J4-CC1): track 0.00 -> 2.69 mm
- net +3V3: track 54.3 -> 56.2 mm, vias 48 -> 49
- net Net-(J4-CC2): track 0.00 -> 1.82 mm
- net Net-(U10-REF): track 0.00 -> 1.21 mm
- net Net-(U10-~{RESET}): track 0.00 -> 1.10 mm
