File: PCB/PCB.kicad_pcb (KiCad board)
At the start: 6 copper layers, 22 x 80 mm, 266 parts, among them J1 Bus_M.2_Edge_M, J2 Conn_ARM_SWD_TagConnect_TC2030, J4 TYPE-C-31-M-12, J7 HDMI_D_1.4, SW1 SW_Push, U1 XC7A50T-FGG484, U10 FT2232HQ, U11 MT41J128M16JT-125:K, U12 PCA9306DC1, U14 UCL0524P, U15 UCL0524P, U16 UCL0524P, U17 TPS62132, U2 MAX20029ATIA/V+, U3 TPD2EUSB30, U4 TPD2EUSB30, U5 TPS2121RUXR, U6 TPD2EUSB30, U7 MT25QL128ABA1EW7-0SIT, U9 M93C56-WMN6TP, Y2 12MHz, Y3 100MHz

Commit message: a bunch more routing
Parts:
- moved R49 0.43 mm to (144.8, 65.8), turned to -90 degrees
- moved R56 0.17 mm to (143.9, 64.3)
- moved C105 0.12 mm to (143.3, 67.0)
- moved C103 0.10 mm to (141.4, 66.9)
- moved R39 0.08 mm to (143.6, 66.2)
- moved R40 0.06 mm to (142.6, 66.2)
Routing:
- net GND: track 175.2 -> 185.4 mm, vias 207 -> 220
- net Net-(J2-SWDIO/TMS): track 11.5 -> 19.8 mm
- net Net-(U10-OSCO): track 0.00 -> 4.03 mm, vias 0 -> 1
- net Net-(U10-OSCI): track 0.00 -> 4.03 mm, vias 0 -> 1
- net +VBUS: track 1.98 -> 5.40 mm
- net Net-(J2-SWCLK/TCK): track 8.55 -> 11.4 mm, vias 2 -> 3
- net /Artix 7 Configurations and Flash/JTAG_TDI: track 1.76 -> 4.56 mm, vias 1 -> 2
- net Net-(J4-CC1): track 0.00 -> 2.56 mm
- net /Artix 7 Configurations and Flash/JTAG_TDO: track 2.82 -> 4.95 mm, vias 1 -> 2
- net /Artix 7 Configurations and Flash/JTAG_TCK: track 4.23 -> 6.34 mm, vias 1 -> 2
- net /Artix 7 Configurations and Flash/JTAG_TMS: track 2.65 -> 4.61 mm, vias 1 -> 2
- net +3V3: track 56.9 -> 58.4 mm, vias 49 -> 50
- net Net-(U10-~{RESET}): track 0.00 -> 1.22 mm
- net Net-(U10-REF): track 0.00 -> 1.21 mm
- net Net-(J2-~{RESET}): track 17.8 -> 18.1 mm, vias 4 -> 5

Commit message: some more chill routing before bed
Parts:
- moved R19 1.22 mm to (139.9, 73.2), turned to -90 degrees
- moved C102 0.89 mm to (141.6, 73.1)
Routing:
- net +3V3: track 58.4 -> 67.0 mm, vias 50 -> 53
- net /USB to JTAG/1V8_INTERNAL_LDO: track 1.64 -> 10.2 mm, vias 1 -> 2
- net GND: track 185.4 -> 190.9 mm, vias 220 -> 222
- net /Artix 7 Banks/QSPI_DQ2: track 4.81 -> 0.00 mm, vias 1 -> 0
- net Net-(U10-EEDATA): track 0.00 -> 4.68 mm, vias 0 -> 1
- net Net-(U10-EECLK): track 0.00 -> 2.35 mm, vias 0 -> 1
- net Net-(U10-EECS): track 0.00 -> 1.46 mm, vias 0 -> 1
- net /Artix 7 Banks/QSPI_CS: track 3.87 -> 4.97 mm
- net /Artix 7 Configurations and Flash/JTAG_TCK: track 6.34 -> 5.58 mm
